Commit message: cad: the roll motor's plate is a separate bolt-on mount, its cheeks removed (forearm_roll_motor_mount, 4x M3x12 countersunk into captive nuts)
The forearm roll motor's vertical plate and its two cheeks were fused onto the top of the elbow block
(forearm_roll_block). That meant supports under a 48 mm overhang when the block prints front face down, and a reprint of
the whole block for any change to the mount. The mount is now its own printed part fastened with bolts and nuts, and
the cheeks are gone (they were judged unnecessary).

The motor's height is fixed by the 240-2GT roll belt, and its board sits only 3.4 mm above the block's top at the
nominal slot position (0.9 at the slot's low end). So the mount's base cannot sit on the top. Instead it fills a
mount_base_t (4) step cut into the block's top, from the rear face to the plate's front face + mount_fit (0.2). Its
top is where the block's top was, and the motor, the 20T, the belt and every station are unchanged. The base's
countersunk M3s sit flush under the motor, and their M3 nuts slide in along two channels from the block's rear face.
The mount therefore comes off with the arm assembled (motor first), and no nut can fall into the bore.

- lib/fasteners.py: M3_CSK (ISO 10642: d 3, dk 6.72, k 1.86, socket 2 x 1.1), M3_NUT (ISO 4032: 5.5 AF x 2.4),
  M3_PITCH, csk() (head top on z=0, cone + shank in +Z, length overall) and csk_volume(); re-exported by
  lib/params.py with ROLL_MOUNT_SCREWS_MASS_G 3.3 / ROLL_MOUNT_NUTS_MASS_G 1.4 g (the modelled steel).
- lib/forearm/params.py RollDriveParams: new mount_base_t 4, mount_fit 0.2, mount_bolt_x 20, mount_bolt_z (-34, 2),
  mount_screw (M3_CSK), mount_screw_len 12, mount_bolt_dia M3_CLEAR, mount_nut (M3_NUT), mount_nut_roof 3,
  mount_channel_add 0.3, mount_hole_past 0.5; cheek_t / cheek_h / cheek_gap removed.
- lib/forearm/layout.py stack_positions: y_step 32, z_step_riser 10.25, y_mount_nut 29, y_channel_floor 26.3,
  z_channel_end 5.175 (the front nut, pushed home, centred under its screw), y_mount_hole 23.5; z_cheek removed.
  New mount_bolt_points() (x +/-20, z -34 / 2).
- lib/forearm/roll.py:
  - build_block loses the plate, the cheeks and the slot cuts. It gains the step (full width), 4x Ø3.4 down to
    0.5 past the screw tips (3.5 mm off the core bore), and two nut channels 5.8 x 2.7 at x +/-20 along Z from the
    rear face (5.1 mm off the core bore). 5.7 mm of wall is left over the core bore.
  - New build_motor_mount: the base is the block's own rounded outline over the step, plus the 3 mm plate
    (unchanged: the tension slots and the pilot slot) and 4x 90 deg countersinks at the head's own cone.
- New parts: forearm_roll_motor_mount (NATIVE printed), forearm_roll_mount_screws / forearm_roll_mount_nuts (NATIVE
  COTS patterns, 4 solids each), rows of assemblies/forearm_roll_drive.py (the stator). The references were accepted
  (manifest 49 -> 52 entries): the mount 16548.628 mm^3, the screws 416.2, the nuts 183.6.
- forearm_roll_block re-accepted: 210853.072 -> 188631.310 mm^3; bbox y 119.926 -> 72.0 (the plate is the mount's now).
- assemblies/forearm_roll_drive.py EXPECTED:
  - module: leaves 8 -> 11, solids 23 -> 32, volume 424091.544 -> 419018.261;
  - stator: 7 / 22 / 328849.103 -> 10 / 31 / 323775.82;
  - rotor: unchanged.
- tests/test_assembly.py:
  - the roll module: 11 leaves, tints bought / printed 5 / 3 -> 7 / 4;
  - the arm: leaves 73 -> 76, solids 218 -> 227, tints 40 / 33 -> 42 / 34.
- tests/test_bom.py:
  - leaves 73 -> 76;
  - printed parts / qty 26 / 33 -> 27 / 34;
  - bought parts / occurrences 23 / 40 -> 25 / 42;
  - the roll drive's pieces + print set;
  - new test_the_roll_motor_mount_takes_its_m3_screws_and_nuts.

  MULTI_BODY gains the screws + nuts at 4 each.
- tests/forearm/test_roll_drive.py:
  - test_stack drops the cheek asserts and adds the mount's: its top level with the block's; 5 mm of wall under the
    step; the heads on the base's flat, behind the plate and inside the rear face; each tip 2 pitches past its nut;
    the holes and channels >= 2 mm off the core bore; the channels 2 mm before the cavity.
  - test_block_and_shaft_features probes the plate on the new leaf, nothing beside the motor, and the step,
    countersinks, holes and channels.
  - The rolling-forearm clearance test includes the mount.
- robot: elbow_link mass 0.74123 -> 0.738734 kg, COM (-6.259, -27.146, 19.133) -> (-6.251, -27.052, 19.118) mm,
  ixx / iyy / izz 1.342339e-3 / 7.914933e-4 / 1.296253e-3 -> 1.339249e-3 / 7.902239e-4 / 1.295333e-3 (arm.urdf and
  arm.sdf); meshes/elbow_link.stl re-exported. derive --check and validate --strict are clean.
- The hash gate against main's builds on this machine: only forearm_roll_block, forearm_roll_drive and arm STEPs changed.
- tools/bom.py EXTRAS: the roll motor's M3 x 8 now go "to the motor mount's plate".
- docs:
  - forearm_roll.md: §0 block + new motor mount rows, purchased / printed; the §2 station rows; §3 print (the block no
    longer needs support for the plate, the mount prints base down); §4 assembly (new step 6: nuts, mount, screws;
    the motor comes off before the mount); §5; §6.
  - The clearance quoted as "body 1.9 mm above the top" was wrong. Measured: body 3.9 / board 3.4 at nominal, board
    0.9 at the slot's low end. Corrected there and in open_issues.md.
  - robot/, lib/ and assemblies/ CLAUDE.md follow.
- open_issues.md:
  - new: the 3 mm plate is braced only by its root in the base now (check it for flex / creep under the belt's pull;
    thicken pad_t or add gussets outside the motor's footprint);
  - new: the mount's PETG fits (the step, the nut channels, the countersinks);
  - the block's print-orientation row covers the mount's STL too.

Co-Authored-By: Claude Opus 5.5 <noreply@anthropic.com>

File: cad/robot/arm.urdf (robot description, URDF)
Before this commit: robot arm, 10 links, 9 joints
Links:
- link elbow_link: mass 0.74123 -> 0.738734

Commit message: cad: j1_coupler is parametric (lib/yaw_coupler/, LEGACY reproduces the SolidWorks part)
j1_coupler was the last SolidWorks wrapper on the arm's joint chain, and two
docs/open_issues.md rows (the unclamped base_yaw 6806 stack, the empty thrust
groove) wait on its conversion. This commit is the port only: DEFAULT = LEGACY,
no design change. The thrust bearing and the pulley-ready stub follow as their
own commits.

New package lib/yaw_coupler/, built like lib/coupler/ and lib/base/:
- params.py YawCouplerConfig of HubParams (the recess, stub, bore, 4 holes),
  DiscParams (the drafted disc, flats, ears, ring) and YokeParams (the flare,
  the -X cheek, the middle body with its V-grooves, the cradle, pocket,
  channel, notch, the 3 nut pockets). Every number was measured on the
  reference (face census) [REFERENCE].
- layout.py: kernel-free outlines and points.
- body.py build_yaw_coupler(cfg), built in the part frame (revolves about Y,
  prisms along X).
parts/base/j1_coupler.py: CONVERTED = True, REFERENCE_BUILD = LEGACY.

build_yaw_coupler(LEGACY) vs reference/solidworks/j1_coupler.step:
volume 200013.589 vs 199961.363 mm^3 (+52.2, +0.026 %; 91.2 extra and 38.9
missing), bbox equal to 1e-4 mm, 80 faces vs 115. The differences are three
declared simplifications:
- the yoke's +/-Z outer faces are vertical and symmetric (the reference leans
  0.44 / 0.36 deg): +90 mm^3;
- one flare cone over the whole yoke (the reference's last 3 mm toward +X
  carry the x 28.5 section on): -48 mm^3;
- no 0.2 mm channel bevels: < 0.5 mm^3.

The yoke is the drive's housing's shape, and tests/yaw_coupler/ locks that
against lib/cycloidal/params.py: cradle = the housing bore, V-groove ends on
its od, the groove and cheek points on the 45 deg pillar's sides (0.01), the
channel walls the bottom pillar's sides 0.2 out, the nut pockets on its
bolt circle. Plus named feature probes of LEGACY's disc, yoke and hub.

A finding, added to docs/open_issues.md as a fit problem: the drive is not
fastened to j1_coupler. Its M4 x 55 housing bolts end in their own nuts at
x -28.0 in the coupler frame, 0.5 short of the cheek (x -28.5), so the
cheek's 3 nut pockets are empty. The drive's axis also sits 0.21 mm off the
cradle's (placements.json: 0.103 up, 0.186 in z), past the 0.2 a side an M4
has in the cheek's 4.4 holes.

shoulder_link (URDF / SDF inertial, mesh re-exported): mass 1.664416 ->
1.664482 kg, com (-0.000816, 0.015306, -0.011234) -> (-0.000815, 0.015304,
-0.011235), ixx 3.846276e-03 -> 3.846424e-03, ixy 1.395527e-05 ->
1.395277e-05, ixz 1.395735e-05 -> 1.398866e-05, iyy 3.574227e-03 ->
3.574559e-03, iyz -2.839446e-04 -> -2.840645e-04, izz 2.881448e-03 ->
2.881732e-03. The arm / link totals locks hold. Hash gate: only
j1_coupler.step and arm.step changed. Suite: 781 passed, 14 skipped.

tests/test_layering.py LEAF_PACKAGES += yaw_coupler; parts/, lib/ and tests/
CLAUDE.md name the package.

Co-Authored-By: Claude Opus 5.5 <noreply@anthropic.com>

File: cad/robot/arm.urdf (robot description, URDF)
Before this commit: robot arm, 10 links, 9 joints
Links:
- link shoulder_link: mass 1.664416 -> 1.664482

Commit message: cad: the roll motor mount - plain base in a pocket, one 4 mm thickness, nuts pressed in from the bore
This revises forearm_roll_motor_mount (the previous commit) after a review in the viewer:
- The base should not carry the block's rounded edges.
- The plate was too thin, and should match the base.
- The nuts should sit on the other side of the block's top wall, not in slide-in channels from the rear face.

A bolt cannot go straight through the block under the mount: its middle is the core bore the roll shaft turns in. The
nuts therefore press into hex pockets on the inside of the top wall, the way the elbow pulley's nuts sit, and go in
from the bore before the shaft.

- The base is a plain rectangle as wide as the plate (plate_w 46), mount_base_t 4. It sits in a pocket in the block's
  flat top, x +/-23.2 (mount_fit 0.2 round it), open at the rear face. The block keeps a 1.8 mm flat rim and its r 8
  edges; the full-width step and the base that copied the block's rounded outline are gone. The base's top stays level
  with the block's, so the motor's clearance is unchanged.
- One thickness: pad_t 3 -> 4 (= mount_base_t). The plate's front face and the 20T stay put, so the motor's mounting
  face moves back 1 mm: z_motor_face 7.05 -> 6.05, the body -33.45..6.05, the MKS board -47.55..-33.45.
- The screws are 4x M3 x 12 countersunk (unchanged), moved from x +/-20, z (-34, 2) to x +/-18, z (-22, 1): over the
  core bore, their pockets 2 mm clear of the bearing seat and the cavity, the heads 1.6 inside the base's sides.
  - Each goes through the base and the top wall (4.6 mm over the nut) into an M3 nut on its seat, y_mount_nut 27.4;
    the tip ends mount_tip_past (1.0, 2 pitches) past it.
  - Each nut sits in a hex pocket, a flat toward +/-X, mount_nut_pocket_af 5.35 on the 5.5 nut: a press (13.531 mm^3
    for the 4), so a nut stays when its screw is out. The pocket runs on down into the core bore.
  - The nut and the tip stay 2.98 / 2.46 mm clear of the bore, so bearing 1 slides past and the shaft's core turns
    inside.
  - The rear-face nut channels are gone.
- lib/forearm/params.py:
  - mount_bolt_x 18, mount_bolt_z (-22, 1);
  - new mount_tip_past 1.0, mount_nut_pocket_af 5.35;
  - removed mount_nut_roof, mount_channel_add, mount_hole_past.
- lib/forearm/layout.py:
  - new stations y_mount_tip 24, y_mount_nut 27.4;
  - removed y_channel_floor, z_channel_end, y_mount_hole;
  - new mount_nut_pocket_open_y().
- lib/forearm/roll.py: _pocket() replaces _step(); new _y_hex().
- References re-accepted:
  - forearm_roll_block 188631.310 -> 192043.738 mm^3;
  - forearm_roll_motor_mount 16548.628 -> 15378.660 mm^3, bbox x 63.856 -> 46.0;
  - the screws and nuts keep their volumes (416.2 / 183.6), moved to the new points.
- assemblies/forearm_roll_drive.py EXPECTED: volume 419018.261 -> 421260.721, stator 323775.82 -> 326018.28 (leaves
  11 / solids 32, stator 10 / 31, unchanged).
- tests/forearm/test_roll_drive.py:
  - test_stack's mount asserts (one thickness, the rim, the heads inside the base, the tip past the nut, nut + tip
    clear of the bore, the pockets clear of the seat and cavity) replace the channel ones;
  - the probes cover the pocket, the rim, the holes and the hex pockets;
  - the clean-pairs test takes the nuts' designed press (0.9 x .. + 0.5 of 13.53 mm^3).
- robot: elbow_link mass 0.738734 -> 0.741581 kg, COM (-6.251, -27.052, 19.118) -> (-6.629, -27.144, 19.136) mm,
  ixx / iyy / izz 1.339249e-3 / 7.902239e-4 / 1.295333e-3 -> 1.342488e-3 / 7.963497e-4 / 1.303409e-3 (arm.urdf and
  arm.sdf); meshes/elbow_link.stl re-exported; the arm 5.766 -> 5.769 kg. derive --check and validate --strict are
  clean.
- The hash gate against the previous commit's builds: only forearm_roll_block / _motor_mount / _mount_screws /
  _mount_nuts, forearm_roll_drive and arm changed.
- docs: forearm_roll.md §0 / §2 / §3 / §4 (the mount's nuts go in with the pulley's at step 1, before the shaft) / §6;
  open_issues.md (the plate row, the print row, the mount's fits: the pocket, the nuts' press, the countersinks).

Co-Authored-By: Claude Opus 5.5 <noreply@anthropic.com>

File: cad/robot/arm.urdf (robot description, URDF)
Before this commit: robot arm, 10 links, 9 joints
Links:
- link elbow_link: mass 0.738734 -> 0.741581

Commit message: cad: the roll motor mount's screws M3x12 -> M3x16, the nuts seated as near their pockets' mouths as bearing 1 allows
With M3 x 12 each nut sat 3.6 mm (on the pocket's high side) to 8.8 mm (its low side) up its hex pocket from the core
bore, a deep press from inside the bore. A longer screw lets it sit lower.

- The nut's seat is now set by its clearance to the core bore, not by the screw's tip. mount_nut_clear 1.0 is the
  nut's inner flat outside the bore, since bearing 1 slides past the pockets' mouths before the mount goes on.
  - y_mount_nut 27.4 -> 25.043 (each nut 2.36 lower); the nut's lower face 22.643, 1.2 mm above the pocket mouth's
    high side.
  - The top wall over the nut goes 4.6 -> 6.96 mm.
- Screws M3 x 12 -> M3 x 16 countersunk (mount_screw_len). The tip y 24 -> 20 is 2.64 past the
  nut. It comes 0.37 mm out into the core bore's clearance round the shaft's core, still 3.93 off the core. Bearing 1
  would catch on it, so the screws come out before the shaft: in docs/forearm_roll.md §4 and the parts' notes.
- lib/forearm/params.py: mount_tip_past replaced by mount_nut_clear. layout.py: y_mount_nut from the clearance.
- The block's hex pockets end 2.36 lower. forearm_roll_block re-accepted, 192043.738 -> 192191.8 mm^3;
  forearm_roll_mount_screws re-accepted, 416.2 -> 529.3 mm^3 (bbox z 12 -> 16). ROLL_MOUNT_SCREWS_MASS_G 3.3 -> 4.2 g.
  The nuts' part is unchanged: the module row places them.
- assemblies/forearm_roll_drive.py EXPECTED: volume 421260.721 -> 421521.889, stator 326018.28 -> 326279.448.
  block x nuts is still the designed press, 13.531 mm^3.
- tests: test_stack holds the nut at mount_nut_clear off the bore (>= 1), the tip >= 2 pitches past it and >= 2 mm
  off the shaft's core. test_bom holds the "M3 x 16" order.
- robot: elbow_link mass 0.741581 -> 0.742657 kg, COM (-6.629, -27.144, 19.136) -> (-6.634, -27.133, 19.145) mm,
  ixx / iyy / izz 1.342488e-3 / 7.963497e-4 / 1.303409e-3 -> 1.342914e-3 / 7.968956e-4 / 1.303608e-3 (arm.urdf and
  arm.sdf); meshes/elbow_link.stl re-exported; the arm 5.769 -> 5.770 kg. derive --check and validate --strict are
  clean.
- The hash gate against the previous commit's builds: only forearm_roll_block, forearm_roll_mount_screws,
  forearm_roll_drive and arm changed.

Co-Authored-By: Claude Opus 5.5 <noreply@anthropic.com>

File: cad/robot/arm.urdf (robot description, URDF)
Before this commit: robot arm, 10 links, 9 joints
Links:
- link elbow_link: mass 0.741581 -> 0.742657

Commit message: cad: j1_coupler's stub runs to the lip, drilled for a base_yaw 90T
The last step of the j1_coupler conversion. Its hub now takes the base_yaw
90T the way j3_coupler's takes the wrist's, so the pulley, when it is
modelled, bolts on with no change to the coupler. The SolidWorks hub could
not take it:
- the stub (Ø29.8) stopped 0.2 into the lip, 1.1 short of the lip's lower
  face, where the pulley's hub end meets it;
- its 4x Ø3.3 holes (r 10.6) are not the 90T's pattern;
- its Ø15 bore left 1.45 of wall to them.

lib/yaw_coupler DEFAULT [DESIGN] (HubParams gains nut_af / nut_depth;
LEGACY has none):
- stub Ø29.8 -> BEARING_6806_BORE Ø30 (line-to-line in the bearings, like
  every stub - test_params_invariants now includes it);
- the stub's end y -8.2 -> -9.307252, the lip's lower face (base lip_y[0] -
  ring_top_y);
- bore Ø15 -> Ø12.5 (j3_coupler's, the 90T's);
- holes 4x Ø3.3 at r 10.600708 -> 4x M4_CLEAR Ø4.4 at GT2_PULLEY_90T_BOLT_R
  11.0, still on the diagonals, so the 90T mounts turned 45 deg on its own
  pattern and the nuts clear the pocket's X +/-15.2 walls;
- nut pockets j3_coupler's 6.85 AF, M4_NUT.h 3.2 deep, flush in the
  pocket's floor (y 8.0), a corner along Z;
- wall between bore and holes 1.45 -> 2.55.

Volume 192796.5 -> 193586.0 mm^3 (+789.5 = stub Ø30 +91.9, stub to the lip
+549.1, bore +934.5, holes -460.5, nut pockets -325.5). bbox min y -8.2 ->
-9.3073, the rest unchanged.

Tests (tests/yaw_coupler/):
- test_default_hub_takes_the_base_yaw_90t (the hub's numbers; nuts clear of
  the pocket's walls and the bore; 3.2 of material under them);
- test_default_changes_only_the_hub_and_underside (probes of the stub's end
  and Ø30, the bore, each hole end to end, each nut pocket's flats, corner
  and depth).

shoulder_link (URDF / SDF, mesh re-exported): mass 1.678316 -> 1.679319 kg,
com (-0.000809, 0.015178, -0.011875) -> (-0.000808, 0.015169, -0.011927),
ixx 3.944536e-03 -> 3.952462e-03, ixy 1.417583e-05 -> 1.418813e-05, ixz
1.485715e-05 -> 1.492821e-05, iyy 3.668667e-03 -> 3.676363e-03, iyz
-3.003661e-04 -> -3.017000e-04, izz 2.908568e-03 -> 2.908848e-03. Total mass
5.846 kg.

docs/open_issues.md:
- the base_yaw stack row: the stub is ready; the base_yaw 90T is what holds
  the coupler down on the thrust bearing and loads the lower 6806 (a shim
  for the stack's height on assembly);
- the 6806 PETG row drops j1_coupler's Ø29.8;
- the "Not modelled" base_yaw drive: a third 90T bolted to the stub (M4 x 40
  from its outer face ends 1.3 past the nuts), a 20T, and a belt that
  BASE_MOTOR_PATTERN_CENTRE (78.97) wants at 274.2 mm, not a stock length
  (264 -> 73.63, 280 -> 81.97).

Hash gate: only j1_coupler.step and arm.step changed. Suite: 795 passed,
16 skipped.

Co-Authored-By: Claude Opus 5.5 <noreply@anthropic.com>

File: cad/robot/arm.urdf (robot description, URDF)
Before this commit: robot arm, 10 links, 9 joints
Links:
- link shoulder_link: mass 1.678316 -> 1.679319

Commit message: cad: the base_yaw thrust bearing (AXK 6590 + 2x AS 6590) seats j1_coupler
j1_coupler turned on the base's top face: its SolidWorks rim sat flush on it,
and the base's annular groove round the seat ring (Ø65.1 / Ø90.2, 3.0 deep)
was empty (docs/open_issues.md). The user chose a thrust bearing in the
groove to set the coupler's height. The alternative, the clamped 6806 pair
(j3_coupler's shoulder), would over-constrain the joint with a thrust
bearing under it. So the coupler gets no inner-ring shoulder: the upper 6806
locates it radially only.

The bearing (lib/bearings.py THRUST_*, re-exported by lib/params.py):
- INA AXK 6590 needle cage 65 x 90 x 3 between two AS 6590 washers
  65 x 90 x 1; THRUST_STACK = 5.0.
- The washers are the needles' raceways (PETG is none).
- Masses 40 g and 23 g [DATASHEET] (distributor listings; weigh one).

Parts, native COTS (lib/reference.py NATIVE_COTS; reference/native/ written
by import_native.py): parts/base/bearing_axk6590.py (envelope 9130.3 mm^3)
and parts/base/washer_as6590.py (3043.4 mm^3).

Mounts (lib/mounts.py THRUST_MOUNTS, placements.json via mount_placements.py):
- washer_as6590#1 on the groove floor (base y -8.492748) and
  bearing_axk6590#1 on it (-7.492748), both base_link;
- washer_as6590#2 under j1_coupler's seat (coupler y 0.6), shoulder_link.
Also in assemblies/arm.py OCCURRENCES + GROUPS, robot/frames.py LINKS and
lib/mounts.py AXES.

lib/yaw_coupler DEFAULT [DESIGN]:
- the recess's ceiling (the seat) at y 0.5 -> 1.6 = the groove floor (-3.4
  in this frame) + THRUST_STACK;
- the recess Ø90.05 -> Ø90.4 (THRUST_CLEAR 0.2 round the stack, the rim now
  wholly outside the Ø90.2 groove);
- the underside / rim y -0.4 -> 0.1 (RIM_CLEAR 0.5 over the base's top face).
The part keeps its placement. Volume 200013.6 -> 192796.5 mm^3 (-7217.1),
bbox unchanged.

lib/base DEFAULT [DESIGN]: the seat ring Ø65.1 -> Ø64.8 (RING_CLEAR 0.1 a
side inside the stack's Ø65 bore; the SolidWorks ring was over it). Volume
286499.6 -> 286395.6 mm^3 (-104.0). Its docstrings no longer say the coupler
bears on the ring.

Tests:
- tests/test_mounts.py test_thrust_bearing_carries_j1_coupler: the four
  contacts face to face, each the washers' whole annulus; base-cage 0.1
  (RING_CLEAR), coupler-cage 0.2 (THRUST_CLEAR), base-coupler 0.5
  (RIM_CLEAR); no overlap with the 6806 pair.
- tests/yaw_coupler DEFAULT tests; tests/base ring test.

Locks:
- arm leaves 76 -> 79, solids 227 -> 230, bought / printed leaves
  42 / 34 -> 45 / 34;
- BOM bought (25 kinds, 42 pieces) -> (27, 45);
- placements leaf_occurrences 49 -> 52, solids 121 -> 124, the mounted list.

Inertials (URDF / SDF, meshes re-exported):
- base_link: mass 0.850854 -> 0.913722 kg, com (-0.050363, 0.000023,
  0.044115) -> (-0.046897, 0.000021, 0.047559), ixx 1.231537e-03 ->
  1.426810e-03, ixy 2.563886e-06 -> 2.631768e-06, ixz -5.513392e-04 ->
  -6.989411e-04, iyy 2.465551e-03 -> 2.809310e-03, iyz 1.147680e-06 ->
  1.215159e-06, izz 2.423921e-03 -> 2.669327e-03.
- shoulder_link: mass 1.664482 -> 1.678316 kg, com (-0.000815, 0.015304,
  -0.011235) -> (-0.000809, 0.015178, -0.011875), ixx 3.846424e-03 ->
  3.944536e-03, ixy 1.395277e-05 -> 1.417583e-05, ixz 1.398866e-05 ->
  1.485715e-05, iyy 3.574559e-03 -> 3.668667e-03, iyz -2.840645e-04 ->
  -3.003661e-04, izz 2.881732e-03 -> 2.908568e-03.
- The URDF ledger names the thrust parts' links. Total mass 5.845 kg.

docs/open_issues.md:
- the "thrust bearing not modelled" row is closed (deleted);
- the base_yaw stack row now reads: the joint is not held down (the pulley
  under the lower 6806 would), the stub 1.1 short of the lip's lower face;
- a row for the thrust fits in PETG and its masses.
Also assemblies/, lib/, robot/ and tests/ CLAUDE.md.

Hash gate: only base.step, j1_coupler.step and arm.step changed (plus the
two new parts' STEPs). Suite before the rebase onto 0863cd2 (the roll motor
mount, whose counts the locks above add to): 794 passed, 16 skipped (the new parts'
vendor-frame checks).

Co-Authored-By: Claude Opus 5.5 <noreply@anthropic.com>

File: cad/robot/arm.urdf (robot description, URDF)
Before this commit: robot arm, 10 links, 9 joints
Links:
- link base_link: mass 0.850854 -> 0.913722
- link shoulder_link: mass 1.664482 -> 1.678316
