Commit message: cad: robot description - the cycloidal drive rides in link1 (inertials re-derived)
- robot/frames.py: LINKS['link1'] gains the designed-module key cycloidal_drive#1 (housing in the
  j1_coupler yoke, hub on j1_link: physically a shoulder-pitch joint, NOT modelled as a joint
  yet - [ASSUMPTION]); the j1 note no longer calls the drive its actuator.
- robot/_links.py, tools/robot_frames.py: links and inertials iterate world_rows(), so a designed
  module expands into its 18 parts (COTS masses / PETG volumes).
- robot/meshes/link1.stl re-exported (61 solids, 2.79 MB); arm.urdf + arm.sdf link1 inertial
  re-derived (0.895 -> 2.416 kg); URDF ledger rewritten (drive assumption, motor mapping
  unconfirmed); --check, strict validators and tests/test_robot.py green.

File: cad/robot/arm.urdf (robot description, URDF)
Before this commit: robot arm, 8 links, 7 joints
Links:
- link link1: mass 0.894546 -> 2.415794

Commit message: cad: model the cycloidal drive as the shoulder_pitch joint; descriptive link/joint names
The holder (j1_coupler) yaws on the base and carries the drive's housing + motor; the
drive's output hub is bolted to j1_link - so the drive is a joint, not a rigid part of
link1. robot/frames.py splits the old link1 into shoulder_link (holder + drive stator)
and upper_arm_link (drive rotor + j1_link + j1_cap) with the new shoulder_pitch joint
about the drive axis, and renames the chain base_yaw / shoulder_pitch / elbow_pitch /
wrist_pitch (links shoulder_link / upper_arm_link / forearm_link / wrist_pitch_link).

- assemblies/cycloidal_drive.py BODIES (stator / rotor) + per-body totals lock;
  _occurrences.split_key / world_rows expand one rigid body via "<key>:<body>"
- lib/params.py: BASE_YAW / SHOULDER_PITCH / ELBOW_PITCH / WRIST_PITCH limits
- robot/arm.urdf: new link + joint, re-derived inertials/origins, ledger rewritten;
  arm.sdf regenerated; arm.srdf home state + adjacent pairs; link models and meshes
  renamed, shoulder_link.stl + upper_arm_link.stl exported
- assemblies/arm.py GROUPS relabelled (drive kept whole under shoulder_link)
- tests: body partition/totals, world_rows expansion, joint on the drive axis, FK
  per-chain tolerance 5 um; ./cadtool pytest 457 passed / 9 skipped, --check and
  validate --strict green
- docs: cad/README.md, cad/CLAUDE.md, docs/cycloidal_drive.md, CHANGELOG.md

Motor-to-joint mapping (src/config.py J1..J3) stays unconfirmed; src/config.py untouched.

File: cad/robot/arm.urdf (robot description, URDF)
Before this commit: robot arm, 8 links, 7 joints
Links:
- removed link link1
- removed link link2
- removed link link3
- added link forearm_link, mass 0.684302; collision mesh filename=meshes/forearm_link.stl scale=0.001 0.001 0.001; visual mesh filename=meshes/forearm_link.stl scale=0.001 0.001 0.001
- added link shoulder_link, mass 1.629416; collision mesh filename=meshes/shoulder_link.stl scale=0.001 0.001 0.001; visual mesh filename=meshes/shoulder_link.stl scale=0.001 0.001 0.001
- added link upper_arm_link, mass 0.786378; collision mesh filename=meshes/upper_arm_link.stl scale=0.001 0.001 0.001; visual mesh filename=meshes/upper_arm_link.stl scale=0.001 0.001 0.001
- added link wrist_pitch_link, mass 0.440548; collision mesh filename=meshes/wrist_pitch_link.stl scale=0.001 0.001 0.001; visual mesh filename=meshes/wrist_pitch_link.stl scale=0.001 0.001 0.001
Joints:
- removed joint j1
- removed joint j2
- removed joint j3
- added joint base_yaw: type revolute, parent base_link, child shoulder_link, origin xyz=0 0 0.18591 rpy=0 0 0, axis 0 0 1, limit lower=-3.054326 upper=3.054326 effort=5 velocity=1
- added joint elbow_pitch: type revolute, parent upper_arm_link, child forearm_link, origin xyz=0.210003 0 0.009998 rpy=0 0 0.010227, axis 0 0 1, limit lower=-2.094395 upper=2.094395 effort=5 velocity=1
- added joint shoulder_pitch: type revolute, parent shoulder_link, child upper_arm_link, origin xyz=0.002441 -0.034915 0 rpy=-1.570796 -0.830504 0.064484, axis 0 0 1, limit lower=-2.094395 upper=2.094395 effort=5 velocity=1
- added joint wrist_pitch: type revolute, parent forearm_link, child wrist_pitch_link, origin xyz=0.21 0 0.041998 rpy=0 0 0.299075, axis 0 0 1, limit lower=-2.094395 upper=2.094395 effort=5 velocity=1
- joint wrist_roll: parent link3 -> wrist_pitch_link

Commit message: cad: the belt joints' NEMA 17 x 40 + MKS SERVO42D kits on their pads, the drive's board on its motor
The SolidWorks arm cut NEMA 17 pads into base / j1_link / j2_link but never placed the
base_yaw / elbow_pitch / wrist_pitch motors. From the user's nema17x40_with_mks export
(kept outside the repo next to the monolith, lib.reference.MKS_EXPORT_NAME):

- tools/reference/split_mks_motor.py splits the kit by geometry into vendor/nema17_40mm.step
  (body + D-shaft, re-framed like the drive motor, shaft trimmed 23 -> 22) and
  vendor/mks_servo42d.step (board + cover + standoffs + M3x30, z=0 at the motor's rear face);
  import_solidworks.py mirrors them into reference/solidworks/ (rel=None, the pancake pattern).
- parts/joints/nema17_40mm.py and mks_servo42d.py (COTS; envelopes at the vendor bboxes);
  the drive motor's envelope builder moved to lib/cycloidal/motor.py (nema17_48mm.step is
  byte-identical) and the 40 mm envelope reuses it with other MotorParams.
- lib/mounts.py declares the six mounted occurrences (frames as data in the host's frame,
  spins and the wrist slide position [ESTIMATE]); tools/reference/mount_placements.py
  materialises them into placements.json as ordinary part records (parent None, rel == world,
  a mount block; motor +Z checked against the joint axis) - extract_placements.py appends them,
  the merge mode needs no monolith. lib/placements: to_record(), keys(mounted=), importable
  without the JSON.
- assemblies/arm.py OCCURRENCES / GROUPS, robot/frames.py LINKS + joint notes; the drive gains
  the board row (stack_positions z_mks_board = -48), EXPECTED 19 / 71.
- URDF / SDF inertials of base, shoulder, upper_arm and forearm re-derived, the four link
  meshes re-exported, ledger updated. Tests: counts bumped (59 leaves / 166 solids, 17 bought /
  25 pieces, 40 + 19 / 95 + 71), tests/test_mounts.py (axis on the joint, face on the pad,
  zero interference, base stack above the base bottom), the drive's bbox lock without the board.
  ./cadtool pytest: 630 passed, 9 skipped.

File: cad/robot/arm.urdf (robot description, URDF)
Before this commit: robot arm, 9 links, 8 joints
Links:
- link base_link: mass 0.363435 -> 0.678435
- link forearm_link: mass 0.684302 -> 0.999302
- link shoulder_link: mass 1.629416 -> 1.664416
- link upper_arm_link: mass 0.786378 -> 1.101378

Commit message: cad: the base_yaw motor is the 48 mm one
lib/mounts.py places nema17_48mm#1 (the drive's motor, parts/cycloidal) on the base's pad instead of a
40 mm motor; the elbow and wrist keep nema17_40mm#2..3. MOTORS / board_frame(body_length) replace the
single MOTOR / BOARD_FRAME. Consequence, locked rather than hidden: the 48 mm motor + board (62.1) reach
BASE_MOTOR_STACK_PROUD = 6.1 mm below the base's bottom face (56 mm of depth under the plate) -
lib/params.py, test_params_invariants, tests/test_mounts.py. Mounted records regenerated (100 solids),
arm 177 / no-caps 174 solids, base_link inertials + mesh re-derived (total 5.288 kg), purchase notes
2 x 40 mm + 2 x 48 mm kits. ./cadtool pytest: 632 passed, 8 skipped.

File: cad/robot/arm.urdf (robot description, URDF)
Before this commit: robot arm, 9 links, 8 joints
Links:
- link base_link: mass 0.678435 -> 0.798435

Commit message: cad: the forearm's roll end - the flange wall replaces the elbow disc, the wrist motor moves to where a 264-2GT belt puts it
lib/forearm/params.py RollEndParams (roll axis at y 0, z 25 = the wrist centre's N-station; the wall at x -96..-88,
z -10..60; the rotor flange's Ø60.3 x 2 locating recess, 4x M3 on Ø46, the Ø28 cable bore; plug clearance 10;
wrist belt 264-2GT) and DEFAULT = replace(LEGACY, roll=True, motor_x = wrist_x + centre_distance(264) = -136.37,
slide (-141.5, -130), central slot 22.3 wide (the Ø22 pilot passes - the open-issues row closes), both slots
shortened to end >= 4 mm before the wall; the lid's window follows the motor and its pocket arc widens r55 -> r50
so the body's wrist face clears it). link.py: roll_wall() (x_cylinder for the roll-axis features) replaces the
elbow disc when roll=True; caps.py: both caps end flush at the wall (they are slated for removal - no further
design work, docs/open_issues.md). lib/params.py re-exports WRIST_BELT_LENGTH, FOREARM_ROLL_AXIS_Z / WALL_X /
WALL_Z / PLUG_CLEARANCE / FLANGE_DIA and adds FOREARM_ROLL_LIMIT_DEG = 170 [ESTIMATE]; the slide lock in
tests/test_params_invariants.py is its derivation now (belt length, plug rule, boss rule); tests/test_mounts.py
budget gone (0 interference); tests/forearm/test_roll_end.py locks the wall, the slots, the motor's clearance.
mount_placements.py moved nema17_40mm#3 / mks_servo42d#3 (placements.json); forearm_link's inertial re-derived
(0.999 -> 0.807 kg) into arm.urdf / arm.sdf, its mesh re-exported.

Verified: fast lane 399 passed; full suite 653 passed + 8 skipped; rebuild after `daemon stop` changed exactly
j2_link, j2_cap_1, j2_cap_2, arm, arm_no_caps, forearm_link; derive.py --check clean after the paste; validate x3
OK; snapshots arm.png / arm_no_caps.png looked at (the forearm now starts at the wall; the elbow pulley + coupler
wait for M3's block).

File: cad/robot/arm.urdf (robot description, URDF)
Before this commit: robot arm, 9 links, 8 joints
Links:
- link forearm_link: mass 0.999302 -> 0.807053

Commit message: cad: the forearm roll drive - the 6th joint: elbow block, hollow roll shaft with its 90T ring, 6808 bearings, the roll motor; elbow_link + forearm_roll in the robot description
assemblies/forearm_roll_drive.py: a code-driven module (rows from lib/forearm stack_positions, BODIES stator /
rotor, EXPECTED) placed by lib/mounts.py MODULE_MOUNTS on j2_link's roll axis (module +Z toward the wrist, +X the
motor side). Stator: the elbow block (the SolidWorks disc's j3_coupler interface + a Ø60 tube: closed end with the
cable window, the lip, one Ø52.15 seat for both bearings, retainer lugs, the motor pad tower with radial tension
slots), 2x 6808-2RS (envelope-only NATIVE_COTS bearing_6808), the bolted retainer with the hard-stop post, the 40 mm
kit motor + MKS board, the 20T. Rotor: the hollow roll shaft - Ø40.3 journals (+0.3 in the inner races), Ø44
shoulders, the integral flanged 90T GT2 ring (lib/forearm/pulley.py gt2_ring: 90 round-bottom grooves), the stop-pin
boss, the Ø60 flange with 4x M3 (nuts captive) and its spigot into the forearm wall's recess, the Ø28 bore. All
numbers lib/forearm/params.py RollDriveParams; the three printed parts are NATIVE (reference/native/*.step accepted
with tools/reference/import_native.py). robot/frames.py: elbow_link (elbow pulley + coupler + the stator) between
upper_arm_link and forearm_link (the rotor + the forearm), Joint forearm_roll along the forearm through the wrist
centre (WRIST_CENTRE = WRIST_PITCH_ORIGIN - 17 N; the three wrist axes concurrent to 5 um); arm.urdf / srdf / sdf
(elbow_link, forearm_roll, wrist_pitch re-derived, inertials, the ledger), meshes elbow_link + forearm_link,
robot/links/elbow_link.py; arm.py: the elbow_link group, MODULES / MODULE_TINTS; tools/bom.py EXTRAS (belts, the
drive's fasteners, the stop pin, the home sensor); docs/open_issues.md rows (a 4th CAN id, the open belt, ...).
Tests: tests/forearm/test_roll_drive.py (the axis through the wrist centre, the module frame, the stack, press fits
on the journals / slip in the seat, every other pair clean, the block's and shaft's features, the module clear of
its neighbours at the capture pose and of the upper arm swung to the elbow's limits), the locks in test_assembly
(67 leaves / 200 solids; no_caps 64 / 197), test_placements (the mounted module record), test_bom (29 printed /
37; 18 bought / 30), test_robot, test_mounts, test_lazy_kernel.

Verified: fast lane 418 passed; full suite green; rebuild after `daemon stop`; derive.py --check clean; validate
x3 OK (10 links, 9 joints, 5.692 kg); snapshots forearm_roll_drive.png, arm.png, arm_no_caps.png, arm_urdf.png and
arm_urdf_roll90.png (--joint-values forearm_roll 90: the forearm, wrist and gripper turn about the forearm, the
block stays with the elbow) looked at.

File: cad/robot/arm.urdf (robot description, URDF)
Before this commit: robot arm, 9 links, 8 joints
Links:
- added link elbow_link, mass 0.628206; collision mesh filename=meshes/elbow_link.stl scale=0.001 0.001 0.001; visual mesh filename=meshes/elbow_link.stl scale=0.001 0.001 0.001
- link forearm_link: mass 0.807053 -> 0.775187
Joints:
- added joint forearm_roll: type revolute, parent elbow_link, child forearm_link, origin xyz=0 0 0.025 rpy=3.141593 -1.570795 0, axis 0 0 1, limit lower=-2.96706 upper=2.96706 effort=5 velocity=1
- joint elbow_pitch: child forearm_link -> elbow_link
- joint wrist_pitch: origin xyz=0.21 0 0.041998 rpy=0 0 0.299075 -> xyz=0.016998 0 0.21 rpy=-1.570799 -1.271722 -1.570793

Commit message: cad: the roll drive laid out like the diagram - motor up in the swing plane, the 90T inside the housing between the bearings, an end cap
lib/forearm/params.py RollDriveParams re-cut: a Ø70 housing (housing_od) round a Ø62 cavity the shaft's flanged ring
runs in (bearing 1's Ø52.15 seat + lip at the elbow end, the belt window in the +Y wall, the cable window in the +X
wall, a FLAT underneath at flat_x -33 - host z -8, 0.5 mm above the upper arm's slab -, two lugs at +X and -Y), the
bolt-on END CAP (forearm_roll_retainer, name kept: bearing 2's seat + lip, the same flat, two ears, the hard-stop post
at -X on its outer face), the motor UP in the swing plane (+Y) at (motor_x 18, motor_y 58.2) - lifted 18 mm along N
so its body clears the elbow disc's top face by 1 mm - with a 240-2GT belt setting the centre distance (60.9; motor_y
is a property), the pad plate / filler / tension slots along the axis -> motor direction. The shaft: a journal each
side of the ring, a Ø38 NECK bearing 2 slides over, the stop lug on it (+X, 10 deg, 1 mm overlap with the post) and
a Ø39.7 END SPIGOT the forearm wall bolts straight onto (4x M3 self-tapped on Ø32, bore Ø24) - no separate flange:
with the ring and a Ø60 flange both integral, bearing 2 could never be mounted (the M3 layout's sequence was
impossible). RollEndParams (the wall side): recess Ø40, bolt circle Ø32, cable bore Ø24 - j2_link follows.
lib/forearm/layout.py stack_positions per the plan's table, cap_bolt_points / pad_slot_angle_deg; roll.py the three
builders; the module rows; lib/params.py FOREARM_ROLL_MOTOR_XY / FOREARM_ROLL_HOUSING_OD; tests/forearm updated
(the stack's new rules: everything beyond journal 2 < the bearing bore, the flat vs the slab, the motor vs the
disc, the spigot's walls; the cap's seat and lip, the belt window, the flat, the stop lugs); tools/bom.py EXTRAS
(240 belt, the end-spigot M3s, the cap's M3s, no stop pin - printed lugs); docs/forearm_roll.md sections 2-5;
docs/open_issues.md rows; part docstrings. The three native references re-accepted; elbow_link + forearm_link
inertials re-derived into arm.urdf / arm.sdf, both meshes re-exported.

Verified: fast lane 418 passed; full suite green; rebuild after `daemon stop` changed exactly the three roll parts,
j2_link, the module, both arms, both links; derive.py --check clean; validate x3 OK (5.723 kg); snapshots
forearm_roll_drive.png, arm.png, arm_no_caps.png, arm_urdf.png, arm_urdf_roll90.png and arm_side.png (--camera 0:0:
the diagram's silhouette - the housing in line with the elbow pulley, the motor on top) looked at.

File: cad/robot/arm.urdf (robot description, URDF)
Before this commit: robot arm, 10 links, 9 joints
Links:
- link elbow_link: mass 0.628206 -> 0.660437
- link forearm_link: mass 0.775187 -> 0.77427

Commit message: cad: the elbow block is the elbow coupler - the roll shaft crosses the elbow axis, the forearm starts at 48, j3_coupler#1 retired

File: cad/robot/arm.urdf (robot description, URDF)
Before this commit: robot arm, 10 links, 9 joints
Links:
- link elbow_link: mass 0.660437 -> 0.716573
- link forearm_link: mass 0.77427 -> 0.920216

Commit message: cad: remove the link caps; j1_link parametric (lib/upper_arm/)
The covers over j1_link / j2_link are gone: j1_cap, j2_cap_1, j2_cap_2 (part modules, lib/forearm/caps.py + the
cap params, reference STEPs, CUSTOM rows, manifest entries) and assemblies/arm_no_caps.py (it would equal arm.py).
Their SolidWorks products are lib/reference.py SKIPPED_PRODUCTS; mount_placements.py's merge mode moves their
records to placements.json `skipped` (poses kept; 37 part records, 97 solids). j2_link DEFAULT drops the cap
sockets (LEGACY keeps them).

j1_link is parametric build123d (lib/upper_arm/: UpperArmConfig, build_link): LEGACY reproduces the SolidWorks
part (354048.80 vs 354048.81 mm3, same bbox; REFERENCE_BUILD); DEFAULT drops the 10 cap sockets, puts the NEMA 17
holes on the 31 mm square about the shoulder axis (closes the open issue) and the hub holes on the cycloidal
drive's arm-mount bolts (the SolidWorks ones were 3.36 deg off). upper_arm_link / forearm_link inertials re-derived
(arm.urdf / arm.sdf), meshes re-exported; tests/upper_arm/ new; docs updated.

File: cad/robot/arm.urdf (robot description, URDF)
Before this commit: robot arm, 10 links, 9 joints
Links:
- link forearm_link: mass 0.920216 -> 0.759089
- link upper_arm_link: mass 1.101378 -> 0.910943

Commit message: cad: the belt joints' 6806-2RS bearing stacks (base_yaw, elbow_pitch, wrist_pitch)
The user fitted two 30 x 42 x 7 bearings (6806-2RS / 61806) at each belt joint; the housings are cut for them
(a bore split by a lip, one bearing each side) but neither the SolidWorks capture nor the model had them, and the
docs called the elbow's "6702-class" (a 6702 is 15 x 21 x 4). Measuring the stacks found three fits that did not
close; all three are fixed here, three others are recorded.
- lib/bearings.py (a leaf, re-exported by lib/params.py): BEARING_6806_BORE / OD / WIDTH 30 / 42 / 7, the
  inner-ring shoulder Ø33, BEARING_6806_MASS_G 26 [ESTIMATE: the 6808's by ring area].
- parts/joints/bearing_6806.py: a native COTS part like bearing_6808 (step.parts has no bearing above a 20 mm
  bore); reference/native/bearing_6806.step accepted (4750.1 mm^3), lib/reference.py NATIVE_COTS, vendor/README.md.
- lib/mounts.py BEARING_MOUNTS: bearing_6806#1..6, a pair per joint standing on the lip of the base's bore,
  j1_link's elbow bore and j2_link's wrist boss (coupler side first), riding with the housing's link; AXES +
  tools/reference/mount_placements.py check a bearing's +Z / a pulley's +Y ON the joint axis.
- The 90T pulleys sat 3.0 mm too close to their couplers: SolidWorks mated each hub flat onto the stub, which puts
  its Ø34.76 ring inside the lower bearing (~363 mm^3). gt2_pulley_90t#1 / #2 are RETIRED (lib/placements.py) and
  re-declared as mounts #3 / #4 hosted on them, PULLEY_SEAT_SHIFT 3.0 out along +Y: the hub's Ø30 x 7 journal fills
  the lower bearing, its ring under that inner ring. At the elbow this also fixes the M4 x 40 pulley bolts: as
  captured their tips ran 2.6 mm past the heat-set inserts' blind holes, now 0.4 short (7.6 of 8 mm engaged).
- Nothing clamped the upper bearings: the couplers' Ø40 journal face stopped 0.7 above them (and would have borne
  on the outer ring) while their Ø62 boss sits 0.5 above the link's recess floor. A Ø33 x 0.7 inner-ring shoulder
  now sits on each: RollDriveParams step_dia / step_x (stub -47..-40.3 -> -47..-41; coupler_steps() builds it;
  forearm_roll_block re-accepted, 209371.3 -> 209475.2 mm^3; forearm_roll_drive EXPECTED 422609.743 -> 422713.651,
  stator 327367.302 -> 327471.21) and j3_coupler's DEFAULT step (y 15.3..16, +103.9 mm^3).
- The base's bore: DEFAULT takes the wrist's seats and lip - Ø42.4 / Ø31.73 / Ø43.4 -> Ø42.2 / Ø37.65 / Ø42.2 (the
  lower seat let its bearing wobble 0.7 a side, the lip ran under the upper inner ring).
- Tables: assemblies/arm.py OCCURRENCES + GROUPS, robot/frames.py LINKS + joint notes, the URDF ledger (it also
  said forearm_link for the elbow 90T: elbow_link since the roll joint).
- Tests: test_mounts.py test_bearings_and_pulleys_sit_on_their_joint_axes, test_bearing_stacks (every contact
  face at 1e-3, zero overlap; the belt-plane test keeps the wrist only - the elbow 90T is driven from j1_link's x 128
  second stage), test_params_invariants 6806 fits, test_bom 6806 row, tests/base and tests/coupler DEFAULT diffs,
  tests/forearm keys and the stub -> shoulder -> journal chain.
Counts: placements parts 37 -> 45, solids 97 -> 105, volume 1849734.223 -> 1927856.167; arm leaves 63 -> 69,
solids 196 -> 202, bought / printed leaves 30 / 33 -> 36 / 33; bom bought (18, 30) -> (19, 36).
Links (kg): base_link 0.798435 -> 0.850854, upper_arm_link 0.910943 -> 0.962943, forearm_link 0.759089 -> 0.811089,
elbow_link 0.716573 -> 0.716705, wrist_pitch_link 0.440548 -> 0.44068 (inertials + meshes re-derived); total
5.574 -> 5.731. The wrist belt plane moves 15.7 -> 18.7 mm along the 22 mm motor shaft (a 20T still reaches it).
open_issues.md: the elbow's "6702-class" row closed; added the base's unclosed stack (j1_coupler has no shoulder,
nothing in the lower bearing until the base_yaw pulley - probably a third "J1" 90T - is modelled), the 6806
mass / ring estimates and the PETG seat fit gauge, the elbow drive's second stage through j1_link's x 128 seats
(its BearingParams no longer "purpose unknown") and GT2_RATIO provisional for elbow_pitch.
Full suite 732 passed, 10 skipped; urdf / srdf / sdf validate; lint clean.

File: cad/robot/arm.urdf (robot description, URDF)
Before this commit: robot arm, 10 links, 9 joints
Links:
- link base_link: mass 0.798435 -> 0.850854
- link elbow_link: mass 0.716573 -> 0.716705
- link forearm_link: mass 0.759089 -> 0.811089
- link upper_arm_link: mass 0.910943 -> 0.962943
- link wrist_pitch_link: mass 0.440548 -> 0.44068
