Commit message: cad: the elbow's and the wrist's stubs reach the re-seated pulleys (bolted flat again)
The 90T pulley and the part above it are one bolted joint (4x M4: into the elbow block's heat-set inserts, through
j3_coupler into nuts in its flange pockets) - which is why SolidWorks had them touching. Re-seating the pulleys
PULLEY_SEAT_SHIFT (3.0) out on their lower bearings left a 3 mm gap: the screws spanned air and the pulley's torque
would have run through the bearings. Each stub now reaches that much further, on through the lip, and ends on the
pulley's hub: a solid face-to-face joint again, the pulley where it is. The stub's 2 mm inside the lip spaces the
two inner rings exactly as the lip spaces the outer rings (the shoulder above, the pulley's ring below - no play),
and the upper bearing's inner ring now sits on the stub over its whole 7 mm (6 before).
- lib/bearings.py: PULLEY_SEAT_SHIFT moves here from lib/params.py (which re-exports it) so the leaf packages use it.
- lib/forearm/params.py RollDriveParams: stub_x (-47, -41) -> (-50, -41), pin_bore_x starts at the stub's end;
  forearm_roll_block re-accepted 209475.2 -> 211045.1 mm^3 (bbox x 80 -> 83); forearm_roll_drive EXPECTED
  422713.651 -> 424283.607, stator 327471.21 -> 329041.166.
- lib/coupler/params.py DEFAULT: stub_y1 22 -> 25 (+1594.0 mm^3). The wrist screws need 46.8 mm (M4 x 50; the
  SolidWorks stack took 43.8 / M4 x 45) - recorded in open_issues.md for the fasteners branch. The elbow's M4 x 40
  do not change (the pulley did not move).
- tests: test_bearing_stacks checks the stub's end and the pulley's hub share a face (a real annulus) and pulley /
  coupler / housing do not overlap; test_roll_drive has one ELBOW_PULLEY_FACE_Z again (-22 - PULLEY_SEAT_SHIFT)
  with the stub's end and the pulley on it; test_j3_coupler: DEFAULT = LEGACY + the shoulder + the longer stub,
  the volume exact.
- Fixed a latent bug in test_forearm_clears_the_elbow_while_rolling: it took the stator's parts from the moved
  module compound, whose children stay in the MODULE frame, so the rolled forearm was never checked against them
  where they are; the longer stub reached into the forearm's region in that wrong frame and exposed it.
  _placed_part() moves each part into j2_link's frame; placed right, the rolled forearm clears the block, the end
  cap, the motor and the board at +/-90 and +/-170 degrees (0 mm^3).
Links (kg): elbow_link 0.716705 -> 0.718699, wrist_pitch_link 0.44068 -> 0.442705 (inertials + meshes re-derived);
total 5.731 -> 5.735. Docs: forearm_roll.md (stub -50..-41, the assembly step), the base's open-issue row (the
same fix when j1_coupler and its pulley are drawn), the j3_coupler docstring.
Full suite 733 passed, 10 skipped; urdf / srdf / sdf validate; lint clean.

File: cad/robot/arm.urdf (robot description, URDF)
Before this commit: robot arm, 10 links, 9 joints
Links:
- link elbow_link: mass 0.716705 -> 0.718699
- link wrist_pitch_link: mass 0.44068 -> 0.442705

Commit message: cad: the elbow 90T bolts into captive nuts in the elbow block (heat-set inserts retired)
Every other 90T in the arm is held by a bolt and a nut: at the wrist 4x M4 run from the pulley's outer face through
j3_coupler into hex nut pockets in its flange's underside, the face wrist_link then covers. The elbow was the
exception: the roll drive's block took j3_coupler#1's place, and its M4s ended in 8 mm heat-set inserts. The block has
no free face for a pocket: the bolts run up the elbow axis straight at the roll shaft's core bore, only 6.7 mm of
floor above the underside. So the pocket opens onto the face the next part covers, as at the wrist - here the core
bore, which the roll shaft fills: each nut drops in from inside the bore (block underside down) before the shaft goes
in, which the assembly order already allows (the pulley is bolted at step 2, the shaft goes in at step 4).
- lib/forearm/params.py RollDriveParams: insert_dia / insert_x removed; nut_af 6.85 (j3_coupler's pocket: an ISO 4032
  M4, s 7, presses in), nut_t 3.2, nut_seat_x -36 (in the Ø62 boss), nut_channel_past 1, pulley_hub_len 21.4 (the
  90T's plain Ø3.9 holes run its whole length: the heads sit on its outer face), pulley_screw_len 40. The M4 x 40 stays:
  its tip (-31.4) ends 1.4 mm (2 pitches) past its nut (-36..-32.8); nut top 6.5 mm and tip 5.1 mm under the core bore
  (bearing 1 slides past the channel mouths).
- Each channel is a hex prism with a flat toward the elbow axis, from the seat up into the bore (lib/forearm/layout.py
  nut_channel_end); the Ø4.4 clearance runs from the stub's end to the seat (-50..-36).
- pulley_bolt_deg 45: the pattern turns off the axes, the elbow 90T with it (lib/mounts.py gt2_pulley_90t#3 frame
  (0, 45, 0); its placements.json record 93.438897 / 42.891416 / 174.954347 -> 89.871228 / -1.993488 / 176.303304).
  On the axes the +z channel would reach z 14.4, 1.6 mm from the ring cavity (cavity_z0 16, pinned by the ring's
  flange at 16.8); at 45 deg the channels reach z 11.6: 4.4 mm (the inserts left 2.2). The pulley's inertia does not
  change (4-fold symmetry). The wrist's #4 keeps its capture spin.
- pin_bore_x (-50, -29) -> (-50, -37): it ends 1 mm under the nut seats (beside the channels its wall would be 1.3).
- forearm_roll_block re-accepted 211045.1 -> 210853.1 mm^3 (bbox unchanged); forearm_roll_drive EXPECTED
  424283.607 -> 424091.544, stator 329041.166 -> 328849.103.
- tools/bom.py EXTRAS: the M4 heat-set insert row -> M4 hex nut (ISO 4032) x 4, captive in the block's hex channels;
  the M4 x 40 row now reads into those nuts.
- tests: test_stack's wall rules (seat in the boss, tip 2 pitches past the nut, nut and tip >= 2 mm under the core
  bore, each channel >= 2 mm from the cavity, the pin bore ending under the seats) and the block probes (the hex's flat
  and corner, the seat beside the clearance hole, the mouth in the bore); test_mounts: the elbow 90T's 45 deg spin and
  the new slow test_the_elbow_pulley_holes_line_up_with_the_block_bolts (each bolt axis through the pulley's hole and
  the stub's clearance, the hub solid 3 mm beside it).
Links (kg): elbow_link 0.718699 -> 0.718455 (inertial + mesh re-derived); total 5.734668 -> 5.734424.
Docs: forearm_roll.md (§0, the underside / core bore / cavity rows, the torque path, §4 steps 1-2 - a screw taken
right out once the shaft is in can drop its nut into the gap round the core, §6), the block's and the 90T's
docstrings, assemblies/CLAUDE.md; open_issues.md: the heat-set insert creep row closed, the nut channels' 6.85 AF
press added to the PETG fit-gauge row.

File: cad/robot/arm.urdf (robot description, URDF)
Before this commit: robot arm, 10 links, 9 joints
Links:
- link elbow_link: mass 0.718699 -> 0.718455

Commit message: cad: j1_link's elbow relief - the elbow block clears the upper arm by 2.0 mm (was 0.5)
The roll drive's block turns with the elbow over j1_link. Its flat underside and its end cap's, swept out to r 57.6
about the elbow axis, rode 0.5 mm above j1_link's top face (the slab's 1.5 mm lip), and its Ø62 boss 0.5 mm above
the Ø80 recess floor, at every elbow angle. Those are printed PETG faces, and the forearm's moment tilts the block on
a 16 mm bearing base: 0.5 mm is only 0.5 deg of tilt at r 58, so they would rub. The tests missed it because every
check was overlap volume < 1 mm^3, which a 0.5 mm gap, or contact, passes.
- lib/upper_arm/params.py ElbowParams: new relief_r (0 = none: LEGACY, the SolidWorks part, is unchanged). DEFAULT
  relief_r 60 cuts the lip back to its root (y1) within r 60 of the elbow axis, and recess_y -4.5 -> -5.5.
  lib/upper_arm/link.py cuts the relief after the lip. The upper 6806 seat stays 7.5 deep.
- Gaps (closest_points, at elbow 0 / +/-45 / +/-90): block and cap underside 0.5 -> 2.0 mm, boss 0.5 -> 1.5. The
  block's nearest point is now its journal's edge by the bore's rim: 1.02 mm, a radial gap the bearings set.
- j1_link DEFAULT volume 354456.7 -> 346810.0 mm^3 (-4005.6 relief, -3641.1 recess ring), 450.16 -> 440.45 g.
Links (kg): upper_arm_link 0.962943 -> 0.953232 (inertial + mesh re-derived); total 5.783919 -> 5.774208.
- tests: test_roll_drive has the relieved face (host -10), UPPER_ARM_RELIEF_R and FACE_GAP 1.5. test_stack holds
  the underside and the boss FACE_GAP clear and the block's and cap's corners (r 57.6) 2 mm inside the relief.
  test_module_clears_the_folded_upper_arm (now also at 0 deg) asserts the minimum gaps: the cap's is the designed
  2.0, the block's the journal's 1.02. test_j1_link: DEFAULT = LEGACY + the relief + the deeper recess, with the
  volume exact and probes on both sides of the relief's edge.
Docs: forearm_roll.md (§0 clearances row, §2 block row); the block comments in lib/params.py and
lib/forearm/params.py; j1_link's params docstring; lib/CLAUDE.md.

File: cad/robot/arm.urdf (robot description, URDF)
Before this commit: robot arm, 10 links, 9 joints
Links:
- link upper_arm_link: mass 0.962943 -> 0.953232

Commit message: cad: elbow_pitch limited to +/-90 deg (the forearm wall hit the upper arm past +/-93)
The forearm roll put j2_link's wall 48 mm from the elbow axis, 3 mm outside j1_link's r 45 end, and its lower edge
(host z -10) sits 1.5 mm below j1_link's top face (-8.5). Folded past 90 deg, the wall swings over the upper arm's
side. closest_points goes 3.04 mm (90 deg) -> 1.14 / 0.27 mm (+93 / -93) -> contact at +/-94. The 120 deg estimate
drove the wall into j1_link: 520 / 534 mm^3 of overlap at +/-120 with the roll at 0, and 1.0-4.0 cm^3 rolled. No test
folded j2_link against j1_link, and the roll sweep ran only with the elbow straight. At +/-90 the wall keeps
>= 2.59 mm at every roll (0, +/-45, +/-90, +/-135, +/-170). Other forearm_link parts never touch the upper arm.
- lib/params.py: ELBOW_PITCH_LIMIT_DEG 120 -> 90, re-tagged [ESTIMATE] -> [DESIGN] (the wall sets it).
- robot/arm.urdf / arm.sdf: elbow_pitch limit +/-2.094395 -> +/-1.570796 (from the derive.py drafts; --check clean).
  The SRDF group states hold elbow 0. software/ has no joint limits to follow.
- tests: test_forearm_clears_the_upper_arm_at_the_elbow_limits (slow): j2_link rolled to
  0 / +/-90 / +/-FOREARM_ROLL_LIMIT_DEG against j1_link folded to +/-ELBOW_PITCH_LIMIT_DEG, >= 2.0 mm apart.
  test_module_clears_the_folded_upper_arm now folds to +/-90.
Docs: forearm_roll.md §0 clearances row (the fold limit and why).

File: cad/robot/arm.urdf (robot description, URDF)
Before this commit: robot arm, 10 links, 9 joints
Joints:
- joint elbow_pitch: limit lower=-2.094395 upper=2.094395 effort=5 velocity=1 -> lower=-1.570796 upper=1.570796 effort=5 velocity=1

Commit message: cad: the elbow and wrist 90T bolts and nuts are modelled (the 90T's holes opened to M4 clearance)
Each belt joint's 90T is clamped flat onto the part above it by 4x M4 screws and nuts, but none of that hardware was
in the model: the elbow's were two tools/bom.py EXTRAS rows, the wrist's only an open_issues.md "Not modelled" row
(46.8 mm of screw needed, so M4 x 50). They are now four purchased pattern parts, mounted like the bearings (Recipe B),
riding with elbow_link / wrist_pitch_link. The SolidWorks 90T's Ø3.9 holes took no M4 shank (53.1 mm^3 of overlap per
joint), so the pulley's model opens them to M4 clearance and the printed pulley takes the screws as is.
- lib/fasteners.py (new leaf, re-exported by lib/params.py, tests/test_layering.py LEAF_MODULES): M4_SHCS (ISO 4762:
  d 4, head 7 x 4, socket 3 x 2), M4_NUT (ISO 4032: 7 AF x 3.2, the Ø4 bore), M4_PITCH, shcs() / hex_nut() (plain
  geometry, no thread) and their volumes; M3/M4/M5_CLEAR move here from lib/params.py, M4_CLEAR 4.5 -> 4.4 (unused
  before; now the 90T's holes and RollDriveParams.pulley_bolt_dia, whose value is unchanged).
- lib/belts.py: GT2_PULLEY_90T_FACE_Y (-13.2, 8.2: the hub's end .. the outer face), GT2_PULLEY_90T_BOLT_R 11,
  pulley_90t_bolt_points(). RollDriveParams.pulley_hub_len / nut_t now read them (21.4 / 3.2 unchanged);
  CouplerParams.pulley_screw_len 50 (a class default: LEGACY == DEFAULT on it).
- parts/joints/elbow_pulley_screws (4x M4 x 40), elbow_pulley_nuts (keyed radially, a flat toward the axis, as the
  block's channels hold them), wrist_pulley_screws (4x M4 x 50), wrist_pulley_nuts (a corner along the coupler's Z,
  as its pockets are cut): native COTS pattern parts (lib/reference.py NATIVE_COTS, reference/native/*.step accepted:
  2564.018 / 382.322 / 3066.672 / 382.322 mm^3, 4 solids each; manifest 45 -> 49 entries); MASS_G from the modelled
  steel 20.128 / 3.001 / 24.073 / 3.001 g (lib/params.py).
- gt2_pulley_90t becomes a diverged part: the SolidWorks body with its 4 holes cut to M4_CLEAR (CONVERTED = True,
  REFERENCE_BUILD = the untouched reference); 24810.708 -> 24531.703 mm^3 (-279.005, the analytic ring volume).
- lib/mounts.py FASTENER_MOUNTS: each screw set hosted on its 90T (heads on the outer face, +Z into the hub), each nut
  set on its screws at the host's seat (elbow 35.4: nut_seat_x; wrist 43.6: the pocket floor); AXES checks each
  pattern is centred on its joint axis. placements.json (mount_placements.py): parts 45 -> 49, solids 105 -> 121,
  volume 1927856.167 -> 1933693.491 (#3 / #4 records 24810.708 -> 24531.703).
- assemblies/arm.py OCCURRENCES + GROUPS, robot/frames.py LINKS; tools/bom.py EXTRAS: the elbow M4 x 40 and M4 nut
  rows removed (now modelled).
- tests: test_mounts test_the_pulley_bolts_reach_their_nuts (the stack arithmetic: tip 2 pitches past each nut,
  both hosts on the pulley's hole circle) and the slow test_pulley_bolts_clamp_their_joints (heads on the pulley's
  face, the nuts on the channel seats / pocket floors, the M4_CLEAR holes probed, the ring the heads sweep clear of
  the parent link through a whole turn, the nut press two-sided); the neighbours test's one budget is the nuts'
  designed press, computed: elbow nuts x the roll drive 23.03, wrist nuts x j3_coupler 20.15 mm^3 (4 x (hex 7.0 -
  hex 6.85) x 3.2 / 2.8), + 0.5 (wrist nuts x wrist_link 0.014: the 0.4 proud corner in its central hole);
  test_bom the four rows; test_parts_convention MULTI_BODY and PURCHASE_QTY == solids for *_screws / *_nuts.
Counts: arm leaves 69 -> 73, solids 202 -> 218, bought / printed leaves 36 / 33 -> 40 / 33; bom bought
(19, 36) -> (23, 40). Hash gate: only gt2_pulley_90t and arm changed (forearm_roll_block, j3_coupler and the
modules byte-identical), plus robot/links elbow_link / wrist_pitch_link.
Links (kg): elbow_link 0.718455 -> 0.74123, wrist_pitch_link 0.442705 -> 0.469425 (inertials + meshes
re-derived); total 5.734424 -> 5.783919.
Docs: open_issues.md (the arm's-fasteners row keeps the rest; the nut press row points at _press; the 90T in the
wrappers row; a new fit row: j3_coupler's Ø4.1 pulley-bolt holes for M4 in PETG), forearm_roll.md §0 purchased row,
§4 steps 1-2, §5; assemblies / lib / parts / robot / tests CLAUDE.md, vendor/README.md, the docstrings.
Full suite 759 passed, 14 skipped (the 4 new skips: no vendor file for the new parts); urdf / srdf / sdf validate; lint clean.

File: cad/robot/arm.urdf (robot description, URDF)
Before this commit: robot arm, 10 links, 9 joints
Links:
- link elbow_link: mass 0.718455 -> 0.74123
- link wrist_pitch_link: mass 0.442705 -> 0.469425

Commit message: cad: j1_link's elbow relief 1 mm deeper, the recess down to the bearing (gaps 3.0 / 2.0)
More room between the elbow block and the upper arm it turns over. The underside gaps were 2.0 mm and the boss's
1.5 mm; that is still little for printed PETG faces with the forearm's moment tilting the block on its 6806 pair.
The boss can't get more than this without changing the block: the recess floor now sits level with the upper 6806's
top face (j1 y -6.0), leaving the seat exactly BEARING_6806_WIDTH (7.0) deep.
- lib/upper_arm/params.py ElbowParams: new relief_y, the relief's floor (0 = the lip's root). DEFAULT relief_y -1.0
  (host -11), recess_y -5.5 -> -6.0. lib/upper_arm/link.py cuts the relief down to relief_y. The plate under the
  relief is still >= 15 mm thick, because the relief starts past the chamfer.
- Gaps (closest_points, at elbow 0 / +/-45 / +/-90): block and end cap underside 2.0 -> 3.0 mm, boss 1.5 -> 2.0.
  The block's nearest point, the journal's edge by the bore's rim, goes 1.02 -> 1.22 mm; it is a radial gap the
  bearings set.
- j1_link DEFAULT volume 346810.0 -> 342220.6 mm^3, 440.45 -> 434.62 g.
Links (kg): upper_arm_link 0.953232 -> 0.947403 (inertial + mesh re-derived); total 5.774208 -> 5.768379.
- tests: test_roll_drive's UPPER_ARM_FACE_Z -10 -> -11, the recess floor -15.5 -> -16, FACE_GAP 1.5 -> 2.0.
  test_j1_link's relief probes and volume read relief_y. test_the_6806_pair_fits_every_belt_joint_bore holds the
  seat at 7.0.
Docs: forearm_roll.md (§0 clearances row, §2 block row); the block comments in lib/params.py and
lib/forearm/params.py; j1_link's params docstring.

File: cad/robot/arm.urdf (robot description, URDF)
Before this commit: robot arm, 10 links, 9 joints
Links:
- link upper_arm_link: mass 0.953232 -> 0.947403

Commit message: cad: the base's motor lobe is a bolt-on part (base_motor_mount, 4x M4 into captive nuts), the motor slotted at the 280-2GT's centre distance
The base printed as one piece: the round bearing tower and the box-shaped +X lobe whose 5 mm plate carries the
base_yaw 48 mm motor. A change to the motor seat or the belt meant reprinting the whole base, and the lobe's plate and
U rim printed as a large overhang. The lobe is now its own part, bolted back on across a vertical joint face at
x = split_x (55, 1.66 past the tower's round), so it can be reprinted or swapped alone and prints plate down without
supports.

The joint: a rib inside each side wall on both parts (rib_w 12 deep, rib_t 8 thick, from the bottom face up to the
plate's underside), 2x M4 SHCS per rib along X (bolt_inset 8 under the plate and above the bottom face). The heads sit
on the mount's ribs and are turned from inside the mount, beside the motor (the ribs start 15 mm outside the motor's
face). The nuts are pressed into hex pockets in the base's ribs (nut_pocket_af 6.85 on the 7.0 nut, a corner up, their
outer faces flush with the ribs' back faces), so a reprinted mount needs no nuts. M4 x 20: the tips 4.0 past the nuts,
into the base's cavity below the plate. Nothing extra locates the parts: the bolts, the shared bottom face and the
belt's pull toward the axis, which presses the faces together.

The motor moves to where a stock belt puts it. The SolidWorks centre (78.97 from the axis) wanted a 274.2 mm 2GT belt;
YAW_BELT 280 (the stock list's) sets 81.97 (264 would pull the motor to 73.6, across the joint). The holes become
slots of +/- MOTOR_TRAVEL 2.5 along X (Ø M3_CLEAR 3.4, was Ø3.2) to tension the belt. The pilot's window slides with
them (x 68.27..95.67, was 67.99..90.15) and is cut only as high as the pilot needs (+/- 11.2 in Z, was +/- 21.3, which
would have run into the -X slots; 2.6 mm web left). The rim's +X side follows the slots out (slot_x1 100.27 ->
105.77), and the belt slot starts at the joint face, so the base's plate neck stays whole.

- lib/base/params.py:
  - new JointParams (split_x, rib_w, rib_t, bolt_inset, bolt_dia M4_CLEAR, screw M4_SHCS, screw_len 20, nut M4_NUT,
    nut_pocket_af 6.85);
  - MotorParams.travel (LEGACY 0);
  - BaseConfig.joint (LEGACY None, so build_base(LEGACY) still reproduces the SolidWorks part and REFERENCE_BUILD is
    untouched);
  - YAW_BELT, MOTOR_TRAVEL, WINDOW_CLEAR 0.2; DEFAULT gains the joint and the slotted seat.
- lib/base/layout.py: joint_bolt_points(), joint_stations().
- lib/base/body.py:
  - build_base(DEFAULT) keeps the -X side of the joint face and adds the ribs, the holes and the nut pockets;
  - new build_motor_mount(DEFAULT) keeps the +X side and adds its ribs and holes, the belt slot from the joint face;
  - _plate cuts slots when travel > 0.
- New parts in parts/base/:
  - base_motor_mount (NATIVE printed);
  - base_motor_mount_screws / _nuts (NATIVE COTS patterns, 4 solids each).
  The references were accepted (manifest 54 -> 57 entries): the mount 94793.893 mm^3, the screws 1558.7, the nuts
  382.3.
- lib/params.py: BASE_MOUNT_SCREWS_MASS_G 12.2 / BASE_MOUNT_NUTS_MASS_G 3.0 (the modelled steel);
  BASE_MOTOR_PATTERN_CENTRE (78.971441, -44.9, 0.08362) -> (81.971675, -44.9, 0.08362).
- lib/mounts.py:
  - new BASE_MOUNTS, declared first: the mount on base#1 at identity, the screws on the mount, the nuts on the screws;
  - nema17_48mm#1 is re-hosted on base_motor_mount#1.
  assemblies/arm.py OCCURRENCES / GROUPS and robot/frames.py LINKS["base_link"] take the three keys.
- base re-measured: 286395.592 -> 213232.726 mm^3; bbox x max 114.839 -> 55.
  Base + mount 308026.619: +21631 of ribs, less the holes and pockets.
- reference/placements.json (mount_placements.py):
  - leaf_occurrences 52 -> 55;
  - solids 124 -> 133;
  - solid_volume 1948910.581 -> 2045645.504.
- tests:
  - test_placements: 55 records, 133 solids; the mounted keys; NATIVE parts are known record parts.
  - test_assembly: leaves 79 -> 82, solids 230 -> 239, tints.
  - test_bom:
    - leaves 79 -> 82;
    - printed (27, 34) -> (28, 35);
    - bought (27, 45) -> (29, 47);
    - new test_the_base_motor_mount_takes_its_m4_screws_and_nuts.
  - test_parts_convention MULTI_BODY: the screws + nuts, 4 each.
  - test_mounts:
    - a motor's host may be the printed mount;
    - the mount is a neighbour in the clearance check;
    - the nuts' press in the base's ribs is budgeted.
  - tests/base/test_base.py: DEFAULT also splits; its bbox ends at split_x.
  - New tests/base/test_motor_mount.py:
    - the belt arithmetic;
    - the seat, the joint layout;
    - the faces meeting without overlap, the nut pockets, the slotted seat;
    - the screws' heads and tips;
    - the motor and board clear of the mount at both ends of the travel.
- robot: base_link mass 0.913722 -> 0.956431 kg, COM (-46.897, 0.021, 47.559) -> (-48.670, 0.021, 46.744) mm,
  ixx / iyy / izz 1.426810e-3 / 2.809310e-3 / 2.669327e-3 -> 1.528945e-3 / 2.926819e-3 / 2.833294e-3, ixy / ixz / iyz
  2.631768e-6 / -6.989411e-4 / 1.215159e-6 -> 2.729990e-6 / -7.265972e-4 / 1.197490e-6 (arm.urdf and arm.sdf);
  meshes/base_link.stl re-exported. derive --check and validate --strict are clean.
- The hash gate against the branch point's builds on this machine: only the base, arm and base_link STEPs changed.
- docs:
  - the base's docstring;
  - lib/, assemblies/, robot/ CLAUDE.md;
  - open_issues.md:
    - the base_yaw drive row names YAW_BELT and the slots, no longer the 274.2 mm belt;
    - the 6.1 mm row points at the mount;
    - new Estimates rows: the joint's PETG fits; the 280-2GT belt and the motor held by its M3s' clamp alone (no
      tension screw); the two parts' print orientations.

File: cad/robot/arm.urdf (robot description, URDF)
Before this commit: robot arm, 10 links, 9 joints
Links:
- link base_link: mass 0.913722 -> 0.956431
