Commit message: cad: base_motor_mount narrows to the motor + 10 mm of wiring room, bolted by outward ears; the base's end opens into it
The motor mount was the whole SolidWorks lobe, the base's full width (106.7). The motor only needs room round it for
its wiring, so the mount is now a box of its own round the motor and its MKS board.

The mount:
- Inside, MountParams.room 10 clear of the board's 43 mm square: the walls ±31.58 inside (±36.58 outside, 73.2 wide).
  The end wall's inside is 10 past the board at the slots' middle, 7.5 at full tension; its outside moves
  114.84 -> 118.47.
- Walls wall 5, from the bottom face (it still stands on the table) up to the plate's top. The plate keeps the
  motor's slotted seat, the window and the U rim. It is open underneath and toward the base.
- The belt slot is gone. It split the plate lengthwise, and the belt runs about 8 mm above the plate by the
  estimate.
- The cable notch in the end wall is gone: the cables now go into the base.

The joint:
- An ear outside each side wall at the joint face: ear_w 12, ear_t 8, full height. The M4 heads sit on the ears'
  outer faces and are turned from outside, along -X beside the walls (2.5 clear of them).
- In the base the internal ribs become posts: post_t 8, from the side walls in to the mount's inside. The window
  between them, full height, opens the mount into the base.
- The M4 x 20 and the nuts pressed into the posts stay (nut_pocket_af 6.85). The bolt z moves 42.34 -> 42.58.
- Where the cables leave the base is not decided yet: a new open_issues row.

- lib/base/params.py:
  - new MountParams (room, wall, ear_w, ear_t) and BaseConfig.mount (LEGACY None);
  - JointParams.rib_w / rib_t -> post_t.
- lib/base/layout.py: new mount_inner_half(), mount_x1(). joint_bolt_points() is on the ears; joint_stations()
  x_base_rib -> x_post.
- lib/base/body.py:
  - build_motor_mount builds the box, no longer clipping the SolidWorks lobe;
  - build_base's _ribs -> _posts;
  - the motor's window and holes are one helper, _motor_seat, shared with the SolidWorks plate. build_base(LEGACY)
    is unchanged at 286169.1 mm^3.
- base 213232.726 -> 217493.959 mm^3 (the posts are wider than the ribs). The base_motor_mount reference is
  re-accepted: 94793.893 -> 86160.255 mm^3, bbox 59.839 x 61 x 106.679 -> 63.472 x 61 x 97.167. The screws and nuts
  are re-accepted at the new bolt z (volumes unchanged: 1558.7 / 382.3).
- reference/placements.json (mount_placements.py): solid_volume 2045645.504 -> 2037011.866 (counts unchanged).
- robot: base_link mass 0.956431 -> 0.950878 kg, COM (-48.670, 0.021, 46.744) -> (-48.251, 0.021, 46.552) mm,
  ixx / iyy / izz 1.528945e-3 / 2.926819e-3 / 2.833294e-3 -> 1.438979e-3 / 2.916307e-3 / 2.727519e-3, ixy / ixz /
  iyz 2.729990e-6 / -7.265972e-4 / 1.197490e-6 -> 2.745546e-6 / -7.315278e-4 / 1.190829e-6 (arm.urdf and arm.sdf);
  meshes/base_link.stl re-exported. derive --check and validate --strict are clean.
- tests/base/test_motor_mount.py:
  - new: the wiring room (in Z at any travel, to the end wall at the middle and at full tension);
  - the ears and posts hold the heads and pockets, and the heads clear the walls;
  - probes of the posts, the window, the ears, the walls, the whole plate and the plain end wall;
  - the board stays room - travel clear of the mount across the travel.
- tests/base/test_base.py: DEFAULT's identity also restores mount.
- The hash gate against the previous commit's builds on this machine: only the base, base_motor_mount (+ screws,
  nuts), arm and base_link STEPs changed.
- docs:
  - the parts' docstrings;
  - lib/, assemblies/, robot/, tests/ CLAUDE.md;
  - open_issues.md: the joint-fits row names the posts and ears; a new Not modelled row for the cables' way out of the
    base.

File: cad/robot/arm.urdf (robot description, URDF)
Before this commit: robot arm, 10 links, 9 joints
Links:
- link base_link: mass 0.956431 -> 0.950878

Commit message: cad: base_motor_mount loses the U rim under its plate
The mount still carried the SolidWorks base's U rim: a 2 mm wall, 7 deep, hanging under the plate round three sides
of the motor's face, 0.3 mm clear of it. It is not wanted. The motor is located by its 4 M3s in the slots (Ø3.4 for
an M3: ±0.2 across them), so nothing hangs under the plate now.

- lib/base/body.py: build_motor_mount no longer adds _rim. _rim is the SolidWorks base's only again: its ends on the
  shell's round, the joint branch gone. build_base(LEGACY) is unchanged (286169.1 mm^3, the reference match), and so
  is build_base(DEFAULT) (the base's STEP is byte-identical).
- lib/base/params.py: DEFAULT drops its slot_x1 override, the rim's +X inside (only the rim and the SolidWorks belt
  slot read it). The MotorParams docstring says the belt slot and the rim are the SolidWorks base's only.
- base_motor_mount re-accepted: 86160.255 -> 84086.2 mm^3 (bbox unchanged, 63.472 x 61 x 97.167).
- reference/placements.json (mount_placements.py): solid_volume 2037011.866 -> 2034937.859.
- robot: base_link mass 0.950878 -> 0.948244 kg, COM (-48.251, 0.021, 46.552) -> (-48.138, 0.021, 46.535) mm,
  ixx / iyy / izz 1.438979e-3 / 2.916307e-3 / 2.727519e-3 -> 1.437827e-3 / 2.911101e-3 / 2.721369e-3, ixy / ixz /
  iyz 2.745546e-6 / -7.315278e-4 / 1.190829e-6 -> 2.738857e-6 / -7.321631e-4 / 1.191813e-6 (arm.urdf and arm.sdf);
  meshes/base_link.stl re-exported. derive --check and validate --strict are clean.
- tests:
  - tests/base/test_motor_mount.py: the rim asserts go; a probe finds nothing under the plate where the rim stood.
  - tests/base/test_base.py test_layout: DEFAULT's slots, no longer its rim.
- The hash gate against the previous commit's builds on this machine: only base_motor_mount, arm and base_link
  changed.
- The mount's docstrings follow.

File: cad/robot/arm.urdf (robot description, URDF)
Before this commit: robot arm, 10 links, 9 joints
Links:
- link base_link: mass 0.950878 -> 0.948244

Commit message: cad: wrist_link is parametric (lib/wrist/, LEGACY reproduces the SolidWorks part)
The wrist body was still the imported SolidWorks shape, so none of its features could be re-sized; it becomes code
first. This commit is the port only: DEFAULT = LEGACY, no design change. Every number was measured on the reference
(face / vertex census) [REFERENCE].

- lib/wrist/ (a leaf, in tests/test_layering.py LEAF_PACKAGES): params.py WristConfig (PlateParams, SeatParams,
  TowerParams, EndFaceParams; LEGACY = the SolidWorks part, DEFAULT = LEGACY), layout.py (seat_bolt_points,
  end_face_holes, slope_x), link.py build_wrist_link(cfg).
- parts/wrist/wrist_link.py: CONVERTED = True, REFERENCE_BUILD = build_wrist_link(LEGACY), LOCAL_FROM_REF =
  IDENTITY (the SolidWorks part frame, which placements.json places).
- tests/wrist/test_wrist_link.py: the seat is j3_coupler's flange (its Ø, bolt circle, holes, nut pockets), the end
  face's M3 are the NEMA 17 pattern about the roll axis; LEGACY's plate, seat, tower, fillet, cheeks, back opening,
  block and end-face holes probed by name (slow); DEFAULT == LEGACY.

Kept as SolidWorks made them (later commits can change DEFAULT): the end face's M3 / M4 are drilled through the whole
part along X, so the z 6.5 pair score the coupler's seat face 0.1 / 0.6 deep; the back opening is out to y 30 on +Y
but only to the bore on -Y; the seat's holes are Ø4.1 over 2 mm nut pockets.

Match (LEGACY against reference/solidworks/wrist_link.step):
- volume, adaptive integration (BRepGProp eps 1e-7): 113609.023 vs 113601.567 mm^3 (+7.46, +0.007 %); an 8 x 6 x 4
  grid of cells agrees to 0.4 mm^3 a cell but for the fillet's top: +4.57 in each of the two cells at |y| < 10,
  z > 35.
- bbox identical (min (-84.446, -39, 0), size (124.446, 78, 44)); 71 faces vs 104 (the reference splits its
  holes' and fillet's faces).
- One simplification: where the slope's edge with the bore runs out at the tower's top (a point), SolidWorks rolled
  the R10 ball along the top edge for the last ~3 mm (|y| < 13.8); build123d's fillet() cannot run through that
  point, so it is made on a core carried above the top and trimmed there: +9.1 mm^3 at the top, -1.8 along the
  fillet's sides, +7.3 net.
- OCCT's default .volume reads the trimmed fillet face low: 113541.932 (-59.47 against the reference, -0.052 %,
  inside test_reference_match's 0.5 %), and the error jumps with unrelated construction changes (the fillet core's
  height) - lib/CLAUDE.md Kernel gotchas now says so. derive.py's inertials use the same integration.

wrist_pitch_link: derive.py --check named it (ixy and iyz past its 1e-3 relative tolerance); its inertial is pasted
from the drafts into robot/arm.urdf and arm.sdf and its mesh re-exported:
- mass 0.469425 -> 0.469349 kg (-0.076 g: the default integration's -59.5 mm^3 at PETG density)
- COM (0.056998, 0.000064, -0.015489) -> (0.057, 0.000066, -0.015487) m
- ixx 2.263282e-04 -> 2.263088e-04, ixy -8.075530e-07 -> -8.101134e-07, ixz 2.195330e-05 -> 2.196099e-05,
  iyy 9.982938e-04 -> 9.982734e-04, iyz 3.914792e-08 -> 5.072278e-08, izz 1.039618e-03 -> 1.039608e-03 kg.m^2

No lock moved: the arm / link totals take a converted part's own build (tests/totals.py). Hash gate: only
wrist_link.step and arm.step changed. Suite: 823 passed, 18 skipped.

Docs: lib/CLAUDE.md (wrist/, the fillet's volume gotcha), parts/CLAUDE.md Part states, tests/CLAUDE.md,
docs/open_issues.md (the wrist_link "Not converted yet" row removed).

File: cad/robot/arm.urdf (robot description, URDF)
Before this commit: robot arm, 10 links, 9 joints
Links:
- link wrist_pitch_link: mass 0.469425 -> 0.469349

Commit message: cad: base_motor_mount's walls become V trusses, 4 mm thick
The mount's solid 5 mm side walls and end wall were ~63 % of its plastic, but they carry little. The belt's pull
runs along the plate straight into the ears, and the top M4 sits 8 mm under the plate. The motor and its board weigh
~0.44 kg. The walls only stand the plate on the table and keep the ears square. They are now open V trusses: less
plastic and weight, and the wiring can be reached from the sides and the end.

Each wall below the plate keeps a frame, MountParams.strut 6 wide:
- a rail under the plate and a rail on the table;
- a post at each end, from the outer corner, so the corner posts take in the other wall. The side walls' post at the
  joint is as deep as the ears (8), so each ear stays backed by solid wall.

Inside the frame a V: two 6 mm struts from its top corners down to the middle of the bottom rail, with the three
triangles between open. The struts stand at 61.2 deg in the side walls and 56.1 deg in the end wall. Printed
plate-down, the middle triangle is self-supporting and the side ones bridge only their table edge: 20.8 mm in the
side walls, 26.0 in the end wall. No supports.

The walls also go from 5 to 4 mm (MountParams.wall):
- the outside ±36.58 -> ±35.58, the ears ±35.58..±47.58;
- the bolt z ±42.58 -> ±41.58;
- mount_x1 118.47 -> 117.47.
The inside, and so the wiring room, is unchanged.

- lib/base/params.py: MountParams.wall 5 -> 4, a new strut 6; the docstring describes the truss.
- lib/base/layout.py: new truss_panels() - per wall its plane, the frame's inside and the V's centrelines, shared by
  the builder and the tests.
- lib/base/body.py: new _strut() and _truss_windows(); build_motor_mount cuts the windows. build_base and LEGACY are
  untouched (286169.1 mm^3); the base's bolt holes and nut pockets move with the bolt z (volume unchanged at
  217494.0 mm^3).
- base_motor_mount re-accepted: 84086.2 -> 51397.2 mm^3 (-39 %; ~107 -> ~65 g solid PETG), bbox 63.472 x 61 x
  97.167 -> 62.472 x 61 x 95.167. The screws and nuts are re-accepted at the new bolt z (volumes unchanged).
- reference/placements.json (mount_placements.py): solid_volume 2034937.859 -> 2002248.785.
- robot: base_link mass 0.948244 -> 0.906729 kg, COM (-48.138, 0.021, 46.535) -> (-45.849, 0.022, 47.342) mm,
  ixx / iyy / izz 1.437827e-3 / 2.911101e-3 / 2.721369e-3 -> 1.376604e-3 / 2.765055e-3 / 2.559417e-3, ixy / ixz /
  iyz 2.738857e-6 / -7.321631e-4 / 1.191813e-6 -> 2.784035e-6 / -6.939329e-4 / 1.207728e-6 (arm.urdf and arm.sdf);
  meshes/base_link.stl re-exported. derive --check and validate --strict are clean.
- tests/base/test_motor_mount.py:
  - new test_the_walls_are_trussed (the layout: struts >= 45 deg, bridges <= 30 mm, the ears backed);
  - new test_the_truss_windows_are_open (per wall the three triangles open; the struts, rails and posts solid);
  - the joint test's wall probes move onto the rails.
- The hash gate against the previous commit's builds on this machine: only the base, base_motor_mount (+ screws,
  nuts), arm and base_link STEPs changed.
- docs:
  - the mount's docstring;
  - the open_issues print row names the truss's struts and bridges.

File: cad/robot/arm.urdf (robot description, URDF)
Before this commit: robot arm, 10 links, 9 joints
Links:
- link base_link: mass 0.948244 -> 0.906729

Commit message: cad: the drive housing has 6 pillars, j1_coupler's yoke holds the two at +/-30 degrees
The cycloidal drive's housing (motor plate + ring gear body) goes from 8 outer
pillars to 6: HousingParams.bolt_count 8 -> 6, the same 0-degree start, so the
pillars and their M4 housing bolts sit at 0, 60 .. 300 degrees from the drive's
+X. Three bolts now line up with ring pins 0 / 7 / 14, 8.5 mm out, as the
port's bolt 0 already did; the pillar trapezoid (18 / 10) is unchanged, so the
windows at the bore widen from ~28 to ~43 mm.

The port stays checkable. lib/cycloidal/params.py keeps the CadQuery port as
LEGACY_CONFIG and builds DEFAULT_CONFIG (bolt_count 6). The motor plate, the
ring gear body and the housing bolts / nuts declare REFERENCE_BUILD (their
LEGACY_CONFIG build); test_port and test_cots_envelope_tracks_reference_bbox
now compare that, as test_reference_match already did. The pillar outline moves
into lib/cycloidal/layout.py (pillar_corners, pillar_half_width,
PILLAR_OVERSHOOT), shared by the housing's cutter and the yoke.

j1_coupler's DEFAULT yoke follows the housing. In the arm the drive's +X lies
on the coupler's +Z, so the 6 pillars sit at +/-30, +/-90 and +/-150 degrees
from the cradle's bottom: none at the bottom or at +/-45 any more. The
SolidWorks channel, bolt-head notch and V-grooves go (the middle body up to the
cheek's top line), and the two pillars at +/-30 sit in closed sockets
(YokeParams.socket_deg, the pillar's sides and end socket_clear 0.2 out). The
cheek's nut pockets move under those two bolts (bolt_deg). The pillars come
down close to the ring: near the motor-plate end the flare left 0.4-0.6 mm
under each socket's floor corner, so each socket carries a socket_wall 2.0
wall even where the flare trims the yoke - a small rib under it at the ends.
LEGACY (the SolidWorks part) is untouched and still matches its reference.

Numbers:
- drive module: solids 77 -> 73, volume 679467.512 -> 659601.475 mm^3
  (stator 71 -> 67 solids, 579459.085 -> 559593.048; rotor unchanged),
  bbox 140 x 140 x 127.1 -> 140 x 124.908 x 127.1 (no pillar on the drive's Y)
- cycloidal_motor_plate 99475.823 -> 96993.785 mm^3,
  cycloidal_ring_gear_body 158114.513 -> 142692.276,
  housing bolts 8 -> 6 (6760.707 -> 5070.531), nuts 8 -> 6 (1086.342 -> 814.757)
- CYCLOIDAL_HOUSING_BOLTS_MASS_G 53.1 -> 39.8, CYCLOIDAL_HOUSING_NUTS_MASS_G
  8.5 -> 6.4; the drive's buy list 53 -> 49 pieces
- j1_coupler (DEFAULT) 193586.007 -> 202541.237 mm^3, bbox unchanged;
  socket skin >= 2.0 mm
- arm: solids 230 -> 226, volume 2897394.375 -> 2886483.568 mm^3
- interference budgets: housing bolts x nuts 322.0 -> 241.3 mm^3;
  drive x j1_coupler 150 -> 35 (measured 30.8, was ~118: the pillars now
  clear their sockets, what is left is the cradle against the housing,
  whose axis sits 0.21 off the cradle's)
- shoulder_link inertial (arm.urdf / arm.sdf, mesh re-exported):
  mass 1.679319 -> 1.652554 kg, COM (-0.000808, 0.015169, -0.011927) ->
  (-0.000825, 0.0154, -0.012376), ixx 3.952462e-03 -> 3.863150e-03,
  iyy 3.676363e-03 -> 3.554768e-03, izz 2.908848e-03 -> 2.847775e-03,
  ixy 1.418813e-05 -> 1.624620e-05, ixz 1.492821e-05 -> 1.554289e-05,
  iyz -3.017000e-04 -> -3.118576e-04; the arm 5.848 -> 5.821 kg

test_module_world_bbox_matches_solidworks_node now asks the module to lie
inside the 8-pillar SolidWorks node's box and fill it but along the drive's
+Y (world up). docs/open_issues.md's "not fastened to j1_coupler" row stays
open, rewritten for the cheek's two nut pockets and the sockets; robot/frames.py
no longer calls the stator "bolted" into the yoke.

File: cad/robot/arm.urdf (robot description, URDF)
Before this commit: robot arm, 10 links, 9 joints
Links:
- link shoulder_link: mass 1.679319 -> 1.652554

Commit message: cad: the base and its motor mount reach 11.1 mm lower, the base_yaw motor's board 5 mm clear of the table
The base_yaw 48 mm motor and its MKS board (48 + 14.1 under the motor mount's plate) hung 6.1 mm below the base's
bottom face, the SolidWorks y -100.9, so the arm could not stand on a table. The bottom face now sits BOARD_CLEAR
(5.0) under the board: y -100.9 -> -112.0 (DEFAULT.shell.y0, from the plate, the motor's body length, the board stack
and the clearance). The base's D walls and posts and the whole motor mount reach down to it. The truss walls are
taller, so their struts are steeper: 61.2 -> 66.3 deg in the side walls, 56.1 -> 61.8 in the end wall. Their bridges
are about the same (20.96 / 26.18 mm). The bottom M4s follow the face (bolt_inset 8 above it). This closes the
open_issues row "the base_yaw motor + its MKS board reach 6.1 mm below the base's bottom face" (d9662a3).

The base_link frame stays on the mounting face (lib/datum.py BASE_BOTTOM_Y = DEFAULT.shell.y0, REP-103), so it moves
down with it:
- the base_yaw joint's origin in base_link rises 0.18591 -> 0.19701 m (arm.urdf, arm.sdf);
- arm.step, emitted in that frame, sits 11.1 mm higher;
- no other joint or link frame changes (they are in the capture frame).
LEGACY still reproduces the SolidWorks base at -100.9.

- lib/base/params.py: BOARD_CLEAR 5.0; DEFAULT.shell.y0 derived (-112.0).
- lib/params.py: BASE_MOTOR_STACK_PROUD 6.1 (below the face) -> BASE_MOTOR_TABLE_CLEAR = BOARD_CLEAR (above it).
- lib/datum.py: BASE_BOTTOM_Y's comment ([DESIGN] -112.0).
- base: 217494.0 -> 235439.082 mm^3.
- base_motor_mount re-accepted: 51397.2 -> 56295.1 mm^3, bbox 62.472 x 61 x 95.167 -> 62.472 x 72.1 x 95.167. The
  screws and nuts are re-accepted at the lower bottom bolts (volumes unchanged).
- reference/placements.json (mount_placements.py): solid_volume 2002248.785 -> 2007146.747.
- robot:
  - base_yaw origin z 0.18591 -> 0.19701 m;
  - base_link mass 0.906729 -> 0.93574 kg, COM (-45.849, 0.022, 47.342) -> (-44.986, 0.021, 56.664) mm;
  - ixx / iyy / izz 1.376604e-3 / 2.765055e-3 / 2.559417e-3 -> 1.515585e-3 / 2.940607e-3 / 2.693847e-3;
  - ixy / ixz / iyz 2.784035e-6 / -6.939329e-4 / 1.207728e-6 -> 2.801067e-6 / -6.562157e-4 / 1.172646e-6
    (arm.urdf and arm.sdf);
  - meshes/base_link.stl re-exported.
  derive --check and validate --strict are clean.
- tests:
  - test_mounts: test_base_motor_stack_hangs_below_the_base_by_the_documented_amount ->
    test_base_motor_stack_clears_the_table (the board BASE_MOTOR_TABLE_CLEAR above the face, the base and mount
    down to it).
  - test_params_invariants: the same arithmetic, the other way.
  - tests/base/test_base.py: BASE_BOTTOM_Y is DEFAULT's, below the SolidWorks record's; DEFAULT.shell is LEGACY's
    deeper; the bbox min follows.
- The hash gate against the previous commit's builds on this machine: only the base, base_motor_mount (+ screws,
  nuts), arm and base_link STEPs changed.
- docs:
  - the base's docstring;
  - lib/mounts.py, assemblies/ and robot/ CLAUDE.md name BASE_MOTOR_TABLE_CLEAR;
  - open_issues.md loses the 6.1 mm row.

File: cad/robot/arm.urdf (robot description, URDF)
Before this commit: robot arm, 10 links, 9 joints
Links:
- link base_link: mass 0.906729 -> 0.93574
Joints:
- joint base_yaw: origin xyz=0 0 0.18591 rpy=0 0 0 -> xyz=0 0 0.19701 rpy=0 0 0
