Commit message: cad: the cycloidal drive shrinks to a Ø100 pin ring (housing Ø140 -> Ø132)
The shoulder drive took more room than its parts need: the discs carried ~15 mm of
material outside their output-pin holes, and the housing is stacked outside the ring
pins. DEFAULT_CONFIG now moves the ring-pin circle and everything outside it RING_INSET
(4 mm, radial) in from the port, so every wall outside the pins keeps the port's
thickness and the drive is 8 mm smaller across:

  ring-pin circle   Ø108 -> Ø100
  bore (the outline between the pillars)  Ø116 -> Ø108
  bolt circle       Ø125 -> Ø117
  od (pillar tips)  Ø140 -> Ø132

The bore moves with the pins, not further: between the pillars the housing's outline
IS the bore, 1.9 outside the pin holes; a Ø106 bore left 0.9 there and the 1.5 edge
chamfer broke into the holes. The limit on the pins is the wall between their far ends
and the 6814 seat: 6.8 -> 2.8 over the 3.5 mm the pins sit in it
(test_pin_holes_dont_breach_bearing_seat floor 5 -> 2.5); test-print the seat.

Discs: tips R - r + e 53.5 -> 49.5, bbox 105.9 / 107.0 -> 98.0 / 99.0; K1 = e*N/R
0.583 -> 0.630, no undercut; valley to output-pin hole wall ~15 -> ~12. Each ring pin
carries ~8 % more force for the same torque (54 / 50). Unchanged: the ratio, the motor,
the 6003 / 6814 / 625, the hub and its j1_link pattern, the output pins, the shaft, the
stack-up (60 deep), the fasteners, the BOM, the drive's pose in the arm.

The discs and the ring pins now declare REFERENCE_BUILD (their LEGACY_CONFIG build), like
the housing parts, so test_port / test_cots_envelope_tracks_reference_bbox keep matching
the CadQuery exports.

j1_coupler: DEFAULT's yoke takes its cradle_r / od_r / bolt_circle_r from DEFAULT_CONFIG's
housing (58 / 70 / 62.5 -> 54 / 66 / 58.5) with the drive's axis where it was, so the
cradle's floor rises 4 mm and the cheeks' top on the cradle rises y 55.78 -> 63.11. Its
sockets follow the pillars; the rib under the socket walls now sits inside the flare.

Measured:
- drive module solid volume 659601.475 -> 589029.752 mm^3 (stator 559593.048 ->
  489021.325; rotor 100008.427 unchanged); bbox 140 x 124.908 x 127.1 -> 132 x 117.972 x
  127.1; housing parts' Y extent 124.908 -> 117.972
- printed drive parts (plate + body + 2 discs) 398.9 -> 328.3 cm^3; j1_coupler 202.5 ->
  230.3 cm^3
- drive vs j1_coupler contact (the 0.21 axis offset of the capture, open_issues)
  ~30 -> 45.2 mm^3 (motor plate 11.3 + ring gear body 34.0: the cradle wraps a longer
  arc); limit 35 -> 50
- shoulder_link mass 1.652554 -> 1.598232 kg, COM (-0.000825, 0.0154, -0.012376) ->
  (-0.000855, 0.015917, -0.013816), ixx / iyy / izz 3.863150e-03 / 3.554768e-03 /
  2.847775e-03 -> 3.689181e-03 / 3.286729e-03 / 2.697849e-03; arm total 5.842 -> 5.788 kg;
  shoulder_link.stl re-exported

Tests: the SolidWorks-node bbox check requires the fill only along the drive's axis; the
LEGACY yoke is compared with LEGACY_CONFIG's housing, DEFAULT's with DEFAULT_CONFIG's; the
yoke's socket probes are relative to the housing's od. Checks: ./cadtool lint; the full
suite (812 passed, -n 4); derive.py --check clean; validate --strict (URDF, SRDF, SDF);
the hash gate changed only the discs, motor plate, ring gear body, ring pins, housing
bolts / nuts, j1_coupler, cycloidal_drive and arm STEPs; snapshots of the drive, the arm
and arm.urdf looked at.

File: cad/robot/arm.urdf (robot description, URDF)
Before this commit: robot arm, 10 links, 9 joints
Links:
- link shoulder_link: mass 1.652554 -> 1.598232

Commit message: cad: the drive's pillar tips trimmed, housing od Ø132 -> Ø129.2
The six bolt pillars stood 3.3 mm of plastic past a corner of each M4 nut pocket. Each
housing nut and its pocket now turn a flat outward (HousingParams.bolt_nut_turn_deg 30,
new; 0 in the port) and LUG_WALL = 2.5 stands past the pocket, so DEFAULT_CONFIG's od is
the bolt circle + the pocket's AF + 2 * LUG_WALL: 132 -> 129.2. The edge chamfer goes
1.5 -> 1.0 so the external faces keep 1.5 past the nut pockets (1.4 past the plate's
counterbores); a 1.5 chamfer would have left 1.0.

Kept: the M4 x 55 bolts and nuts, six pillars, their widths (18 at the bore, 10 at the
tip: they bridge the windows and key the housing in the yoke; 3.1 of wall beside the
turned nut, the bolt hole's 5.05), and the bolt circle (Ø117): pulled in, j1_coupler's
cheek nut pockets for the +/-30 degree bolts would break into its cradle. The hub's
captive nuts keep their orientation (the turn is applied at the ring gear body's and the
housing nuts' call sites, not in hex_pocket).

Measured:
- motor plate 84369 -> 83650 mm^3, ring gear body 110430 -> 105057 mm^3; printed drive
  parts 328.3 -> 322.2 cm^3; housing parts' bbox 132 x 117.972 -> 129.2 x 116.023
- drive module solid volume 589029.752 -> 582937.149 mm^3 (stator 489021.325 ->
  482928.722; rotor unchanged); bbox 132 x 117.972 x 127.1 -> 129.2 x 116.023 x 127.1
- j1_coupler (its od points and sockets follow od_r 66 -> 64.6) 230.3 -> 233.3 cm^3;
  drive vs j1_coupler contact 45.2 -> 45.5 mm^3 (limit 50)
- shoulder_link mass 1.598232 -> 1.594247 kg, COM (-0.000855, 0.015917, -0.013816) ->
  (-0.000858, 0.015952, -0.013965), ixx / iyy / izz 3.689181e-03 / 3.286729e-03 /
  2.697849e-03 -> 3.674871e-03 / 3.263627e-03 / 2.686198e-03; arm total 5.788 -> 5.784 kg;
  shoulder_link.stl re-exported

Tests: CYCLOIDAL_HOUSING_OD and the od lock 132 -> 129.2, edge_chamfer 1.5 -> 1.0, the
bbox and EXPECTED locks; the yoke's "stopped by the cheek" probe moves from 3 to 1 mm
inside the pillar's tip (3 now lands in the cheek's empty nut pocket). Checks: ./cadtool
lint; the full suite (812 passed, -n 4); derive.py --check clean; validate --strict
(URDF, SRDF, SDF); the hash gate changed only the housing nuts, motor plate, ring gear
body, j1_coupler, cycloidal_drive and arm STEPs; the drive's output side looked at.

File: cad/robot/arm.urdf (robot description, URDF)
Before this commit: robot arm, 10 links, 9 joints
Links:
- link shoulder_link: mass 1.598232 -> 1.594247

Commit message: cad: upper arm and forearm 40 mm shorter, the wrist belt 258-2GT, the shoulder's upper limit 75 deg
The arm's reach is long for its NEMA 17 drives: stretched out horizontally
the shoulder carries ~9.8 N.m (200 g payload) against ~5-6 available, the
elbow ~4.1 against ~1.1-1.8. The upper arm and the forearm each lose 40 mm
(upper arm SHORTENING -40, forearm SHORTENING +40 in their params); the
wrist follows in the next commit.

- j1_link: elbow_x 210 -> 170; every elbow-end feature moves with the
  axis (chamfer 145.5 -> 105.5, step 153.5 -> 113.5, stepped slot
  163 -> 123, the second stage's seat 128 -> 88: its 82 mm to the elbow
  kept, so a stock 258-2GT fits stage 1 at CD 88.08). The two through
  slots of unknown purpose are gone: the moved seat's boss landed on them.
- j2_link: wrist_x -210 -> -170. The wrist-pitch belt 264-2GT -> 258-2GT:
  J2_MOTOR_SLIDE_X -136.37 -> -99.52 (plug 5.52 mm inside its clearance
  rule, body 4.48 off the boss; a 264 would have left 2.37), the slide
  (-141.5, -130) -> (-103.5, -94), slots centre (-110, -88), side
  (-119, -78.5). DEFAULT.motor_x read LEGACY's web; now its own.
- lib/placements.py SHIFTS move everything beyond: T1 = -40 along j1_link
  +X, then +40 along j2_link +X. mount_placements.py rewrote the 13
  mounted records on the moved hosts; every SolidWorks record unchanged.
- A new contact: with the arm pitched down in front and the elbow folded
  back (shoulder +78 deg and up, elbow -90..-58), the forearm roll drive's
  MKS board and motor reach j1_coupler and the base (today's arm clears by
  14 mm everywhere above the table). SHOULDER_PITCH_LIMIT_DEG 120 ->
  SHOULDER_PITCH_LIMITS_DEG (-120, +75): 3 deg short of the first contact,
  4.41 mm clear at +75 / -90; costs 25 of 1,955 usable poses (1.3 %).
  tests/test_sweeps.py (slow, ~50 s) checks exact distances along the
  limit.

Numbers:
- reach to the fingertips, stretched: 646 -> ~566 mm (~546 after the wrist)
- j1_link 342,221 -> 299,936 mm3 (434.6 -> 380.9 g solid PETG);
  j2_link 254,434 -> 215,465 mm3 (323.1 -> 273.6 g)
- upper_arm_link 0.947403 -> 0.893701 kg, COM x 0.063934 -> 0.04954 m;
  forearm_link 0.811089 -> 0.761574 kg, COM z 0.124212 -> 0.098002 m;
  URDF total 5.784 -> 5.681 kg
- URDF/SDF: elbow_pitch x 0.210003 -> 0.170003, wrist_pitch z 0.21 -> 0.17,
  shoulder_pitch upper 2.094395 -> 1.308997
- arm: volume 2,847,774 -> 2,766,520 mm3, bbox 639.0 x 217.1 x 679.3 ->
  584.8 x 217.1 x 620.5 mm; leaves / solids unchanged (82 / 235)

Checks: hash gate - j1_link, j2_link, arm, upper_arm_link, forearm_link
changed; elbow / wrist_pitch / wrist_roll / jaw links only moved with
their frames (inspect diff: same geometry, 1e-6); derive --check OK after
copying the drafts; meshes re-exported for upper_arm_link, forearm_link;
URDF / SRDF --strict and SDF validate; full suite 844 passed; snapshots
of the arm and the URDF looked at.

File: cad/robot/arm.urdf (robot description, URDF)
Before this commit: robot arm, 10 links, 9 joints
Links:
- link forearm_link: mass 0.811089 -> 0.761574
- link upper_arm_link: mass 0.947403 -> 0.893701
Joints:
- joint elbow_pitch: origin xyz=0.210003 0 0.009998 rpy=0 0 0.010227 -> xyz=0.170003 0 0.009999 rpy=0 0 0.010227
- joint shoulder_pitch: limit lower=-2.094395 upper=2.094395 effort=5 velocity=1 -> lower=-2.094395 upper=1.308997 effort=5 velocity=1
- joint wrist_pitch: origin xyz=0.016998 0 0.21 rpy=-1.570799 -1.271722 -1.570793 -> xyz=0.016998 0 0.17 rpy=-1.570799 -1.271722 -1.570793

Commit message: cad: wrist body 20 mm shorter, the wrist pitch limits set to the measured clear range
The last 20 mm of the shortening (arm reach, previous commit): wrist_link's
block ends SHORTENING = -20 nearer the pitch axis (block_x1 40 -> 20), and
lib/placements.py SHIFTS moves what bolts to its end face - the gripper
bracket, the pancake, the 20T, the gripper - 20 mm along F.

- The weight-saving pocket behind the slope would break through the new
  end face: the slope's top moves slope_x1 30 -> 14 (the steepest whose cut
  stays inside the fillet's core), leaving 6 mm of block over the pocket.
- The wall and the plate's R39 round end reached x 39; both are now
  clipped at the end face (LEGACY unchanged: same faces / edges / bbox, the
  volume within 0.015 mm3 of float noise), and the cheeks end there.
- EndFaceParams.m3_rows: DEFAULT drops the NEMA 17 pattern's upper M3 pair
  (nothing uses them; they would run through the pocket). The bracket's 4
  M4 through the block become about M4 x 25 (open_issues row).
- WRIST_PITCH_LIMIT_DEG 120 -> WRIST_PITCH_LIMITS_DEG (-105, +70): the
  wrist body's back corners meet j2_link's web at -109 / +74.5 at any roll,
  today's arm as well; 4 deg of margin. tests/test_sweeps.py checks exact
  distances at both limits at roll 0 / 90 / 180 / 270. open_issues rows
  for this and for the shoulder's upper limit (previous commit).

Numbers:
- reach, stretched out (URDF forward kinematics): fingertips 646 -> 547 mm,
  wrist centre 420 -> 341 mm (this commit: fingertips 567 -> 547)
- wrist_link 113,542 -> 72,321 mm3 (144.2 -> 91.8 g solid PETG)
- wrist_pitch_link 0.469349 -> 0.416999 kg, COM x 0.057 -> 0.044801 m;
  URDF total 5.681 -> 5.629 kg
- URDF/SDF: wrist_roll x 0.109643 -> 0.089643; wrist_pitch limits
  +/-2.094395 -> -1.832596 / +1.22173
- arm: volume 2,766,520 -> 2,725,300 mm3, bbox 584.8 x 217.1 x 620.5 ->
  567.5 x 217.1 x 610.5 mm; leaves / solids unchanged (82 / 235)

Checks: hash gate - wrist_link, arm, wrist_pitch_link changed; wrist_roll
and the jaw links only moved with their frames (inspect diff: same
geometry, 1e-6); mount_placements.py: placements.json unchanged; derive
--check OK after copying the drafts; wrist_pitch_link mesh re-exported;
URDF / SRDF --strict and SDF validate; full suite 846 passed; the part and
the arm looked at.

File: cad/robot/arm.urdf (robot description, URDF)
Before this commit: robot arm, 10 links, 9 joints
Links:
- link wrist_pitch_link: mass 0.469349 -> 0.416999
Joints:
- joint wrist_pitch: limit lower=-2.094395 upper=2.094395 effort=5 velocity=1 -> lower=-1.832596 upper=1.22173 effort=5 velocity=1
- joint wrist_roll: origin xyz=0.109643 0.000005 -0.016998 rpy=-1.570799 -0.055534 -1.570796 -> xyz=0.089643 0.000005 -0.016998 rpy=-1.570799 -0.055534 -1.570796

Commit message: cad: the base_yaw 90T placed under j1_coupler, clamped by 4x M4 x 45 + nuts
Why: the base_yaw joint was not held down. j1_coupler stood on the thrust
bearing with nothing pulling it onto it, the lower base 6806 held nothing, and
the joint's driven pulley was not in the model. The coupler's stub was already
drilled for it (lib/yaw_coupler/params.py DEFAULT).

The pulley: gt2_pulley_90t#5, a mount hosted on j1_coupler#1 (lib/mounts.py
PULLEY_MOUNTS), hub up: frame ((0, -22.507252, 0), (180, 45, 0)) in the
coupler's frame = stub_y0 + the hub's end, turned HubParams.hole_deg onto the
stub's diagonal holes; world y -27.6. Its hub end lies on the stub's end in the
plane of the lip's lower face, its journal in the lower 6806, its ring under
that bearing's inner ring. It rides in shoulder_link. No existing part's
geometry changed: the hash gate names only arm.step and shoulder_link.step.
Fit: 0 interference with every neighbour, 3.72 mm from the base; its mid-plane
19.8 mm along the 48 mm motor's 22 mm shaft.

The bolts: two new purchased pattern parts in parts/base/.
- yaw_pulley_screws: 4x M4 x 45 (HubParams.pulley_screw_len), heads on the
  pulley's outer face, 5.8 mm from the base; 2815.345 mm^3, 22.1 g
  (YAW_PULLEY_SCREWS_MASS_G). The M4 x 40 the open-issues row planned ends
  1.29 mm past the nut, under the two pitches the other joints' bolts are
  tested to; x 45 ends 6.29 past it, 22.0 mm from the drive's housing.
- yaw_pulley_nuts: 4x M4, their bearing faces 35.507252 from the heads' - flush
  in the floor of the pocket over the hub -, a corner at hole_deg - 90 from the
  pattern's +X (the coupler's Z); 382.322 mm^3, 3.0 g. In the pockets with
  exactly the designed press, 23.03 mm^3.

A new part state for them, envelope COTS (lib/reference.py ENVELOPE_COTS): a
purchased part with no vendor model and no export keeps NO reference file and
no manifest entry; its own test holds its numbers (pieces, volume, bbox) and
feature probes - tests/base/test_yaw_pulley_bolts.py. It replaces, for new
parts, a golden STEP under reference/native/ (NATIVE_COTS stays as it is).
tests/test_parts_convention.py checks the state; test_robot.py's link-mass
check follows parts.bought() instead of the COTS registry.

Tests: test_mounts.py takes base_yaw into STACKS (the coupler + the 90T; no
shoulder there, NO_SHOULDER: the thrust stack sets the height) and
PULLEY_BOLTS, and the base motor's shaft into the belt-plane check;
test_bearing_stacks now also holds each 90T's ring on the inner ring.

Numbers that changed:
- placements.json expected: leaf_occurrences 55 -> 58, solids 133 -> 142,
  solid_volume 2007146.747 -> 2034876.117; 3 mounted records added (27 parts
  + 1 module mounted).
- the arm: leaves 82 -> 85, solids 235 -> 244, bought / printed leaves
  47 / 35 -> 49 / 36.
- the lists: printed 28 parts, 35 -> 36 to print (a third 90T); bought
  29 parts / 47 occurrences -> 31 / 49.
- shoulder_link: mass 1.594247 -> 1.650504 kg, COM (-0.000858, 0.015952,
  -0.013965) -> (-0.000828, 0.015409, -0.01717), ixx 3.674871e-03 ->
  4.185559e-03, iyy 3.263627e-03 -> 3.760526e-03, izz 2.686198e-03 ->
  2.713967e-03, ixy 2.317943e-05 -> 2.392286e-05, ixz 1.803046e-05 ->
  2.241258e-05, iyz -3.530535e-04 -> -4.345619e-04 (arm.urdf, arm.sdf); its
  mesh re-exported (78 solids, 746996.4 mm^3). The robot: 5.629 -> 5.685 kg.

docs/open_issues.md: the row "the base_yaw joint is not held down" is closed.
A row is added in its place: the joint is now set axially twice (the thrust
stack and the 90T's ring under the lower 6806), line-to-line in the model - a
shim between the hub end and the stub's end on assembly. The "not modelled"
row keeps the motor's 20T and the belt; the nut-pocket fit row takes
j1_coupler's pockets.

File: cad/robot/arm.urdf (robot description, URDF)
Before this commit: robot arm, 10 links, 9 joints
Links:
- link shoulder_link: mass 1.594247 -> 1.650504

Commit message: cad: j2_link's roll wall a round flange on a necked web, braced by two gussets
The wall j2_link bolts onto the roll shaft with was a bare 90 x 70 x 8 mm rectangle: full width and z -10..60,
sized under / over the link caps' tray and lid, which were removed on 2026-09-25. Its skirt hung 1.5 mm below
j1_link's top face, and that lower edge is what met the upper arm's side at +/-92 degrees of elbow.

Now (lib/forearm/link.py roll_wall, necked_web, wall_gussets; RollEndParams):
- the wall is a Ø60 round flange about the roll axis (wall_od, over the stop lug and post that turn in front of it,
  r 28 / 30) on a foot as wide as itself: the hull of the circle and the web's end section, z -5..55;
- the web necks down to that 60 mm foot (neck_half_w 30) from the wrist boss, its sides tangent to the boss
  (layout.neck_tangent, web_half_width) - the wrist motor's footprint stays on it over its whole slide;
- two 6 mm gussets on the web's top face against the wall's wrist face (rib_y 24..30, rib_len 30, rib_h 20, their
  tops cut by the round outline), either side of the wrist motor: 3.0 mm off its body over the whole slide.
The recess, the cable bore, the Ø32 bolt circle and the wall's station (48 mm from the elbow axis) are unchanged.
RollEndParams.wall_z and lib/params.py FOREARM_WALL_Z are replaced by wall_od / FOREARM_WALL_OD.

Measured:
- j2_link: 215465 -> 173542 mm^3 (273.6 -> 220.4 g at PETG_DENSITY); z -10..60 -> -5..55.
- The wall's farthest point from the roll axis: r 57 -> 30 (the web's corner at the wall: r 34.5).
- forearm_link inertial: mass 0.761574 -> 0.708332 kg, COM (0.003934, -0.000011, 0.098002) ->
  (0.004589, -0.000012, 0.100201), ixx 2.600065e-03 -> 2.441454e-03, iyy 2.534882e-03 -> 2.420877e-03,
  izz 4.808943e-04 -> 3.847050e-04 (arm.urdf and arm.sdf from derive.py's drafts); URDF total 5.629 -> 5.576 kg.
- The forearm, rolled anywhere (every 5 degrees), now stays 2 mm off j1_link to about +/-102 degrees of elbow (was
  +/-90); at 90 degrees the least gap is 3.36 mm. The wrist motor and its board stay 23 mm off there.
  ELBOW_PITCH_LIMIT_DEG stays 90: SHOULDER_PITCH_LIMITS_DEG was swept over that range, so opening it is a new
  docs/open_issues.md row.

Tests: tests/forearm/test_roll_end.py gains test_the_neck_the_round_wall_and_its_gussets (the neck tangent to the
boss, the wall over the recess and the stops, the gussets outside the motor and its board) and probes of the round
outline, the neck's side and the gussets; its wrist-end comparison with the SolidWorks part now probes only beyond
the wrist pivot (the web between the pivot and the wall is narrower by design).

Recipe C: arm rebuilt, hash gate on the same machine: only j2_link.step, arm.step and forearm_link.step changed.
robot/meshes/forearm_link.stl re-exported; derive.py --check OK; validate URDF / SRDF --strict and SDF OK.
./cadtool pytest 848 passed (fast lane 544); lint clean.

File: cad/robot/arm.urdf (robot description, URDF)
Before this commit: robot arm, 10 links, 9 joints
Links:
- link forearm_link: mass 0.761574 -> 0.708332

Commit message: cad: base_yaw at 6:1 - a 120T driven pulley in place of the 90T
Why: a higher base_yaw ratio than the 4.5:1 of the shared 90T (2.0 -> 2.7 Nm at
the joint from the 0.45 Nm motor, a stiffer hold, finer steps), chosen from a
to-scale preview. The 90T sat Ø59 in the base's Ø97 cavity; 120 teeth is the
largest that still passes through the opening in the base's plate with room
to spare.

The pulley: gt2_pulley_120t (parts/base/), lib/pulley/params.py YAW =
DEFAULT with GT2_PULLEY_120T_TEETH and its rim's inside grown with the teeth
(rim_dia 53 -> 72.098593, the 90T's 3.788 wall under them kept); the hub, the
web's height, the bore and the M4 holes are the 90T's, so it takes the same
mount frame on j1_coupler (gt2_pulley_120t#1 replaces gt2_pulley_90t#5) and
the same M4 x 45 screws and nuts. Flange Ø59.188 -> Ø78.286; volume
37623.954 mm^3, 47.8 g (the 90T: 31.2 g). Fit: 0 interference with every
neighbour; 9.2 mm to the base's wall (was 18.7), 3.2 inside the plate
opening's radius, 3.72 from the base at the bearing boss (unchanged), 25.6 mm
to the motor (was 32.8). The elbow's and the wrist's 90T are unchanged.
BASE_YAW_RATIO = GT2_PULLEY_120T_TEETH / GT2_PULLEY_20T_TEETH = 6 in
lib/params.py; robot/AGENTS.md names it as the base_yaw reduction.

The motor: where the stock belt round 120T / 20T puts it - YAW_BELT
280 -> 320, BASE_MOTOR_PATTERN_CENTRE x 81.972 -> 83.967 (the motor and its
board move 1.995 out). The motor mount grows with it: its far end 117.472 ->
119.467, volume 56295.1 -> 57246.1 mm^3; its native reference re-accepted
(import_native.py --only base_motor_mount --force). The base is unchanged.

One registry for parts designed here that keep no reference file:
lib/reference.py NO_REFERENCE (the ENVELOPE_COTS of the previous commit, now
for printed parts too): gt2_pulley_120t (REFERENCE = None, its numbers in
tests/pulley/test_gt2_pulley_120t.py) and the base_yaw pulley bolts.
tests/test_parts_convention.py checks the state for both kinds; tools/bom.py
lists such a printed part as "no reference". parts/AGENTS.md makes it the
state for every new part designed here (the existing NATIVE parts keep their
accepted builds).

Numbers that changed:
- placements.json expected: solid_volume 2034876.117 -> 2048919.285 (58 part
  records, 142 solids, unchanged).
- print list: 28 -> 29 parts (36 to print, unchanged).
- base_link: mass 0.93574 -> 0.936947 kg, COM (-0.044986, 0.000021,
  0.056664) -> (-0.046028, 0.000021, 0.056669), ixx 1.515585e-03 ->
  1.516875e-03, iyy 2.940607e-03 -> 3.015555e-03, izz 2.693847e-03 ->
  2.768958e-03, ixy 2.801067e-06 -> 2.865620e-06, ixz -6.562157e-04 ->
  -6.700869e-04, iyz 1.172646e-06 -> 1.172743e-06; mesh re-exported
  (34 solids, 390735.8 mm^3).
- shoulder_link: mass 1.650504 -> 1.667132 kg, COM (-0.000828, 0.015409,
  -0.01717) -> (-0.00082, 0.015255, -0.01817), ixx 4.185559e-03 ->
  4.365000e-03, iyy 3.760526e-03 -> 3.936070e-03, izz 2.713967e-03 ->
  2.737501e-03, ixy 2.392286e-05 -> 2.413298e-05, ixz 2.241258e-05 ->
  2.378057e-05, iyz -4.345619e-04 -> -4.600069e-04; mesh re-exported
  (78 solids, 760088.7 mm^3).
- the robot: 5.685 -> 5.703 kg.

The hash gate names base_motor_mount.step, arm.step, base_link.step and
shoulder_link.step (+ the new gt2_pulley_120t.step).

File: cad/robot/arm.urdf (robot description, URDF)
Before this commit: robot arm, 10 links, 9 joints
Links:
- link base_link: mass 0.93574 -> 0.936947
- link shoulder_link: mass 1.650504 -> 1.667132
