Commit message: cad: the forearm wall screws into nuts in the roll shaft; a channel under the web for the bottom one
The wall's 4x M3 self-tapped into the shaft's end, and the joint could not be assembled as drawn:
- the bottom screw's hole (y 0, z 9) opened on the wall's wrist face right where the web butts onto it (web z 8..19,
  the hole z 7.3..10.7): no way in for the screw and no seat for its head - only 0.7 mm of the hole was open;
- the M3 x 20 on the buy list was 6 mm too long: 6 mm of wall at the holes (8 less the recess) + 8 mm tap holes = 14;
- a self-tapped thread in PETG creeps and strips on re-assembly, and this joint comes apart to take the forearm off.

Now:
- 4x M3 x 25 (ISO 4762, lib/fasteners.py M3_SHCS; RollEndParams.screw / screw_len) from the wall's wrist face through
  the wall and the shaft's end into M3 nuts buried in the Ø44 core behind bearing 2 (RollDriveParams.end_nut, stations
  z_end_tip 31, z_end_nut 32..34.4): head and nut clamp 21.6 mm of PETG - the spigot, the neck and journal 2 - instead
  of hanging the load on a thread in the end layers.
- Each nut sits in a slot from the cable bore outward along its screw's angle (layout.end_nut_pocket: the nut's 5.5
  across flats wide, end_nut_fit 0.2 past its corner and over it), pushed in from the bore before the wall goes on;
  3.3 mm of the core outside it, 1.6 mm before journal 2.
- Bolt circle Ø32 -> Ø31: the Ø3.4 clearance holes sit centred in the neck's wall, 1.8 mm either side (at Ø32 they
  would leave 1.3 outside; the old Ø2.5 taps left 1.75 / 2.75).
- The bottom screw's head gets a channel in the web's underside (layout.screws_under_the_web / screw_channel,
  RollEndParams.channel_clear): 6.5 wide, z 8..12.75, from the wall into the central motor slot (x -88..-56); the web
  keeps 6.25 mm over it. The screw lays in from the belt side, a key reaches it through the channel.
The screws and nuts stay tools/bom.py EXTRAS rows (M3 x 20 -> M3 x 25, + 4x M3 nut). A screw with its head is 28 mm,
the wrist motor's body 22.6 mm from the wall: docs/forearm_roll.md §4 now bolts the wall on before that motor.

Measured:
- forearm_roll_shaft: 95222.909 -> 94377.799 mm^3 (forearm_roll_drive EXPECTED: rotor and whole module
  421502.356 -> 420657.246); its native reference re-accepted (import_native.py --only forearm_roll_shaft --force).
- j2_link: 173542.2 -> 172893.5 mm^3 (220.4 -> 219.6 g).
- forearm_link inertial: mass 0.708332 -> 0.706435 kg, COM (0.004589, -0.000012, 0.100201) ->
  (0.004618, -0.000012, 0.100337), ixx 2.441454e-03 -> 2.435994e-03, iyy 2.420877e-03 -> 2.415092e-03,
  izz 3.847050e-04 -> 3.841204e-04, ixz 8.800633e-05 -> 8.885513e-05, iyz 6.559725e-08 -> 6.462437e-08,
  ixy 2.488887e-07 -> 2.486815e-07; URDF total 5.576 -> 5.574 kg.

Tests: test_roll_end.py test_the_wall_screws_way_in (only the bottom head lands in the web; its channel opens below,
runs into the slot, leaves 5 mm of web) and, on the part, every head's room behind the wall probed open - the check
that would have caught the blocked hole; test_roll_drive.py holds the holes centred in the neck, the screw's stations,
the nut behind bearing 2 and clear of the ring, and probes each hole, seat and pocket. tests/test_bom.py's check that
the motor mount's countersunk screws / nuts are not EXTRAS now names the mount (the wall's nuts are a new EXTRAS row).
docs/open_issues.md: the spigot row is rewritten for the nuts; a row for the pockets' fit (line-to-line, unmodelled
nuts: print a fit gauge).

Recipe C: hash gate against the first commit's builds: only forearm_roll_shaft, j2_link, forearm_roll_drive, arm and
forearm_link changed. forearm_link mesh re-exported; derive.py --check OK; validate URDF / SRDF --strict and SDF OK.
./cadtool pytest 849 passed (fast lane 545); lint clean.

File: cad/robot/arm.urdf (robot description, URDF)
Before this commit: robot arm, 10 links, 9 joints
Links:
- link forearm_link: mass 0.708332 -> 0.706435

Commit message: cad: the shoulder drive's shell turns - a 6814 at each end, 57 apart, the yoke a fork round it
The shoulder_pitch cycloidal drive carried the whole upper arm on two 6814s pressed side by side in one
seat, centres 10 mm apart: their play and the PETG's give tipped the arm. The drive now holds its carrier
(the output hub and its pins) and its motor, and turns its housing shell as the output, on one 6814 at each
end of the gear stack - the hub's in the seat's outer slot, the other on a sleeve behind the motor plate,
over the front of the motor (its 70 mm bore clears the motor and the MKS board, 61 across the corners).

Drive (lib/cycloidal/params.py ShellParams, DEFAULT_CONFIG only; LEGACY_CONFIG builds the port unchanged, and
tests/cycloidal/test_port.py still matches every port build to its CadQuery export):
- ratio 20:1 -> 21:1 (DriveConfig.ratio: the ring pins, the carrier held; GearParams.gear_ratio removed); the
  output now turns the same way as the motor. Theoretical output 9.0 -> 9.45 N.m (0.45 N.m motor).
- 6814 centres 10 -> 57 mm (z 37 / 47 -> 47 / -10).
- cycloidal_motor_plate is the carrier's motor end: a Ø90 plate inside the shell, its face relieved over the
  turning outer race, and a sleeve back over the motor (bore 62, od 70, the 6814 pressed on its last 10 at
  70.3); 83649.806 -> 93978.074 mm^3, Ø90 x 57.
- new cycloidal_shell_ring (no reference, tests/cycloidal/test_shell_ring.py): the port plate's housing half -
  the ring-pin ends, the bolt counterbores - plus a skirt round the motor-end 6814 with a lip; 45127.781 mm^3.
- ring gear body: end wall 3 -> 8 (housing depth 60 -> 65, body 51 -> 56) so j1_link keeps its pose; no nut
  pockets; 105056.631 -> 126498.988 mm^3.
- output hub: held, 28 -> 42.272 tall (proud 5 -> 14.272: through j1_link to the yoke), a Ø76 shoulder that
  stops the hub-end 6814; its arm-mount pattern now bolts it to the yoke (M4 x 45, EXTRAS);
  96871.427 -> 143422.642 mm^3. It gets a REFERENCE_BUILD (its port build).
- housing bolts M4 x 55 -> M4 x 70 (39.8 -> 48.7 g), through the shell into nuts sunk 6.97 in j1_link
  (nuts z 56 -> 71.3); 5070.531 -> 6201.504 mm^3.
- the stator / rotor split swaps: rotor = ring gear body, shell ring, ring pins, housing bolts + nuts, both
  6814s; stator = motor plate, hub, output pins, 625, motor + board, gear train.
- EXPECTED: leaves 19 -> 20, solids 73 -> 74, volume 582937.149 -> 707517.743; stator 16 / 67 / 482928.722
  -> 13 / 37 / 469372.949, rotor 3 / 6 / 100008.427 -> 7 / 37 / 238144.795; bbox Z 127.1 -> 141.372;
  printed leaves 6 -> 7.
- lib/params.py: CYCLOIDAL_RATIO 21, STACK_DEPTH 65, HUB_PROUD 14.272, OUTPUT_FACE_Z 65 (the shell's face),
  new HUB_FACE_Z 79.272 and SHELL_BOLT_CIRCLE / _COUNT (117, 6); CYCLOIDAL_ARM_MOUNT_* renamed HUB_BOLT_*.

Yoke (lib/yaw_coupler ForkParams, DEFAULT): the cheek, middle body, cradle and pillar sockets go; a fork on the
drive's own axis (the placement's, 0.21 off the old cradle's) holds an end plate the hub bolts to, past j1_link,
and a clamp round the sleeve split at the axis - the saddle on a windowed post, the cap a new part,
j1_coupler_cap (no reference, 72706.126 mm^3, 4 M4 x 25 + nuts in side slots: EXTRAS). The ring drops 2
(RING_DROP: the turning pillars 0.68 -> 2.68 above it); the disc is cut back where j1_link swings.
j1_coupler 233294.911 -> 338641.472 mm^3. This closes the open issue "the drive is not fastened to
j1_coupler".

Upper arm (lib/upper_arm ShellMountParams, DEFAULT): j1_link bolts to the shell's output face with the 6
housing bolts on Ø117 (the hub's 4 on Ø50), a round root r 66 round a Ø74.4 hole for the held hub. The elbow
motor leaves the shoulder axis (the fork holds it now): its pad moves to x 88.028, ELBOW_MOTOR_CENTRES = 81.97
from the elbow, the centre distance of a stock 280-2GT belt (ELBOW_BELT_LENGTH, EXTRAS) straight from its 20T
to the 90T; the second-stage seat goes (BearingParams None; gt2_pulley_20_60t stays unplaced).
j1_link 299935.717 -> 308908.639 mm^3.

Checked: the shoulder's whole range (-120..75, every 15 deg) keeps the upper arm - j1_link, its motor, the
shell - its 1.0 mm running gap off the fork's end plate (new test_sweeps case; the old yoke's disc came 0.2 off
j1_link at +75, the swing cut removes it); the elbow motor stays >= 18 mm off the forearm roll drive over the
elbow's +/-90 (tests/forearm/test_roll_drive.py now sweeps it instead of a radial bound). Limits unchanged.

Robot: shoulder_link 1.667132 -> 1.639152 kg, upper_arm_link 0.893701 -> 1.324862 kg (COM, inertia
re-derived, URDF + SDF); arm 5.648 -> 6.051 kg; meshes re-exported (shoulder_link 49 solids, 924585.6 mm^3;
upper_arm_link 55 solids, 636782.2 mm^3). placements.json: j1_coupler_cap#1 added, nema17_40mm#2 /
mks_servo42d#2 moved; expected leaves 58 -> 59, solids 142 -> 143, volume 2048919.285 -> 2121625.411. Arm
locks: leaves 85 -> 87, solids 244 -> 246, printed leaves 36 -> 38; BOM printed 29 / 36 -> 31 / 38.

Docs: docs/cycloidal_drive.md (new §5.5 the turning shell, §2-5, §7, §12), open_issues.md (the fits of the
sleeve, the skirt and the clamp; the fork's first-pass stiffness; the elbow drive one stage, its belt plane
2.7 off the motor's face), robot/AGENTS.md, the URDF ledger, software/control/README.md's ratio.

File: cad/robot/arm.urdf (robot description, URDF)
Before this commit: robot arm, 10 links, 9 joints
Links:
- link shoulder_link: mass 1.667132 -> 1.639152
- link upper_arm_link: mass 0.893701 -> 1.324862

Commit message: cad: the upper arm rises off the turning shell's middle; the shell the same at both ends, the yoke two thin legs
Round 1 kept j1_link as a plate bolted to the turning shell's hub end, the hub reaching through it to a yoke end plate
and the motor sleeve held in a 30 mm clamp block, the ring gear body carrying an empty second-bearing slot. Asked for:
the shell part of the upper arm link, the empty slot gone, the pillars end to end, the drive symmetrical, the yoke's
grip equally thin on both sides, and the arm going straight up from where the discs are (PAROL6-like), not from the
side of the gearbox - the end effector need not stay centred.

The drive (lib/cycloidal/params.py ShellParams, layout.py, housing.py):
- the two ends mirror each other about the middle of the discs (z 24): from the outside in an end_lip (3), a 6814, a
  plate_dia plate in a ring_bore_dia pin ring (the motor plate; at the hub end a new 9 mm flange on the hub, its face
  relieved over the outer race), then the 4 mm clearance to its disc. StackUp: output_clearance 2 -> 13 (the clearance
  + the flange), output_bearing_total 20 -> 10, output_wall 8 -> 3. New helpers hub_flange, shell_ends, arm_zone,
  sleeve_end.
- the shell z -12..65 -> -13..61 (74 long); the 6814s z 47 / -10 -> 48 / -10, centres 57 -> 58 apart.
- the body round the discs (build_shell_body, z 9..61: bore, pin ring, seat, lip, bolt holes, the housing nuts' hex
  pockets) is printed as one with j1_link; cycloidal_ring_gear_body leaves the drive - its model builds the port
  (LEGACY_CONFIG) for test_port and declares UNPLACED.
- cycloidal_shell_ring -12..9 -> -13..9 at full shell diameter (lip, seat, pin ring, blind ring-pin holes; the skirt,
  skirt_od / skirt_lip, gone): volume 45127.781 -> 75740.748 mm^3.
- the hub 42.27 -> 23 tall (z 37 -> 39, its face 79.27 -> 62 on the yoke's leg): the Ø90 x 9 flange replaces the
  Ø76 shoulder (hub_shoulder_dia gone), pin holes 19 -> 18 deep, its 4 captive nuts hub_nut_depth 4.7 deep.
- the motor plate's sleeve ends at the motor leg's outer face, z -48 -> -22: volume 93978.074 -> 72414.182 mm^3.
- ring pins 4 x 35 -> 4 x 40 (z 5.5 -> 4, 5 into each pin ring), output pins z 11 -> 12, housing bolts M4 x 70 ->
  M4 x 65 end to end (heads z 0.5 -> -12.5, nuts 71.3 -> 53.3 in the body); masses 72.5 -> 82.9 g, 48.7 -> 45.7 g.
- the discs, shaft, support pin, motor and the motor plate's plate do not move (the datum z 0 stays the NEMA face).
- assemblies/cycloidal_drive.py: the ring gear body row and its ROTOR entry go; EXPECTED leaves 20 -> 19, solids
  74 -> 73, volume 707517.743 -> 551156.383; stator 13 / 37 / 469372.949 -> 13 / 37 / 407955.132; rotor
  7 / 37 / 238144.795 -> 6 / 36 / 143201.251; the module's z -62.1 .. 79.27 -> -62.1 .. 62.

The upper arm (lib/upper_arm/, ShellMountParams -> ArmParams):
- j1_link is the shell's body plus an arm: the plate's outline seen along Y (stadium + root_r 66 collar) over the
  drive's arm_zone (z 9..39 -> the link's y 27.5..57.5), fused into the shell's wall from fuse_r 61 (past the housing
  bolts' holes), stopping at the elbow's relief, its motor-side top cut back within swing_r 96 of the elbow axis from
  swing_above_top 9.5 over the slid plate's top - where the forearm roll drive's motor mount, motor and board swing
  with the elbow (the first build touched the board at the rest pose, 27.6 mm^3).
- the plate's elbow end and the elbow motor's pad slide along +Y onto the arm's outer face: arm_slide 39.271993
  (lib/params.py J1_ARM_SLIDE; J1_MOTOR_PAD_FACE_Y -32.5 -> 6.771993). The drive's frame in the link (drive_frame:
  drive_z_at_y0 66.5, drive_x_deg -47.584167) matches the capture to 1e-6.
- j1_link volume 308908.639 -> 378596.739 mm^3 (the shell's body included).
- lib/placements.py LinkShift gains across_w / across_y: everything beyond the elbow moves arm_slide along j1_link's
  +Y (N); lib/mounts.py adds it to the mounts hosted on j1_link#1 (the elbow motor, the elbow 6806s);
  mount_placements.py re-run. The end effector is now off the base_yaw axis (accepted; docs/open_issues.md).

The yoke (lib/yaw_coupler/):
- two alike 8 mm legs (ShellParams.yoke_leg), each end_plate_gap 1 off an end of the shell, mirror images about the
  middle of the discs: the hub leg at the hub's face (z 62..70, was the end plate at 79.27..87.27), the motor leg
  round the sleeve (z -22..-14, was the 30 mm clamp block at -44..-14 on a post and foot), split at the axis. The
  disc's swing cut stays.
- j1_coupler_cap: the motor leg's upper half on 2 x M3 x 25 into M3 nuts in the leg's side slots (was 4 x M4 x 25):
  volume 72706.126 -> 9182.805 mm^3. The hub's screws M4 x 45 -> M4 x 25, ends flush with its nuts.
- ForkParams: plate_t, clamp_z, clamp_half, post_wall, foot_*, cap_bolt_inset gone; cap_bolt_r 40, cap_seat 12,
  cap_nut_y 10.1 new; fork_plate_x / fork_clamp_x -> fork_hub_leg_x / fork_motor_leg_x.

Constants (lib/params.py): CYCLOIDAL_STACK_DEPTH 65 -> 61, CYCLOIDAL_HUB_PROUD 14.27 -> 1, CYCLOIDAL_HUB_FACE_Z
79.27 -> 62; CYCLOIDAL_SHELL_ENDS_Z (-13, 61), CYCLOIDAL_ARM_ZONE_Z (9, 39), CYCLOIDAL_SLEEVE_END_Z -22 new;
CYCLOIDAL_OUTPUT_FACE_Z gone. SHOULDER_PITCH_LIMITS_DEG upper 75 -> 67: the arm, now in the yoke's middle, reaches
j1_coupler's disc at 70.5 deg (the 1 mm running gap held to 69.5); pitched back it clears to -150.

Robot: the elbow_pitch origin z 0.009999 -> 0.049271 (the slide); shoulder_link 1.639152 -> 1.327614 kg, upper_arm_link
1.324862 -> 1.298990 kg (the body moves from the drive's rotor into j1_link); the shoulder limit 1.308997 -> 1.169371
rad; shoulder_link / upper_arm_link meshes re-exported. Arm: 87 -> 86 leaves, 246 -> 245 solids, printed leaves
38 -> 37; print list 31 parts / 38 pieces -> 30 / 37. tools/bom.py EXTRAS: the hub's M4 x 25s, the cap's M3 x 25s +
M3 nuts.

Tests: test_ring_gear_body.py becomes test_shell_body.py (the stack symmetric about the middle of the discs, the
body's numbers and probes); test_shell_ring, test_housing, test_motor_plate, test_output_hub, test_assembly
(cycloidal), test_j1_link (the arm, the drive's frame, the slide), test_j1_coupler (the legs, the cap),
test_placements (across_y), test_params_invariants, test_bom, test_assembly re-locked. Docs: cycloidal_drive.md
§1-5, §5.5, §10, §12; open_issues.md (the fits, the legs, the arm's first pass, the end effector off the axis, the
shoulder limit); robot/AGENTS.md (the stator / rotor rows were the port's), lib/ tests/ assemblies/ AGENTS.md.

Checks: ./cadtool lint; ./cadtool pytest (full, slow lane included); derive.py --check (urdf, sdf OK); validate urdf
--strict, srdf --strict, sdf; the hash gate (only the drive's parts, j1_link, j1_coupler + cap, the two assemblies and
the two link STEPs changed); a part-by-part overlap check of the whole arm (only the fits the branch already had);
snapshots of the arm, the drive and the URDF looked at.

File: cad/robot/arm.urdf (robot description, URDF)
Before this commit: robot arm, 10 links, 9 joints
Links:
- link shoulder_link: mass 1.639152 -> 1.327614
- link upper_arm_link: mass 1.324862 -> 1.29899
Joints:
- joint elbow_pitch: origin xyz=0.170003 0 0.009999 rpy=0 0 0.010227 -> xyz=0.170004 0 0.049271 rpy=0 0 0.010227
- joint shoulder_pitch: limit lower=-2.094395 upper=1.308997 effort=5 velocity=1 -> lower=-2.094395 upper=1.169371 effort=5 velocity=1

Commit message: cad: the upper arm a plain bar off two filled windows of the turning shell; the elbow motor on the arm's other side
Round 3 wrapped the turning shell in an r 66 collar where the upper arm joined it, closing all six windows over the
discs. Asked for: fill in two of the windows and run the arm out of them, the others open so the discs show; keep the
arm a simple rectangle as a placeholder (the arm only - the elbow end, its bearing seat and the motor stay - 90 wide);
and flip the elbow motor to the arm's other side, the drive motor's and the forearm's (+N). On that side the forearm
roll drive's motor and board swing onto it when the elbow lifts the forearm back: the elbow's lower limit -90 -> -21
was accepted.

The shell (lib/cycloidal/params.py, housing.py):
- HousingParams.bolt_start_deg (new, 0 for the port): DEFAULT's 6 pillars / housing bolts start at ARM_DEG 47.584167
  (the upper arm's centreline in the drive's frame, ArmParams.drive_x_deg turned round; a literal, checked against
  j1_link's frame by tests/upper_arm/test_j1_link.py), so one pillar sits under the arm. compute_housing_bolt_angles adds
  it; the shell ring, the body, the housing bolts and nuts turn with it (their volumes unchanged: ring 75740.748, bolts
  5824.513, nuts 814.757 mm^3). LEGACY (the port, test_port) unchanged.
- ShellParams.arm_windows = 2 (new): build_shell_body takes arm_root - the sector over the two windows either side of
  the first pillar, edges through the middle of the pillars that bound them - out of the window cutter, so those two
  are solid over the body's length (z 9..61), the arm's root; the other four open on the discs and the ring pins (the
  shell ring keeps all six). Body 99536.499 -> 152304.812 mm^3.
- the drive module's box 129.2 x 116.023 x 124.1 -> 127.775 x 125.532 x 124.1 (the turned pillars); EXPECTED leaves /
  solids / volume unchanged (19 / 73 / 551156.383).

The upper arm (lib/upper_arm/, ArmParams):
- _arm is a plain bar: the plate's width (2 SlabParams.r, 90), y_outer .. y_inner (30), from the shoulder axis to the
  elbow axis, cut back inside fuse_r (61) and by the elbow's relief as before; its motor-side top stepped down flat from
  swing_r (96) short of the elbow axis, swing_above_top (9.5) over the slid plate's top - replacing the arc. The r 66
  collar goes (ArmParams.root_r removed).
- the elbow motor turned over onto the arm's +N side at the same place along it (PadParams.x): down a square hole
  through the bar (motor_hole_half 21.6) onto a 6 mm plate under the arm's outer face (motor_plate_t 6,
  motor_plate_half 26, motor_pilot_dia 22.5, its 4 holes PadParams.holes), its face at y_outer; its 22 mm shaft back
  through the plate to y 5.5, past the elbow 90T's toothed rim (y 2.87 .. 12.27), so the 20T now reaches the belt's
  plane (the pad's face was 2.7 short of it). The pad's tube is LEGACY's only.
- j1_link 378596.739 -> 376985.495 mm^3.

Mounts and limits:
- lib/params.py J1_MOTOR_PAD_FACE_Y 6.771993 -> 27.5 (ArmParams.y_outer); lib/mounts.py nema17_40mm#2's frame
  (-90, 0, 90) -> (90, 0, 0): body +N, shaft -N, spun so its plug points -Z (toward the elbow the roll block would pass
  it 0.17 mm off at +40 deg); mount_placements.py re-run (nema17_40mm#2, mks_servo42d#2, and the cap's stale note).
- ELBOW_PITCH_LIMIT_DEG 90 -> ELBOW_PITCH_LIMITS_DEG (-21, 90): lifting the forearm back, the roll drive's MKS board
  comes within 1 mm of the elbow motor at -24.4 deg (3.62 mm at -21; 3 deg short, as the shoulder's limits are set);
  bending down in front, everything past the elbow stays >= 5 mm off it to +90. robot/frames.py takes the pair.
- the whole arm along the shoulder axis 175.4 -> 146.9 mm (the motor and board stand 23.6 out of the arm's +N face,
  were 74.3 out of its -N face); the shoulder's sweep keeps the flipped motor + board >= 5 mm off the fork and the base
  over -150..80; the bar's front contact (70.5 deg) unchanged, SHOULDER_PITCH_LIMITS_DEG (-120, 67) stand.

Robot: upper_arm_link mass 1.298990 -> 1.296943 kg, COM (0.056594, 0.000006, 0.025075) -> (0.058957, 0.000068,
0.040525), ixx / iyy / izz 2.317521e-03 / 7.141428e-03 / 7.063853e-03 -> 1.600035e-03 / 6.133599e-03 / 6.633113e-03,
ixz 1.001679e-03 -> 3.296841e-04; the elbow's lower limit -1.570796 -> -0.366519 rad (URDF + SDF); upper_arm_link mesh
re-exported.

Tests: test_shell_body (the two windows under the arm solid end to end, the four others open, the root's and the open
zone's section areas, the volume), test_housing / test_shell_ring / test_purchased (probes and boxes taken about the
first pillar), cycloidal test_assembly (the box), test_j1_link (the volume and box, the bar, the windows, the step, the
motor's hole and plate, the pillar on the arm's centreline, the motor's frame), test_params_invariants, test_roll_drive
(the elbow motor >= 1 mm off the roll drive over the elbow's range, the limits as a pair, the upper arm turned the
joint's way), test_sweeps (the asymmetric elbow range), test_j1_coupler (the collar's clearance gone). Docs:
cycloidal_drive.md (§5.2 the pattern's start and the root, §5.5, §12), open_issues.md (the arm a placeholder, the
elbow's limit, the 20T now reaching the belt), forearm_roll.md, robot/ lib/ tests/ AGENTS.md, tools/bom.py's elbow
belt note; a stale test pointer in lib/cycloidal/params.py.

Checks: ./cadtool lint; ./cadtool pytest (full, slow lane included); derive.py --check (urdf, sdf OK); validate urdf
--strict, srdf --strict, sdf; the hash gate (only the shell ring, the housing bolts and nuts, j1_link, the drive, the
arm and upper_arm_link changed); an overlap check of the changed parts against the whole arm (only the fits the branch
already had); snapshots of the arm, the drive, j1_link and the URDF (elbow at -21) looked at.

File: cad/robot/arm.urdf (robot description, URDF)
Before this commit: robot arm, 10 links, 9 joints
Links:
- link upper_arm_link: mass 1.29899 -> 1.296943
Joints:
- joint elbow_pitch: limit lower=-1.570796 upper=1.570796 effort=5 velocity=1 -> lower=-0.366519 upper=1.570796 effort=5 velocity=1
