Commit message: cad: the elbow motor's 20T placed level with the elbow 90T; its plate's holes M3 clearance; its screws on the buy list
Three small follow-ups to the elbow motor's flip (e616513), asked for after it:

- j1_link's motor plate: the 4 NEMA 17 holes Ø3.2 (copied from the SolidWorks pad) -> M3_CLEAR 3.4, as every other M3
  clearance hole in the arm (lib/upper_arm/params.py, DEFAULT's pad holes). j1_link 376985.495 -> 376960.613 mm^3.
- tools/bom.py EXTRAS: 4 x M3 x 10 socket head cap screws - the elbow motor to its plate, up through the 6 mm plate
  (ArmParams.motor_plate_t) into the motor's tapped holes, 4 of thread in their 4.5 (ELBOW_MOTOR_SCREW_THREAD).
- the elbow motor's 20T placed: gt2_pulley_20t#2 (lib/mounts.py MOTOR_PULLEY_MOUNTS, new), on nema17_40mm#2's shaft,
  hub toward the motor, its hub face J1_MOTOR_20T_HUB_Z 8.978 out from the motor's face (through the plate, 2.98 under
  it; lib/params.py, new) - its tooth band (RollDriveParams.t20_hub on) level with the elbow 90T's to < 0.01 and
  ELBOW_MOTOR_CENTRES (81.97) across; 13 of the shaft in its 14.45 bore. AXES checks its bore (+X) parallel to the
  elbow axis. In upper_arm_link (robot/frames.py LINKS, assemblies/arm.py OCCURRENCES and GROUPS); mount_placements.py
  re-run: placements.json expected 59 -> 60 leaf occurrences, 143 -> 146 solids, 2058102.09 -> 2059980.717 mm^3. The
  open issue's elbow half closes (docs/open_issues.md: the wrist's and the base_yaw's 20Ts remain).

Arm: 86 -> 87 leaves, 245 -> 248 solids, bought leaves 49 -> 50; buy list pieces 49 -> 50 (rows 31). Robot:
upper_arm_link 1.296943 -> 1.304912 kg, COM (0.058957, 0.000068, 0.040525) -> (0.059135, 0.000068, 0.040354),
ixx / iyy / izz 1.600035e-03 / 6.133599e-03 / 6.633113e-03 -> 1.606477e-03 / 6.146757e-03 / 6.640055e-03,
ixz 3.296841e-04 -> 3.361408e-04 (URDF + SDF); upper_arm_link mesh re-exported.

Tests: test_mounts test_elbow_motor_20t_runs_in_the_90ts_band (new), test_placements (the mounted keys, the record
counts), test_bom, test_assembly, test_j1_link (the volume). Docs: lib/mounts.py, parts/wrist/gt2_pulley_20t.py,
docs/open_issues.md, lib/ robot/ tests/ AGENTS.md.

Checks: ./cadtool lint; ./cadtool pytest (full, slow lane included); derive.py --check (urdf, sdf OK); validate urdf
--strict, srdf --strict, sdf; the hash gate (only j1_link, the arm and upper_arm_link changed).

File: cad/robot/arm.urdf (robot description, URDF)
Before this commit: robot arm, 10 links, 9 joints
Links:
- link upper_arm_link: mass 1.296943 -> 1.304912

Commit message: cad: the yoke centred on the base_yaw axis - the drive and all it carries moved 7.5 along N; the disc's -X cut gone
j1_coupler looked off centre and lopsided: its two legs mirror each other about the middle of the cycloidal discs, but
the drive sat where the SolidWorks capture put it, the middle of the discs 7.5 off the base_yaw axis toward the motor -
so the hub leg stood on the yoke's disc, inside its -X flat, and the motor leg 5.5 past the +X flat on a foot of its
own; the disc was cut back on -X only (for the elbow motor, which has since moved to the arm's other side), and the ring
under the drive ran from the old cheek's face (-32.8) to the +X flat.

- lib/yaw_coupler/params.py ForkParams.face_x 31.5 [REFERENCE] -> 24.0 [DESIGN]: the drive's z 0 such that the middle of
  its discs (z 24) lies on the base_yaw axis; CAPTURE_FACE_X 31.5 (new) keeps the capture's. The legs x (-38.5, -30.5) /
  (45.5, 53.5) -> (-46, -38) / (38, 46): mirror images about the yaw axis, each straddling a flat of the disc (its low
  bridge now inside it).
- ForkParams.swing_x and lib/yaw_coupler/body.py _swing_cut removed: the disc whole all round (the elbow motor no longer
  swings on -X; the sweeps below find nothing nearer than the 1 mm running gaps).
- DEFAULT's ring on the disc flat to flat (ring_x0 -32.8 -> -flat_x -40), symmetric under the fork.
- j1_coupler 218277 -> 222140.753 mm^3 (j1_coupler_cap 9182.805, unchanged, moved with the motor leg).
- lib/placements.py SHIFTS: a LinkShift for j1_coupler#1 along its +X (N, the drive's axis) by face_x - CAPTURE_FACE_X
  (-7.5): cycloidal_drive#1, j1_link#1 and everything beyond (the elbow-on records) move; the mounts hosted on them
  follow (mount_placements.py re-run: their records in placements.json). The gripper comes 7.5 nearer the yaw axis
  (60.1 -> 52.6 mm off it).
- robot/frames.py SHOULDER_ORIGIN now P.shifted("j1_link#1", the capture point): the shoulder_pitch origin
  (0.002441, -0.034915, 0) -> (0.002924, -0.0424, 0) (URDF + SDF); shoulder_link 1.327614 -> 1.332521 kg, COM
  (-0.001148, 0.020548, -0.019311) -> (-0.000727, 0.014022, -0.019493), ixx / iyy / izz 3.635636e-03 / 2.656839e-03 /
  2.005629e-03 -> 3.607446e-03 / 2.671331e-03 / 1.968791e-03; the other links' inertials and meshes unchanged (their
  link STEPs differ by float noise only: tests/test_robot.py's mesh check), shoulder_link's mesh re-exported.
- the shoulder's range unchanged: the arm reaches the yoke's disc at 70.5 deg in front (limit 67), clears to -155 behind
  (limit -120).

Tests: test_j1_coupler (the middle of the discs on the yaw axis, the legs straddling the flats, the box's X now the
ears', each leg down to the disc's underside past the recess, the ring's ring_x0), test_placements (the yoke's shift),
cycloidal test_assembly (the SolidWorks node's box moved by the drive's shift). Docs: cycloidal_drive.md §12,
open_issues.md (the end effector's offset), parts/base/j1_coupler.py, lib/ assemblies/ AGENTS.md.

Checks: ./cadtool lint; ./cadtool pytest (full, slow lane included: the sweeps, the robot's meshes); derive.py --check
(urdf, sdf OK); validate urdf --strict, srdf --strict, sdf; the hash gate (j1_coupler and its cap, the arm and the link
STEPs changed - shoulder_link by geometry, upper_arm_link / elbow_link / wrist_roll_link by float noise); snapshots
looked at.

File: cad/robot/arm.urdf (robot description, URDF)
Before this commit: robot arm, 10 links, 9 joints
Links:
- link shoulder_link: mass 1.327614 -> 1.332521
Joints:
- joint shoulder_pitch: origin xyz=0.002441 -0.034915 0 rpy=-1.570796 -0.830504 0.064484 -> xyz=0.002924 -0.0424 0 rpy=-1.570796 -0.830504 0.064484

Commit message: cad: the upper arm one flat slab, shoulder to elbow - no steps on either face
j1_link's DEFAULT was three solids fused together: a plain bar (y 27.5..57.5), the SolidWorks plate slid under it, and
a 6 mm motor plate. In side view that gave two drops on the forearm side and three bumps on the belt side:
- forearm side: the bar's top at 57.5, the step to 50.27 for the roll drive's stator, the r 60 relief wall down to 38.27;
- belt side: the motor plate at 21.5, the 45 deg chamfer, the step to 15.27.
The user asked for a smoother, straighter link. After seeing a before/after preview, they chose a flat slab.

The arm is now one slab with the plate's outline (lib/upper_arm/link.py _slab, ArmParams):
- it runs from the elbow half's underside (ElbowParams.y0) up to the relief's floor (relief_y), y 15.27..38.27,
  23.0 thick;
- it goes from the shell (fused from fuse_r 61, as before) to the r 45 end round the elbow axis.
arm_slide stays 39.27, so nothing beyond the elbow moves (SHIFTS, placements, joint origins unchanged).

The elbow motor's square hole goes through the slab. A motor_plate_t web is left across it, its top at y_outer 27.5:
- the motor's face, its 4 holes and the 20T are exactly where they were;
- the BOM screw length is unchanged.

Removed: _arm, _motor_plate, ArmParams.y_inner / swing_r / swing_above_top / motor_plate_half. The elbow stack and the
stepped slot are factored out of _plate (_cut_elbow_stack, _cut_stepped_slot) and shared with the slab; LEGACY still
builds the SolidWorks part (354048.805).

j1_link:
- volume 376960.613 -> 361439.548 mm^3 (PETG 478.7 -> 459.0 g);
- faces 197 -> 189;
- bbox unchanged.

upper_arm_link inertial (robot/arm.urdf, arm.sdf; mesh re-exported):
- mass 1.304912 -> 1.2852 kg;
- COM (0.059135, 0.000068, 0.040354) -> (0.058734, 0.000069, 0.039494);
- ixx 1.606477e-03 -> 1.596738e-03, iyy 6.146757e-03 -> 6.132447e-03, izz 6.640055e-03 -> 6.592728e-03;
- ixy -2.532405e-06 -> -2.567783e-06, ixz 3.361408e-04 -> 3.615956e-04, iyz -2.882007e-06 -> -2.958169e-06;
- the URDF's total 5.725 -> 5.705 kg.

Clearances at the capture pose, today -> slab (mm). The slab's top is flat, so the forearm-side numbers hold at every
elbow angle.
- Wider:
  - roll drive's board 2.50 -> 14.50;
  - its motor mount 6.27 -> 13.00;
  - its motor 7.34 -> 15.00;
  - the elbow motor's board 4.60 -> 8.07.
- Unchanged:
  - elbow block to the bore rim 1.22;
  - the end cap 3.00 over the top;
  - 90T 3.00;
  - 20T 4.72;
  - 90T screws 5.82.

Tests:
- tests/upper_arm/test_j1_link.py: test_default probes the slab (both faces level from x 68 to 211, the hole through,
  the web) and locks the new volume.
- tests/cycloidal/test_assembly.py: the shell-ring seat check now totals the seat's coplanar faces. The old bar's top
  lay in that plane and merged with it outside the ring (2453 mm^2 as one face). The seat is now the shell body's own
  end face: 1829 mm^2 in 4 pieces, the same area the ring bears on, checked against 1500.

Wording: "motor plate" / "the arm's outer face" become the web / the slab in lib/mounts.py (the nema17_40mm#2 note,
so reference/placements.json's note), lib/params.py, robot/frames.py, the docs and docs/open_issues.md. The
placeholder row stays open: the slab is solid, and hollowing or ribbing it for mass is still to do.

File: cad/robot/arm.urdf (robot description, URDF)
Before this commit: robot arm, 10 links, 9 joints
Links:
- link upper_arm_link: mass 1.304912 -> 1.2852

Commit message: cad: model the elbow motor's 4x M3 that hold it down on j1_link's web
Until now the screws holding the elbow motor (nema17_40mm#2) down were a tools/bom.py EXTRAS row only. They are now a
modelled purchased part, elbow_motor_screws (parts/joints/), placed in the arm:
- 4x M3 x 10 SHCS (ISO 4762), lib/fasteners.py shcs(): no thread, the head's hex socket;
- the heads sit on the underside of the web across j1_link's motor hole, in the hole's open lower half round the 20T;
- the shanks run up through the web's M3 clearance holes into the motor's tapped holes.

Part and placement:
- A pattern part with no reference (lib/reference.py NO_REFERENCE, like yaw_pulley_screws). Its pattern is
  j1_link's pad_holes, so the screws sit on the web's holes by construction.
- lib/mounts.py MOTOR_SCREW_MOUNTS, elbow_motor_screws#1: hosted on j1_link#1, +Z up the link's +Y, its axis checked
  parallel to elbow_pitch (AXES). placements.json was rewritten by mount_placements.py. The 20T's note now says "under
  the web".
- assemblies/arm.py OCCURRENCES and the upper_arm_link GROUP, robot/frames.py LINKS.

Length: lib/params.py J1_MOTOR_SCREW_LEN = ArmParams.motor_plate_t (6) + J1_MOTOR_SCREW_THREAD (4.0, moved here from
tools/bom.py) = 10, short of MOTOR_40.bolt_hole_depth (4.5). The motor model's holes are Ø3.2, so there is no overlap.
The tips stop 15.7 short of the kit's long board screws.

Mass: ELBOW_MOTOR_SCREWS_MASS_G 4.237 g (steel over the modelled 539.697 mm^3).

BOM:
- the hand-kept EXTRAS row is gone;
- the buy list's row comes from the part: "M3 x 10 socket head cap screw (ISO 4762)", 4 pieces, envelope;
- bought parts 31 -> 32, pieces 50 -> 51 (occurrences).

Locks bumped:
- placements expected: leaf_occurrences 60 -> 61, solids 146 -> 150, solid_volume 2059980.717 -> 2060520.414;
- arm leaves 87 -> 88, solids 248 -> 252, bought leaves 50 -> 51;
- MULTI_BODY elbow_motor_screws 4;
- test_yaw_pulley_bolts' NO_REFERENCE check scoped to the base group.

upper_arm_link inertial (robot/arm.urdf, arm.sdf; mesh re-exported):
- mass 1.2852 -> 1.289437 kg;
- COM (0.058734, 0.000069, 0.039494) -> (0.058831, 0.000069, 0.039441);
- ixx 1.596738e-03 -> 1.598911e-03, iyy 6.132447e-03 -> 6.138244e-03, izz 6.592728e-03 -> 6.598398e-03;
- ixy -2.567783e-06 -> -2.559267e-06, ixz 3.615956e-04 -> 3.635803e-04, iyz -2.958169e-06 -> -2.962830e-06;
- the URDF total 5.705 -> 5.709 kg.

Tests:
- tests/upper_arm/test_elbow_motor_screws.py locks the part's numbers: 4 solids, 539.697 mm^3, bbox
  (-18.25, -18.25, -3) + (36.5, 36.5, 13).
- tests/test_mounts.py test_elbow_motor_screws_hold_it_down_through_the_web: each screw on a motor bolt axis, the
  heads on the web's underside, the tip J1_MOTOR_SCREW_THREAD into the motor. The existing interference loop covers
  the screws against j1_link and the other mounts.
- tests/test_bom.py: the buy-list row, and no EXTRAS row.

File: cad/robot/arm.urdf (robot description, URDF)
Before this commit: robot arm, 10 links, 9 joints
Links:
- link upper_arm_link: mass 1.2852 -> 1.289437

Commit message: cad: the elbow motor's screws in the drive motor's seat - heads flush in pockets in a 9 mm web
The user asked for the elbow motor's screws to be sunk in, and to be the same screw as the cycloidal drive's motor's.
The drive's motor plate holds its NEMA 17 with M3 x 10 SHCS (ISO 4762, cycloidal_motor_bolts):
- 6 mm of plate under the heads;
- the heads flush in Ø5.7 pockets (motor_bolt_head_dia 5.3 + bolt_clearance_add 0.4), head_h (3) deep, in a 9 mm plate;
- 4 mm of thread in the motor (bolt_hole_depth 4.5 - motor_bolt_thread_margin 0.5).

The web across j1_link's motor hole now does the same:
- the screws were already that screw (M3 x 10 SHCS, 4 mm into the motor) - their part and placement are unchanged;
- the web grows from 6 to 9 mm thick, downward into the hole's open lower half (y 18.5..27.5): motor_plate_t (6)
  stays under the heads, plus the heads' 3;
- four Ø5.7 head pockets in its underside put the heads flush with it, where before they hung 3 mm below the web.
The motor's face, its holes and its 20T do not move. The 20T's hub face sits level with the web's new underside,
inside the Ø22.5 pilot hole (its r 8 against the hole's 11.25), and its set screw stays below the web.

Parameters:
- lib/upper_arm/params.py ArmParams.motor_screw (M3_SHCS) and motor_pocket_dia (the drive's pocket, from its
  DriveConfig);
- lib/upper_arm/link.py _slab cuts the thicker web and its pockets;
- elbow_motor_screws names the drive motor's screw; J1_MOTOR_SCREW_THREAD is documented as the drive's rule.

Numbers:
- j1_link: volume 361439.548 -> 365539.233 mm^3 (the 3 mm more web, less the four pockets); faces 189 -> 197.
- upper_arm_link inertial (robot/arm.urdf, arm.sdf; mesh re-exported):
  - mass 1.289437 -> 1.294643 kg;
  - COM (0.058831, 0.000069, 0.039441) -> (0.058948, 0.000069, 0.039363);
  - ixx 1.598911e-03 -> 1.601839e-03, iyy 6.138244e-03 -> 6.145592e-03, izz 6.598398e-03 -> 6.604746e-03;
  - ixy -2.559267e-06 -> -2.548876e-06, ixz 3.635803e-04 -> 3.665239e-04, iyz -2.962830e-06 -> -2.969747e-06;
  - the URDF's total 5.709 -> 5.714 kg.
- placements.json: only the elbow_motor_screws#1 note.

Tests:
- test_elbow_motor_screws locks the same order line as cycloidal_motor_bolts, and the drive's thread rule, web under
  the heads and pocket.
- test_j1_link probes the 9 mm web and the pockets (wall and floor), and locks the new volume.
- test_bom: the elbow motor's screw row orders what the drive's does.
- test_mounts: the wording follows.

File: cad/robot/arm.urdf (robot description, URDF)
Before this commit: robot arm, 10 links, 9 joints
Links:
- link upper_arm_link: mass 1.289437 -> 1.294643

Commit message: cad: the pulley bolts' heads sunk in counterbores; every pulley screw 5 mm shorter
The 12 M4 socket cap screws that clamp the driven pulleys (the base_yaw 120T, the elbow and the wrist 90T) had their
heads standing 4 mm proud of each pulley's outer face. Each bolt hole now has a counterbore from the outer face, so
the heads sit 1 mm under it. They stay ISO 4762 socket cap screws.

- lib/belts.py GT2_PULLEY_90T_HEAD_SEAT = 5.0 [DESIGN]: the counterbores' floors under the outer face. The heads
  (4.0 tall) sit 1.0 under the face; each screw is exactly 5 shorter, so every tip ends where it did.
- lib/pulley/params.py PulleyParams.counterbore (dia, depth): none on LEGACY (the SolidWorks match is unchanged);
  DEFAULT, and so YAW, take (M4_SHCS.head_dia + 0.4, GT2_PULLEY_90T_HEAD_SEAT) = Ø7.4 x 5.0, the 7.4 of j1_coupler's
  hub leg and the drive's housing bolts. 1.05 mm of wall is left between each counterbore and the Ø12.5 bore.
  lib/pulley/body.py cuts them after the bolt holes.
- lib/mounts.py: each screw set is seated on the counterbores' floors (_SCREWS_IN_COUNTERBORES, y 8.2 -> 3.2 in the
  pulley frame). The nut frames run from the floors (_SEAT_TO_END), so every nut stays where it was in the world
  (z 35.4 -> 30.4 elbow, 43.6 -> 38.6 wrist, 35.507252 -> 30.507252 yaw).
- Screw lengths, from the floors: elbow M4 x 40 -> 35 (RollDriveParams), wrist M4 x 50 -> 45 (CouplerParams),
  base_yaw M4 x 45 -> 40 (HubParams). Tips past the nuts unchanged: 1.4 / 3.2 / 6.3.

Measured:
- gt2_pulley_90t 24531.703 -> 23975.641 mm^3; gt2_pulley_120t 37623.954 -> 37067.892 mm^3 (-556.062 each).
- elbow_pulley_screws 2564.018 -> 2312.690 mm^3, 20.1 -> 18.1 g; wrist_pulley_screws 3066.672 -> 2815.345 mm^3,
  24.1 -> 22.1 g; yaw_pulley_screws 2815.345 -> 2564.018 mm^3, bbox height 49 -> 44, 22.1 -> 20.1 g.
- placements.json expected solid_volume 2059980.717 -> 2057558.549 mm^3.
- Links (arm.urdf / arm.sdf inertials from derive.py): shoulder_link 1.332521 -> 1.329842 kg, elbow_link 0.742657 ->
  0.739978 kg, wrist_pitch_link 0.416999 -> 0.414320 kg (-2.68 g each: 1.97 g steel, 0.71 g PETG); the arm 5.724 ->
  5.716 kg. Their meshes re-exported.
- reference/native/{elbow,wrist}_pulley_screws.step re-imported (import_native.py --force).

Tests: the stack arithmetic and the clamp test check the heads on the counterbores' floors, the counterbores Ø7.4
from the floors to the face, and the screws clear of the pulley; the 90T's DEFAULT lock counts the counterbores; the
120T and yaw screw locks, and the BOM order lines, take the new numbers.

File: cad/robot/arm.urdf (robot description, URDF)
Before this commit: robot arm, 10 links, 9 joints
Links:
- link elbow_link: mass 0.742657 -> 0.739978
- link shoulder_link: mass 1.332521 -> 1.329842
- link wrist_pitch_link: mass 0.416999 -> 0.41432

Commit message: cad: the roll block 14 mm shorter - bearing 1 beside the elbow pulley's nut channels
The question was whether the forearm roll link (the roll drive's stator in elbow_link) could be smaller. Measured on
the builders, only the block's rear had slack. Bearing 1's seat sat at z -35..-28, but it only has to clear the
elbow 90T's nut channels, which reach |z| 11.73.

The rest of the block is fixed by other parts:
- The 66 x 72 section: the Ø62 ring cavity and the 46 mm motor-mount base.
- The front end: the forearm wall sits 48 mm from the elbow axis.
- The motor: the ring sets its position.

The shorter block was previewed (a before / after cut through the roll axis and renders at one scale) and chosen over
also fitting a 72T ring with a 16T motor pulley, which would have taken 5 mm off the block's height.

- lib/forearm/params.py RollDriveParams:
  - block_z (-40, 36) -> (-26, 36): the block 76 -> 62 mm long. Bearing 1's seat moves -35..-28 -> -21..-14, its
    front face 2.27 behind the nut channels. The bearings are 71 -> 57 mm apart, the shaft 86 -> 72 mm long
    (z -36..50 -> -22..50).
  - lip_dia 72 -> 52, boss_dia 62 -> 50 ([REFERENCE] -> [DESIGN]): both kept inside the block's length behind the
    elbow axis.
  - mount_bolt_z (-22, 1) -> (-8.5, 1): the rear pair's nut pockets stay 2 mm past the new core bore. The screw pairs
    are now 23 -> 9.5 mm apart and the mount's base 50 -> 36 mm long, added to the motor-plate row of
    docs/open_issues.md.
- The motor does not move. Its body now reaches 7.45 mm past the block's rear (it was 6.55 inside), its board 21.55
  (was 7.55).
- Native references re-accepted (tools/reference/import_native.py --force):
  - forearm_roll_block: 192191.808 -> 151335.581 mm^3, bbox z 76 -> 62.
  - forearm_roll_shaft: 94377.8 -> 79423.8 mm^3.
  - forearm_roll_motor_mount: 15378.66 -> 12802.66 mm^3.
  - forearm_roll_mount_screws / _nuts: same volumes, their pattern 13.5 mm shorter along z.
- Printed mass, solid PETG: block 244 -> 192 g, shaft 120 -> 101 g, motor mount 19.5 -> 16.3 g; -74 g in all.
- assemblies/forearm_roll_drive.py EXPECTED: volume 420657.246 -> 362271.038, stator 326279.448 -> 282847.22,
  rotor 94377.799 -> 79423.818.
- tests:
  - test_stack holds bearing 1's seat 2.0..2.5 mm behind the nut channels' reach, and the lip and boss inside the
    block's length.
  - test_j3_coupler no longer asks the block's boss for the coupler's Ø62.
- robot (arm.urdf and arm.sdf):
  - elbow_link: mass 0.742657 -> 0.687498 kg, COM (-6.634, -27.133, 19.145) -> (-4.140, -29.312, 19.208) mm,
    ixx / iyy / izz 1.342914e-3 / 7.968956e-4 / 1.303608e-3 -> 1.232094e-3 / 6.996527e-4 / 1.162924e-3.
  - forearm_link: mass 0.706435 -> 0.687443 kg, COM z 100.337 -> 103.860 mm,
    ixx / iyy / izz 2.435994e-3 / 2.415092e-3 / 3.841204e-4 -> 2.115198e-3 / 2.093880e-3 / 3.777410e-4.
  - The arm 5.724 -> 5.650 kg. Both links' meshes re-exported.
- Checks:
  - derive --check is OK for both files; validate --strict passes for the URDF and SRDF, and the SDF validates.
  - Hash gate against the previous builds: only forearm_roll_block, _motor_mount, _shaft, _mount_screws,
    _mount_nuts, forearm_roll_drive and arm changed.
  - ./cadtool pytest: 898 passed. ./cadtool lint is clean.

File: cad/robot/arm.urdf (robot description, URDF)
Before this commit: robot arm, 10 links, 9 joints
Links:
- link elbow_link: mass 0.742657 -> 0.687498
- link forearm_link: mass 0.706435 -> 0.687443
