Commit message: cad: j1_coupler turned from one drafted base; hub leg disc the hub's Ø; a one-piece motor leg replaces the clamp
The fork's two legs were flat 8 mm plates standing at the edge of the coupler's disc, so any thickening looked tacked
on, and the motor end was held by a split clamp with a cap. The user wanted the legs to grow out of the base, thick at
the root and thin at the mounting area; the part that bolts to the cycloidal's output hub to be the hub's own
diameter; and no clamp on the motor side (chosen: a one-piece motor leg bolted to the base). Previewed as a scratch
build first (claude.ai artifact, three rounds) and approved.

What changes (lib/yaw_coupler/, DEFAULT only - LEGACY and the reference match are untouched):
- The disc is turned: drafted round to its rim (DiscParams band_r 53.082571 -> BASE_R 58.0, Ø106 -> Ø116; top_r
  50.843625 -> 54.19268; the draft dr/dy 0.112 -> BASE_DRAFT 12/63, 6.4 -> 10.8 degrees), its flats and ears filled
  under the legs.
- The disc's drafted side is carried up each leg's outer face, within the post (leg_half_z), to flare_seat_flat (1.5)
  under the hub's lowest bolt heads (layout.fork_flare_top: y 67.23), meeting the 8 mm face in a curved edge at
  y 63 in the middle. The legs' root is 19.98 thick (was 8). The bridges (bridge_y1) are gone, filled by the draft.
- Hub leg: its disc hub_plate_r 35.15 = OutputHubParams.od / 2 (was plate_r 45, Ø90 -> Ø70.3), flush with the hub.
  The 4 M4 on Ø50 are unchanged; their counterbores sit 6.45 inside the edge.
- Motor leg: j1_coupler_cap (the clamp's upper half, 9182.805 mm3, 2x M3 x 25 + nuts) is retired. The new part
  parts/base/j1_motor_leg (no reference, body.build_motor_leg, 44356.285 mm3) is a solid Ø90 ring round the sleeve
  (clamp_bore_dia renamed ring_bore_dia, still 70.4) that slides on over the motor and its board. Its post stands on the
  disc's top face. Its foot is the disc's rim past the leg's outer face (x 46), butting the disc there, held by 2x
  M4 x 10 along the drive's axis (motor_bolt_y 10, motor_bolt_z +/-12, heads seated 4.5 out in the foot, sunk under
  the draft) into M4 nuts in slots from the disc's top face (motor_nut_wall 1.6), under the post. The coupler stops at
  x 46 and its ring is cut back motor_leg_gap 0.2 off the leg. The cap_* fields are gone. COUNTERBORE / HEAD_SEAT /
  NUT_SLOT move from body.py to layout.py (fork_flare_top needs them).
- j1_coupler: 222.14 -> 218.83 cm3. The coupler + motor leg: 231.32 -> 263.19 cm3 (+31.86, +13.8 %). The coupler's
  swept radius about base_yaw: 53.08 -> 58.0; the rim keeps RIM_CLEAR 0.5 over the base's top face.
- lib/mounts.py: YOKE_CAP -> YOKE_MOTOR_LEG, the j1_motor_leg#1 mount at identity on j1_coupler#1.
  reference/placements.json (mount_placements.py): the cap's record replaced by the leg's; expected solid_volume
  2060520.414 -> 2095693.894 (solids unchanged, 150). arm.py OCCURRENCES / GROUPS, robot/frames.py LINKS, the
  lib/reference.py NO_REFERENCE row follow. tools/bom.py EXTRAS: the cap's 2x M3 x 25 + 2 M3 nuts -> 2x M4 x 10 +
  2 M4 nuts.
- shoulder_link inertial (arm.urdf, arm.sdf, from derive.py's drafts): mass 1.332521 -> 1.372986 kg; COM
  (-0.000727, 0.014022, -0.019493) -> (-0.000748, 0.014197, -0.022301); ixx 3.607446e-03 -> 3.821325e-03, iyy
  2.671331e-03 -> 2.866005e-03, izz 1.968791e-03 -> 2.066692e-03, ixy 5.770706e-05 -> 5.875142e-05, ixz
  1.814189e-05 -> 2.293973e-05, iyz -3.590909e-04 -> -4.443663e-04. The robot's total mass is now 5.755 kg.
  robot/meshes/shoulder_link.stl re-exported.
- Tests: tests/yaw_coupler (the draft, the flare's top, the hub disc = the hub's od, the motor side's cut-back, slots
  and holes; test_cap -> test_motor_leg with its numbers); test_placements, cycloidal/test_assembly (the sleeve's end
  on the motor leg's outer face, the drive clear of it), test_bom follow the rename.
- Docs: lib/AGENTS.md, tests/AGENTS.md, assemblies/AGENTS.md, docs/cycloidal_drive.md, the j1_coupler and
  cycloidal_motor_plate docstrings. docs/open_issues.md: the fork's shapes row and the shell fits row (the ring's bore,
  the M4 nuts' slots).

Checks: ./cadtool lint clean; ./cadtool pytest -n 4: 909 passed (fast lane 575), test_sweeps included (the forearm
roll drive clears the legs and the Ø116 base); hash gate against main's STEPs: only j1_coupler.step and arm.step
changed (j1_motor_leg new, j1_coupler_cap gone; the drive and the motor plate byte-identical); derive.py --check
clean; validate arm.urdf / arm.srdf --strict and arm.sdf OK; snapshots of the arm, the coupler, the motor leg, the
drive and the URDF looked at.

File: cad/robot/arm.urdf (robot description, URDF)
Before this commit: robot arm, 10 links, 9 joints
Links:
- link shoulder_link: mass 1.332521 -> 1.372986

Commit message: cad: the roll motor on the elbow axis, the roll housing above it - the forearm moves across (an elbow offset)
The forearm roll motor sat on the roll block's top with its body and board hanging behind the elbow. When the forearm
lifted back, the board met the elbow motor, so the elbow stopped at -21 deg. The user chose layout E from four
compared (the motor about the elbow axis):
- the motor sits ON the elbow axis;
- the roll housing sits above it, the 240-2GT roll belt's centre distance away (60.9 mm);
- the forearm, wrist and gripper move across with the roll axis as one piece, unchanged.
The arm gains an elbow offset: the roll axis no longer crosses the elbow axis, and the wrist stays spherical. The
layout was previewed in 3D before this change (built from the part builders, measured in the arm). The housing is the
shorter stack (bearings 57 apart), chosen over main's (71 apart) for the forearm's lift-back room. PR #25 (the shorter
block alone) is closed: this starts from main.

- The offset is data:
  - ForearmConfig.elbow_offset: LEGACY 0, DEFAULT = RollDriveParams.centre_distance, 60.926 mm
    (lib/params.py ELBOW_ROLL_OFFSET).
  - lib/placements.py SHIFTS gains a fifth LinkShift ("forearm_roll_drive", anchor j2_link#1, across j2_link's +Y). It
    moves j2_link#1 and everything beyond the wrist pitch. The elbow's own records (the retired j3_coupler#1 and
    gt2_pulley_90t#1, which the elbow 90T and its bolts hang on) stay. At the capture pose the forearm side moves
    (-44.46, -2.87, +41.55) mm in the base frame.
  - robot/frames.py: ELBOW_ORIGIN follows the retired j3_coupler#1 (it shares j2_link#1's capture origin).
    FOREARM_ROLL_ORIGIN = j2_link#1's shifted origin + FOREARM_ROLL_AXIS_Z * N, which is 25 along N and 60.93 across
    the elbow axis. The wrist centre stays on the roll axis (0.002 off).
- The stator is one printed frame (forearm_roll_block, lib/forearm/roll.py build_block):
  - the housing round the roll axis: main's bores, block_z -40..36 -> -26..36, the belt window moved to its bottom wall;
  - a web under the motor on the upper arm's side (web_t 10, web_z -40..36) down past the elbow axis, carrying the
    elbow flange (lip / boss / journal / shoulder / stub, the pin bore, the elbow 90T's clearance holes and hex nut
    channels, which now open up into the motor's cradle);
  - the motor's plate (its tension slots and pilot slot), integral now.
  The motor, its board and its 20T sit on the elbow axis (motor_y = elbow_y = -60.93).
- Removed: forearm_roll_motor_mount and its screws and nuts (forearm_roll_mount_screws / _nuts), with their parts,
  NATIVE / NATIVE_COTS rows, reference STEPs, manifest entries and masses, and the RollDriveParams.mount_* fields
  and layout helpers. The motor bolts straight to the frame's plate.
- Re-accepted references:
  - forearm_roll_block: 192191.808 -> 223565.8 mm^3 (frame), bbox 83 x 134.9 x 76.
  - forearm_roll_shaft: 94377.8 -> 79423.8 mm^3 (72 long).
  - Printed stator (frame + cap, solid PETG): 293.8 g (block + mount + cap) -> 314.1 g. Shaft 119.9 -> 100.9 g.
- assemblies/forearm_roll_drive.py EXPECTED:
  - leaves / solids 11 / 32 -> 8 / 23;
  - volume 420657.246 -> 420985.637;
  - stator 326279.448 -> 341561.82;
  - rotor 94377.799 -> 79423.818.
- ELBOW_PITCH_LIMITS_DEG (-21, 90) -> (-47, 90): the roll housing's rear end now meets the elbow motor at -50.0 deg (the
  test's own sweep, 1 mm). The roll motor on the elbow axis never reaches it. 3 deg margin, as before.
- robot (arm.urdf and arm.sdf):
  - forearm_roll origin xyz (0, 0, 0.025) -> (0.000001, -0.060926, 0.025);
  - elbow_pitch lower limit -0.366519 -> -0.820305 rad;
  - elbow_link mass 0.739978 -> 0.754696 kg, COM (-6.658, -27.232, 19.402) -> (-3.976, -22.128, 17.163) mm,
    ixx / iyy / izz 1.327244e-3 / 7.830866e-4 / 1.301175e-3 -> 1.318728e-3 / 7.586526e-4 / 1.262434e-3;
  - forearm_link mass 0.706435 -> 0.687443 kg, COM z 100.337 -> 103.860 mm, ixx / iyy / izz 2.435994e-3 / 2.415092e-3
    / 3.841204e-4 -> 2.115198e-3 / 2.093880e-3 / 3.777410e-4;
  - the arm 5.706 -> 5.702 kg;
  - elbow_link and forearm_link meshes re-exported;
  - the ledger says the axes no longer cross.
- reference/placements.json: mount_placements.py re-ran. The mounted records past the elbow bake the new shift, and
  every on-axis mount passed its check against ELBOW_ORIGIN / FOREARM_ROLL_ORIGIN.
- Tests:
  - test_roll_drive is rewritten for the frame: the web, the flange about y_elbow, the cradle, the motor on the elbow
    axis, the bottom belt window, the upper arm turned about the elbow axis at host (0, -offset).
  - test_placements: five shifts, the forearm's offset in j1_link's frame.
  - test_robot: the elbow / roll origins and their offset.
  - test_mounts: the elbow pulley pattern about elbow_y.
  - test_params_invariants: the limit and ELBOW_ROLL_OFFSET.
  - Locks: the arm 88 -> 85 leaves, 252 -> 243 solids, tints 51 / 37 -> 49 / 36; the bom (30, 37) -> (29, 36) printed,
    (32, 51) -> (30, 49) bought.
- Docs:
  - forearm_roll.md is rewritten for the frame.
  - robot/AGENTS.md (the joints table), assemblies/AGENTS.md (the shift), lib/AGENTS.md and the part notes.
  - open_issues.md: the elbow-limit row; the web's flex (replaces the motor plate's); the frame's print orientation;
    the roll belt sets the offset; a new row for the elbow offset in a future IK. The roll motor mount's fits row is
    closed (the mount is gone).
- Checks:
  - The hash gate against main's builds (built in this worktree before the edit): only forearm_roll_block,
    forearm_roll_shaft, forearm_roll_drive, arm and robot/links elbow_link / forearm_link changed. The three removed
    parts are gone. Every part past the elbow is byte-identical: records move them, they are not rebuilt.
  - derive --check is OK for both files; validate --strict passes for the URDF and SRDF, and the SDF validates.
  - ./cadtool lint is clean; ./cadtool pytest: 893 passed (566 in the fast lane).

File: cad/robot/arm.urdf (robot description, URDF)
Before this commit: robot arm, 10 links, 9 joints
Links:
- link elbow_link: mass 0.739978 -> 0.754696
- link forearm_link: mass 0.706435 -> 0.687443
Joints:
- joint elbow_pitch: limit lower=-0.366519 upper=1.570796 effort=5 velocity=1 -> lower=-0.820305 upper=1.570796 effort=5 velocity=1
- joint forearm_roll: origin xyz=0 0 0.025 rpy=3.141593 -1.570795 0 -> xyz=0.000001 -0.060926 0.025 rpy=3.141593 -1.570795 0

Commit message: cad: the roll pulley is the output - the 90T ring out front on a 6806 pair, one round block round the motor, no end cap
The forearm roll's 90T ring sat between its two 6808s inside the housing, in a Ø62 cavity open to the front, so
bearing 2 needed a bolt-on end cap (forearm_roll_retainer) and the belt a window in the housing's bottom wall; the
motor hung off the housing on a plate. Asked for: the pulley as the output with the forearm bolted straight onto
it, a smaller bearing, one block that holds the motor, and a round elbow end (previewed and approved).

The rotor now splits between its bearings (the elbow's 6806 pattern - two hubs meeting inside the lip): both
bearings are pressed onto printed journals, and with the ring at the front end bearing 2 could not go on across
journal 1.
- forearm_roll_pulley (new, no reference: tests/forearm/test_roll_drive.py holds it) - the output: the integral
  90T ring on a Ø44 core, its rear flange sunk in a cup on the block's front face, its hub through bearing 2, the
  Ø39.7 spigot in the forearm wall's recess. The wall bolts onto the ring's face exactly as before onto the shaft
  (Ø31, Ø24 bore - j2_link's STEP is byte-identical); its screws M3 x 25 -> M3 x 16, into nuts in the core.
- forearm_roll_shaft: a collar behind bearing 1 (its hub through bearing 1 to the pulley's, the Ø33 shoulder, a
  Ø40 flange with the stop lug); 79.4 -> 12.3 cm³.
- the rotor clamp (new): 4x M3 x 35 on Ø24.5, turned 45° off the wall's screws, from the pulley's front face through
  both hubs into nuts in the shaft's flange - the drive is whole without the forearm. Rotor bore Ø24 -> Ø18.
- bearings: 2x 6808 (40 x 52 x 7, 57 apart) -> 2x 6806 (30 x 42 x 7, back to back on a 2 mm lip, 9 apart centre to
  centre), bearing 2 1 mm under the ring; the arm now buys 8 6806s (was 6) and no 6808.
- forearm_roll_block: ONE body round the motor - seen along the elbow axis round about it (end_r 45, concentric with
  j1_link's round end) and tangent up to the tower round the roll axis; the motor in a pocket open on the +N face,
  the pocket's front wall the plate (the tension slots) and one flat front face; the cup (Ø66 boss, its rim 0.3
  under the ring's teeth: the belt runs clear, no window); the shaft's bay behind bearing 1, open on +N, deep enough
  to slide the shaft + bearing 1 in; the stop post on the tower's rear face. The elbow flange under it unchanged.
  223.6 -> 299.7 cm³.
- the motor slides toward the wrist so its 20T meets the ring: face 6.05 -> 24.85, board rear -47.55 -> -28.75;
  pulley_lift 0.5 -> 3.5 (the 20T out to the shaft's tip, the tip 1.15 behind the forearm wall's plane).
- removed: forearm_roll_retainer (23.7 cm³) and bearing_6808 - part files, NATIVE / NATIVE_COTS rows,
  reference/native/*.step, manifest entries -, BEARING_6808_MASS_G, the cap's M3 x 16 BOM row. Re-accepted:
  forearm_roll_block (299709.8 mm³), forearm_roll_shaft (12317.7 mm³).

Locks: forearm_roll_drive EXPECTED 8 leaves / 23 solids / 420985.637 -> 429577.799 mm³; stator 7 / 22 / 341561.82
-> 6 / 21 / 391317.151, rotor 1 / 1 / 79423.818 -> 2 / 2 / 38260.648. Printed parts in the drive 326.7 -> 338.0
cm³. BOM bought part types 30 -> 29 (49 pieces). URDF/SDF: elbow_link 0.754696 -> 0.807236 kg (COM -3.976, -22.128,
17.163 -> 2.227, -11.94, 16.945 mm), forearm_link 0.687443 -> 0.635166 kg (COM z 103.86 -> 112.869 mm); total 5.743
kg; both links' meshes re-exported. The elbow motor's gap to the drive at the -47° limit 4.3 -> 9.3 mm; the drive
reaches 1 mm of it at -60° (was -50°) - ELBOW_PITCH_LIMITS_DEG kept, the room noted in open_issues.

Hash gate: only forearm_roll_block, forearm_roll_shaft, forearm_roll_drive, arm and the elbow_link / forearm_link
robot STEPs changed. docs/forearm_roll.md rewritten; open_issues rows rewritten (the frame's flex, the elbow limit,
the stop, the 6806 pair's tilt play and the clamp's thin walls, the nut pockets, the print orientation, the
journals, the home sensor, the Ø18 cable route), the 6808 row removed.

File: cad/robot/arm.urdf (robot description, URDF)
Before this commit: robot arm, 10 links, 9 joints
Links:
- link elbow_link: mass 0.754696 -> 0.807236
- link forearm_link: mass 0.687443 -> 0.635166

Commit message: cad: the base widens along the coupler's cone into a Ø200 foot - a straight chamfer flare, 6 screw holes
Why: the base was too narrow to keep the arm up. Stretched out, the arm's centre of mass is 131 mm off the
base_yaw axis (165 mm with 0.5 kg in the gripper; forward kinematics over the shoulder / elbow / wrist limits on
robot/arm.urdf's masses), but the base reached 53.3 mm on its round side and its flanks, and it had no holes to fix
it down: standing free, 69% of the poses tipped it with the arm pointed the worst way. Its Ø106.7 tower also stood
4.7 mm inside j1_coupler's Ø116 rim. The shape was chosen on a rendered preview, in two rounds: the Ø200 foot with
screw holes, the tower flush with the coupler and sloped, and a straight chamfer for the flare (not a fillet).

What changed (lib/base/):
- ShellParams.draft: the walls lean out going down, inside and out, `wall` thick horizontally. DEFAULT carries
  j1_coupler's disc cone on down: r 53.34 -> 58.08 at the cap's top face (the coupler's rim, RIM_CLEAR above, on
  the same line), 64.63 at the plate's top, 78.36 at the table; BASE_DRAFT 12/63 (10.8 degrees).
- BASE_R / BASE_DRAFT move from lib/yaw_coupler/params.py to lib/base/params.py (the base cannot import the
  coupler, which imports the base); the coupler imports them under the same names.
- New FootParams (BaseConfig.foot): a D flange Ø200, 6 thick, its sides out to the joint face; a straight chamfer
  from the flange's top at r 95.5 up to the wall 24 above the table (r 73.79), 39.66 degrees from the table;
  6x Ø5.5 (M5 clearance) holes down through the flange on r 92.5 - 4 on the round half at 112.5 / 157.5 / 202.5 /
  247.5 degrees, 2 on the sides at x 43 - each with a Ø11 spot-face down to the flange's top.
- layout.py: outer_r() / inner_r(), flare_points(), foot_holes(); side_stub_x() taken at the plate's top (the same
  value when the walls stand straight).
- body.py: _dd is _d leaning - _d's cylinder becomes a cone, its block a wedge between leaning planes - so the cap
  stays a full disc over the open +X side (a lofted D outline would drop its +X half, the thrust groove's floor
  with it). The outside is one cone from the table to the top face plus the sides' wedges: a lower and an upper cone
  fused at the plate's top made a bad face (31 "unable to clean" warnings, a phantom lip under the top face); now
  none. _foot(): the flange + the chamfer's cone and wedges. The posts reach out to the leaning wall, clipped to its
  outside. With no draft and no foot every piece is the old prism: LEGACY rebuilds the reference's 286169.1 mm^3
  exactly.
- base_motor_mount, the joint (posts, 4x M4, nut pockets), BASE_BOTTOM_Y and the URDF joint origins: unchanged.

Measured:
- base (DEFAULT build): 235439.1 -> 413546.1 mm^3, 299.0 -> 525.2 g PETG; bbox x -53.34..55 / z +/-53.34 ->
  x -100..55 / z +/-100 (printed bottom down: 155 x 200 on the bed, no new overhang).
- base_link inertial (robot/arm.urdf, arm.sdf from derive.py's drafts): mass 0.936947 -> 1.163143 kg; COM
  (-0.046028, 0.000021, 0.056669) -> (-0.032609, -0.000038, 0.050662) m; ixx 1.516875e-03 -> 3.015337e-03,
  iyy 3.015555e-03 -> 4.841445e-03, izz 2.768958e-03 -> 5.296522e-03, ixy 2.865620e-06 -> 5.748429e-06,
  ixz -6.700869e-04 -> -2.228810e-04, iyz 1.172743e-06 -> 2.272553e-06 kg m^2. URDF total 5.743 -> 5.969 kg.
- robot/meshes/base_link.stl re-exported: 34 solids, 568842.8 mm^3, bbox 219.5 x 200.0 x 107.5 mm.
- Standing free, worst direction (the old masses): 69% -> 29% of the poses tip it (48% with 0.5 kg in the
  gripper); it is meant to be screwed down - docs/open_issues.md rows for that and for the foot's screws (not
  modelled), the print row and the cable-exit row (a notch through the foot) updated.

Tests: tests/base/test_foot.py (new: the cone is the coupler's, the flange, the chamfer, the holes and spot-faces,
the walls leaning inside and out, the cap a full disc, volume / bbox); tests/base/test_base.py (the shell, the bbox);
tests/test_params_invariants.py (the shared cone, FootParams). Hash gate: only base.step, arm.step and
robot/links/base_link.step changed. Full suite 898 passed, single-process (tests/test_sweeps.py: the wider tower
stays clear of the arm over its range); URDF / SRDF strict and SDF validate; derive.py --check OK.

File: cad/robot/arm.urdf (robot description, URDF)
Before this commit: robot arm, 10 links, 9 joints
Links:
- link base_link: mass 0.936947 -> 1.163143
