Commit message: cad: the joint limits re-measured - the forearm roll 2 deg inside its hard stop, three sweeps more
Every joint end measured against today's geometry (after the elbow offset and the roll pulley merges): the first
angle each pair comes within 1 mm, and where it touches (every contact confirmed by an overlap volume):
- base_yaw +/-175: nothing within 1 mm at any yaw (every 25 deg) at both shoulder limits over the elbow range.
- shoulder_pitch +67: j1_link reaches j1_coupler's disc at 69.5, inside its 1 mm running gap from 68.6 (the note said
  70.5 / 69.5 - measured before the flat slab and the turned j1_coupler); -120: the upper arm reaches the fork at
  -154.2 (1 mm at -153.5), the forearm stays off the base and the shoulder to -140 at any elbow.
- elbow_pitch -47: the roll frame within 1 mm of the elbow motor's board at -59.8, touching at -61.0 (as noted); the
  forearm, the wrist and the gripper stay 1 mm off the upper arm to -62 at any roll (+/-170, +/-90, 0) and wrist
  pitch; +90: the gripper, the wrist at +70, reaches j1_coupler at 104.8 (1 mm at 104.2); the frame is clear to 130.
- forearm_roll +/-170: the stop lug meets the frame's post at +/-168.3 (0.12 mm at 168.0, 0.03 mm^3 into it at 168.5,
  2.8 mm^3 at 170) - the limit was 1.7 deg PAST the hard stop. The lug and the post are straight-sided boxes
  stop_deg_width wide at their outer radius, so wider further in: the post's inner corner (r 21.6) meets the lug's
  side at 180 - 11.7, not at 180 - stop_deg_width as RollDriveParams.stop_deg claimed.
- wrist_pitch -105 / +70: the wrist body's back corners within 1 mm of j2_link's web at -115.4 / +81.2, touching at
  -116.9 / +82.6 at any wrist roll (the note said -109 / +74.5 - before a2c45f7 necked the web): 11 deg kept, not 4.
- wrist_roll +/-180: the gripper clear of the forearm at every 45 deg at both wrist limits.
- jaws +/-10 mm: the capture pose is open already (the sliders 1 mm inside their rails' ends): +10 runs them 9 mm off
  the rails, -10 still leaves 47.9 mm between the jaws (the sliders reach the static servo horn at -20).

Changed (the user's choices: the roll limit inside the stop; the jaw travel, the elbow and the wrist ranges kept; the
notes fixed and the sweeps made tests):
- FOREARM_ROLL_LIMIT_DEG 170 -> 166 ([ESTIMATE] -> [DESIGN]): the shaft 0.88 mm off the frame at +/-166.
  robot/arm.urdf and arm.sdf forearm_roll limit +/-2.96706 -> +/-2.897247 rad; the URDF ledger, frames.py's joint
  note, robot/AGENTS.md, docs/forearm_roll.md and forearm_roll_shaft's docstring say the stop is just past the limit.
- RollDriveParams.stop_deg removed (170, read only by tests/forearm/test_roll_drive.py, which asserted it equal to the
  limit and to 180 - stop_deg_width); stop_deg_width's comment says where the two meet.
- lib/params.py: the shoulder, elbow, wrist and jaw notes carry the measured numbers.
- tests/test_sweeps.py, three slow tests: the elbow's limits keep the forearm, the wrist and the gripper 1 mm off the
  upper arm, the shoulder and the base at 5 rolls x the 2 wrist limits; at any yaw (every 30 deg + the limits) the arm
  at the shoulder's limits stays 1 mm off the base, j1_coupler and its motor leg RIM_CLEAR over its top face; the roll
  limit stops short of the hard stop (0.5 mm clear at the limit, the lug > 1 mm^3 into the post at 180 -
  stop_deg_width). Helpers: _at() poses links by their own joints, _boxed(), _in_table(), and _distance() - BRepExtrema
  returned false zeros at single poses (the roll shaft against the frame at -140 / -145, the frame against j1_link at
  elbow +92, 1.0 / 1.2 mm either side, no overlap): a zero is measured again with the pose moved 0.01 mm three ways and
  the median kept; _closest uses it. The suite gains 4 min, in this file.
- docs/open_issues.md: the wrist row (the corners' new contact, the room to -112 / +78), the elbow row (the forearm
  side swept, the room to about -56), the roll-stop row (2 deg short, where they meet); new rows: the jaw travel does
  not fit the gripper, and the table as a floor (inside the limits the arm reaches below the base's bottom face - e.g.
  the shoulder at -120 with the elbow at -47, 36 mm below, behind the base - and the sweeps skip those poses).
- tests/AGENTS.md: the sweeps' new checks; a gotcha for the false zeros.

Checks: the hash gate - all 75 STEPs (parts, assemblies, robot links) byte-identical to main's builds; derive --check
OK for the URDF and the SDF; validate --strict passes for the URDF and the SRDF, the SDF validates; ./cadtool lint is
clean; ./cadtool pytest: 892 passed (563 in the fast lane).

File: cad/robot/arm.urdf (robot description, URDF)
Before this commit: robot arm, 10 links, 9 joints
Joints:
- joint forearm_roll: limit lower=-2.96706 upper=2.96706 effort=5 velocity=1 -> lower=-2.897247 upper=2.897247 effort=5 velocity=1

Commit message: cad: j1_link prints flat - the arm slid 9.77 mm onto the shell's hub end, the motor web and M3x12 heads flush
j1_link printed badly on a 256 bed (Bambu P2S). Its only usable orientation is the shell's hub end on the plate (it
is longer than the bed's side, so it lies flat, turned 45 degrees), and in that orientation the arm rose off the
middle of the shell: its whole underside, 169 x 90 mm, hung 9.77 mm above the plate on supports, and the web under
the elbow motor sat a further 3.23 mm up in a recess. Now the slab's underside is flush with the shell's hub end and
the web is flush with both: one flat face goes on the bed.

What changed:
- arm_slide puts the slab's underside (ElbowParams.y0) on the shell's hub end (drive z 61, y 5.5); the elbow motor's
  face (ArmParams.y_outer) is the web's thickness above it. arm_slide 39.271993 -> 29.5, so the arm and everything
  past the shoulder move 9.77 mm along N toward the hub end (lib/placements.py SHIFTS, the mounted records, the
  elbow joint's origin). J1_MOTOR_PAD_FACE_Y 27.5 -> 16.5.
- The web across the motor hole runs from the slab's underside to the motor's face: 9 -> 11 thick, the recess gone.
  The screws' heads stay flush in their 3 mm pockets, so the web under the heads (motor_plate_t) is 6 -> 8 and the
  screws are M3 x 10 -> M3 x 12 (stock), with the same 4 mm of thread in the motor; the motor sits 1.23 mm deeper in
  its hole. elbow_motor_screws: 4.2 -> 4.7 g, the volume lock 539.697 -> 596.246 mm3, height 13 -> 15. It is no longer
  the drive motor's order line (cycloidal_motor_bolts stays M3 x 10).
- The 20T moves 1.23 mm nearer the motor on its shaft (J1_MOTOR_20T_HUB_Z 8.978 -> 7.75), so its tooth band, the
  belt and the 90T stay where they were relative to the arm. Its hub now sits 3.25 up in the web's Ø22.5 pilot hole
  (the pulley is Ø16); its grub screws' axis is 0.75 past the face, as it was past the arm's underside before - a
  key still reaches them along the face (tests/test_mounts.py).
- Flush with the hub end, the slab covered the housing-nut pocket on the lug under the arm (41 mm3 of it: its outer
  flat at r 62.1 lies past fuse_r 61). The pockets and bolt holes are cut again after the union:
  housing_bolt_cutters() is factored out of build_shell_body() (lib/cycloidal/housing.py), which still cuts them in
  the same order - every drive part's STEP is byte-identical.

j1_link: volume 365539.233 -> 368453.715 mm3 (+2914.5, the web's fill); bbox unchanged (279.6 x 52 x 116).
Printability (dfam-check on print/j1_link.stl, 45 degrees, the hub-end face down): support area 11768 -> 1090 mm2
(13.8 -> 1.3 % of the surface); bed contact 4561 -> 15364 mm2; thinnest wall 1.77 mm, 5th percentile 2.99 -> 3.63 mm;
watertight, one solid. What is left over open air is short bridges: the nut and screw pockets' roofs (7.2 / 5.7 mm),
the stepped slot's step (10 wide), the elbow seat's 2.3 mm lip ring. Fits 256 x 256 lying flat at 45 degrees (a
228.6 mm square), as before.

The belt side moves 9.77 mm toward j1_coupler's hub leg: the elbow belt now runs wholly past the shell's hub end, level
with the leg. The belt is not modelled, so it was swept separately (a scratch script, not in the repo): the elbow
belt as a 6 mm band round the two pulleys' pitch circles + 1 mm, the 20T, the 90T with its screws and the elbow motor
+ board, turned through SHOULDER_PITCH_LIMITS_DEG (-120 .. 67, 3 deg steps refined to 0.5) against j1_coupler,
j1_motor_leg, the base, its motor mount and the yaw 120T with its screws and nuts. Closest approach, before ->
after: the belt 45.51 -> 45.51 mm, the 20T 44.35 -> 44.88, the elbow motor + board 21.99 -> 21.05 (all to
j1_coupler, at the limits), the 90T > 20 everywhere. tests/test_sweeps.py (j1_link and the modelled parts against the
fork and the base) passes.

Robot: elbow_pitch origin z 0.049271 -> 0.039499 (URDF and SDF); upper_arm_link mass 1.294643 -> 1.298788 kg, COM
(0.058948, 0.000069, 0.039363) -> (0.059039, 0.000069, 0.034048), ixx 1.601839e-03 -> 1.660568e-03, iyy 6.145592e-03
-> 6.207716e-03, izz 6.604746e-03 -> 6.609814e-03, ixz 3.665239e-04 -> 7.202599e-04, ixy -2.548876e-06 ->
-2.539946e-06, iyz -2.969747e-06 -> -2.465453e-06; total 5.973 kg. upper_arm_link.stl re-exported. The links past
the elbow keep their inertials: their geometry moved with their joint frames.

Recipe C (Mac, in a worktree, the before hashes from the main checkout): 10 STEPs changed - j1_link,
elbow_motor_screws, arm, and the links upper_arm, elbow, forearm, wrist_pitch, wrist_roll, jaw_a, jaw_b. The six past
the elbow are the same geometry to 1e-6 mm (`./cadtool inspect diff`), float noise from the moved frames; the other
65 are byte-identical. mount_placements.py regenerated the mounted records (reference/placements.json). derive.py
--check OK; validate --strict OK (URDF, SRDF; SDF --gz-check never). Snapshots of the arm, the URDF and j1_link
looked at. Lint clean. ./cadtool pytest: 902 passed.

Docs: ArmParams, arm_slide, the j1_link and elbow_motor_screws docstrings, lib/AGENTS.md, assemblies/AGENTS.md,
docs/cycloidal_drive.md (the arm no longer leaves the shell over arm_zone, which stays the gear's stretch where the
shell's body starts). docs/open_issues.md: the slab row says the underside and the web are flush with the hub end;
new row - j1_link's print orientation, closed by the first print.

File: cad/robot/arm.urdf (robot description, URDF)
Before this commit: robot arm, 10 links, 9 joints
Links:
- link upper_arm_link: mass 1.294643 -> 1.298788
Joints:
- joint elbow_pitch: origin xyz=0.170004 0 0.049271 rpy=0 0 0.010227 -> xyz=0.170004 0 0.039499 rpy=0 0 0.010227

Commit message: cad: the roll frame grows out to its cup - the Ø66 cup flush on the underside, the +N face and the tower's top
The cup on the roll frame's front face (bearing 2's seat, the pulley's rear flange sunk in it) is centred on the roll
axis, as it must be, but the frame round it was not: flush with the cup on the underside (-33), it stopped 7 mm short on
the open +N face (26) and 4 mm short at the tower's top (29), so the cup hung over two edges and read as stuck on off
centre. The +N face was cut back to 26 when the frame became one body round the motor; the cup kept the old housing's
Ø66. Asked for: the frame grown out to the cup (previewed and approved, against trimming the cup flush or leaving it).

- lib/forearm/params.py: ROLL_FRAME_R (33) - the underside, the open +N face, the tower's top and the cup's radius:
  block_x (-33, 26) -> (-33, 33), tower_y 29 -> 33, cup_od 66 = 2 x ROLL_FRAME_R. The frame is now symmetric about the
  roll axis along N; test_stack holds all four equal.
- forearm_roll_block 299709.793 -> 338986.502 mm³ (+39.3 cm³, +13 %), its native reference re-accepted; bbox unchanged
  (83.0 x 138.926 x 84.5 - the cup already reached both). The motor pocket and the shaft's bay stay open on +N, 7 mm
  deeper; the roll motor's connector, 2 mm proud of the old face, ends 5 mm inside the open pocket.
- Printed parts in the drive 338.0 -> 377.2 cm³.

Locks: forearm_roll_drive EXPECTED 8 leaves / 23 solids / 429577.799 -> 468854.508 mm³; stator 6 / 21 / 391317.151 ->
430593.86, rotor unchanged. URDF/SDF: elbow_link 0.807236 -> 0.857118 kg (COM 2.227, -11.94, 16.945 -> 1.964, -13.366,
18.592 mm; ixx / iyy / izz 1.133437e-03 / 6.678987e-04 / 1.072495e-03 -> 1.313547e-03 / 7.420103e-04 / 1.221014e-03),
total 5.968777 -> 6.018659 kg; elbow_link's mesh re-exported.

Clearances: the upper arm's elbow board to the drive at the -47° limit 9.32 -> 8.44 mm (its motor 10.17 -> 9.33), the
1 mm line -59.8° -> -58.1° (ELBOW_PITCH_LIMITS_DEG kept; open_issues' room to lift further -56 -> -55); the frame to
the base and the shoulder over the shoulder-limit sweep's poses 53.6 -> 53.1 mm; the frame to j1_link (the journal's
edge) 1.22 mm, unchanged. lib/params.py's FOREARM_ROLL_BLOCK_X comment already read (-33, 33): now it is.

Hash gate: only forearm_roll_block, forearm_roll_drive, arm and robot/links/elbow_link changed. Fast lane 570 passed,
full suite 902 passed, lint clean, arm.urdf / arm.srdf --strict and arm.sdf validate, derive.py --check OK.
docs/forearm_roll.md and docs/open_issues.md follow.

File: cad/robot/arm.urdf (robot description, URDF)
Before this commit: robot arm, 10 links, 9 joints
Links:
- link elbow_link: mass 0.807236 -> 0.857118

Commit message: cad: belts at the GT2 multipack lengths - base_yaw 320 -> 300, roll 240 -> 280
Why: the belts are bought as the Amazon GT2 6 mm multipacks (110, 112, 122,
158, 200, 280, 300, 400, 610 - one of each per pack); 320 and 240 are not in
them. The elbow's 280 already is; the wrist's 258 follows in the next commit
(with an idler). Each length still sets its motor's centre distance, so the
motors move to where the stock belt puts them. Chosen from a to-scale preview
(today vs new, plan cuts at each belt's plane).

base_yaw: YAW_BELT 320 -> 300 [DESIGN] (was [ESTIMATE]). The 48 mm motor moves
10.900 nearer the yaw axis: BASE_MOTOR_PATTERN_CENTRE x 83.967 -> 73.067. The
motor mount follows _MOTOR_X: its far end 119.467 -> 108.567 (53.567 long, was
64.467), volume 57246.053 -> 52094.084 mm^3, native reference re-accepted
(import_native.py --only base_motor_mount --force). The motor's face now rests
3.1 mm (5.6 at the slots' near end) on the base's flush side of the plate, and
the -X slots' near ends cross the joint face (split_x) into the base by 1.6 mm:
both parts cut the same seat, so they line up. The base: volume 413546.1 ->
413503.0 mm^3 (tests/base/test_foot.py). tests/base/test_motor_mount.py: the
face is held to the plate outside the base's posts (2.4 to spare) instead of
"on the mount"; the slot probe looks in whichever part holds the slot's end.
Fit (a scratch build of the whole arm): the belt's path 5.8 from the base and
the mount, the motor's board 10.0 from the base.

forearm_roll: roll_belt 240 -> 280 [DESIGN]. Its centre distance is the arm's
elbow offset: ELBOW_ROLL_OFFSET 60.926 -> 81.972, so the forearm, wrist and
gripper sit 21.046 further across (lib/placements.py SHIFTS follows). The roll
frame grows with it: forearm_roll_block 299709.793 -> 359141.394 mm^3, bbox
83 x 138.926 x 84.5 -> 83 x 159.972 x 84.5, native reference re-accepted.
assemblies/forearm_roll_drive.py EXPECTED: solid_volume 429577.799 ->
489009.4, stator 391317.151 -> 450748.752 (leaves / solids unchanged).

robot: forearm_roll origin y -0.060926 -> -0.081972 (arm.urdf, arm.sdf);
base_link mass 1.163143 -> 1.156545 kg, COM (-32.609, -0.038, 50.662) ->
(-27.952, -0.039, 50.606) mm; elbow_link mass 0.807236 -> 0.882714 kg, COM
(2.227, -11.940, 16.945) -> (2.331, -18.632, 17.334) mm (inertias from the
drafts); the arm 5.969 -> 6.038 kg. base_link and elbow_link meshes
re-exported. derive.py --check OK; validate --strict OK.

placements.json: mount_placements.py re-ran (the base_yaw motor + board, and
every mounted record past the elbow, shifted); expected solid_volume
2093271.726 -> 2088119.757.

Every sweep test passes with the bigger offset (the elbow's limits keep the
forearm 1 mm off the upper arm; the roll frame clears the elbow motor over
the elbow's range), so ELBOW_PITCH_LIMITS_DEG stays. The room past the lower
limit quoted in lib/params.py and docs/open_issues.md (-59.8 deg, 9.3 mm, -62,
104.8) is re-measured in a later commit of this branch.

Docs: open_issues - the roll belt row closed (the length is decided), the
base_yaw belt row now the motor's hold and the slots across the joint;
docs/forearm_roll.md and the URDF ledger name the constants instead of 60.9 /
240-2GT. lib/params.py BASE_MOTOR_PATTERN_CENTRE's stale "280-2GT" comment
fixed.

Checks: hash gate (only base, base_motor_mount, forearm_roll_block, arm,
forearm_roll_drive changed); ./cadtool pytest: 902 passed.

File: cad/robot/arm.urdf (robot description, URDF)
Before this commit: robot arm, 10 links, 9 joints
Links:
- link base_link: mass 1.163143 -> 1.156545
- link elbow_link: mass 0.807236 -> 0.882714
Joints:
- joint forearm_roll: origin xyz=0.000001 -0.060926 0.025 rpy=3.141593 -1.570795 0 -> xyz=0.000001 -0.081972 0.025 rpy=3.141593 -1.570795 0

Commit message: cad: wrist belt 258 -> 280 - the motor at its slide's wall end, a GT2 idler under the web takes up the rest
Why: 258 is not a multipack length; 280 is. The wrist motor cannot move the
11.5 mm toward the elbow a 280 needs (its plug would hit the roll wall), so it
sits at its slide's wall end and the modelled GT2 idler (gt2_idler_20t, placed
for the first time) takes up the rest on the belt's back. Chosen from a
to-scale preview.

The belt's path, exactly (lib/belts.py, a leaf): a loop of circles with signed
pitch radii (a back-side idler negative) - belt_runs(), belt_wraps(),
belt_length() - and idler_on_run(), which pushes an idler into a run until the
loop is a given length. GT2_BELT_THICKNESS 1.38 [DATASHEET], GT2_BELT_BACK
0.376 (pitch line to back), GT2_BELT_MASS_G_PER_M 7.5 [ESTIMATE].
STANDARD_2GT_LENGTHS is now the multipacks' set (110, 112, 122, 158, 200, 280,
300, 400, 610) [DESIGN]; tests/test_params_invariants.py holds every belt
constant to it.

Wrist: RollEndParams.wrist_belt 258 -> 280 [DESIGN], wrist_belt_z 0.3 (the
wrist 90T's band, [REFERENCE]). J2_MOTOR_SLIDE_X -99.522 -> -94.0 (the wall
end), slide (-103.5, -94) -> (-99.5, -94): 5.5 of travel left for fitting the
belt; the side slots -119 -> -115 at their boss end, the pilot slot's boss end
-110 -> -100.5 (1 past the slide) to leave web for the idler's nut channel.
The open loop is 268.581; the idler (IdlerParams.along 24 from the motor's
axis, on the run leaving the 20T) is pushed 18.905 in and takes up 11.419; the
20T wraps 192.8 deg (was 143.1: 10.7 teeth in mesh, was 8.0). J2_IDLER_XY
(-118.0, 0.966) in j2_link's frame. Clearances: its flanges 7.0 from the 20T's,
>13 from the 90T's, 4.3 from the other run's tooth tips; +/- 3 of slot
(IdlerParams.travel) moves the loop -3.2 / +3.7 about the belt.

How it is held (IdlerParams): j2_link gets a rib under the web (7 wide - the
idler's bearing inner ring, [ESTIMATE]), an M5 slot along y through rib and web,
and the nut's channel (8.2 across x) down from the top face to 3 above the web's
underside (lib/forearm/link.py idler_mount); j2_link 172893.5 -> 174398.4 mm^3.
New purchased pattern parts with no reference (lib/reference.py NO_REFERENCE,
locked in tests/forearm/test_wrist_idler.py): wrist_idler_screw, M5 x 20 SHCS up
from under the idler (641.783 mm^3, 5.04 g), and wrist_idler_nut, M5 (168.216
mm^3, 1.32 g); M5_SHCS / M5_NUT in lib/fasteners.py. Mounted (lib/mounts.py
IDLER_MOUNTS, forearm_link, wrist_pitch): gt2_idler_20t#1 level with the belt,
its top on the rib; the screw's head under it, its tip 3.2 under the motor's
face; the nut on its channel's floor under the motor's edge. The idler's
UNPLACED and its EXTRAS row are gone.

Locks: placements expected leaf_occurrences 61 -> 64, solids 150 -> 153,
solid_volume 2088119.757 -> 2090066.91; the arm 85 -> 88 leaves, 243 -> 246
solids, bought leaves 49 -> 52; buy list 29 -> 32 parts, 49 -> 52 occurrences.
The slide tests allow the motor at the slide's end.

robot: forearm_link mass 0.635166 -> 0.648435 kg, COM (5.138, -0.013, 112.869)
-> (4.595, 0.002, 110.273) mm; the arm 6.038 -> 6.051 kg; forearm_link mesh
re-exported. derive.py --check OK; validate --strict OK.

Docs: open_issues - the wrist motor's belt-estimate row replaced by the idler's
clamp estimate (its faces on the bearing's inner ring) and the belt's section /
mass; the "where the idler goes" row now the other belts' idlers (the elbow belt
still has no tension adjustment); docs/forearm_roll.md, j2_link's docstring,
lib/AGENTS.md, robot/AGENTS.md.

Checks: hash gate (j2_link changed, besides the previous commit's); ./cadtool
pytest: 917 passed.

File: cad/robot/arm.urdf (robot description, URDF)
Before this commit: robot arm, 10 links, 9 joints
Links:
- link forearm_link: mass 0.635166 -> 0.648435
