Commit message: cad: the roll frame's Ø66 cup becomes a Ø52 bearing boss - no cup round the pulley's flange
The cylinder on the roll frame's front face holds only bearing 2 (bearing 1 sits in the tower behind the front face);
bearing 2's Ø42.15 seat needs about Ø50 with the frame's 4 mm wall. Its Ø66 came from a 1.9 mm cup round the pulley's
Ø59.19 rear flange - a shroud no load goes through. Asked for: the smaller boss (previewed and approved).

- lib/forearm/params.py: cup_od / cup_id_add / rim_under_teeth -> bearing_boss_dia 52 (4.9 of wall round the seat);
  ROLL_FRAME_R keeps the frame symmetric, so the boss sits centred with 7 mm of front face to the underside, the +N
  face and the tower's top.
- lib/forearm/layout.py: the station z_cup -> z_boss (the boss's top = bearing 2's front face); z_rim removed.
- lib/forearm/roll.py build_block: the boss up to bearing 2's face, no cup cut. The ring's rear flange turns run_gap
  (1.000 mm, unchanged) over the boss's top and 3.6 mm past its edge - the gap now open at the side.
- Removes an undercut: the Ø66 cup overhung the tower's r6 rounded top-front corner (a crescent ~38 mm long, up to 5 mm
  deep under the cup's top edge - there before the frame grew, under the old overhang); the Ø52 boss ends on the flat
  of the front face, 1 mm short of the rounding (test_stack holds that).
- forearm_roll_block 338986.502 -> 326642.594 mm³ (-12.3 cm³), its native reference re-accepted; bbox 83.0 x 138.926 x
  84.5 -> 82.6 (the rim gone). Printed parts in the drive 377.2 -> 364.9 cm³. The pulley's STEP is byte-identical.

Locks: forearm_roll_drive EXPECTED 468854.508 -> 456510.6 mm³; stator 430593.86 -> 418249.952, rotor unchanged.
URDF/SDF: elbow_link 0.857118 -> 0.841441 kg (COM 1.964, -13.366, 18.592 -> 1.375, -12.477, 18.472 mm; ixx / iyy / izz
1.313547e-03 / 7.420103e-04 / 1.221014e-03 -> 1.262483e-03 / 7.183065e-04 / 1.161466e-03), total 6.018659 -> 6.002982
kg; elbow_link's mesh re-exported. Clearances unchanged: the elbow board 8.44 mm off the drive at -47°, 1 mm at
-58.1°; the shaft 1.468 mm off the frame.

Tests: the cup's checks become the boss's - the seat's wall >= 4, its top at bearing 2's face, the flange past its
edge, the belt's edge above it, the boss on the flat of the front face; probes round the boss and nothing above it.
Docs: docs/forearm_roll.md (the cup row folded into bearing 2's), docs/open_issues.md (print orientation row).

Hash gate: only forearm_roll_block, forearm_roll_drive, arm and robot/links/elbow_link changed. Fast lane 570 passed,
full suite 902 passed, lint clean, arm.urdf / arm.srdf --strict and arm.sdf validate, derive.py --check OK.

File: cad/robot/arm.urdf (robot description, URDF)
Before this commit: robot arm, 10 links, 9 joints
Links:
- link elbow_link: mass 0.857118 -> 0.841441

Commit message: cad: model the four GT2 belts as purchased parts, and the base_yaw and wrist motors' 20T pulleys
Why: the belts were only buy-list rows (and the base_yaw belt not even that),
so nothing in the model showed where they run or what they clear; the base_yaw
and wrist motors had no 20T on their shafts. Now every belt is a part on its
pulleys, at its stock length.

The belts: purchased parts with no reference (lib/reference.py NO_REFERENCE),
their envelope a smooth band round the exact loop (lib/pulley/belt.py
closed_belt(), from lib/belts.py belt_runs() / belt_wraps()): the land on the
pulleys' tooth tips (GT2_PLD inside the pitch line), the back GT2_BELT_BACK
outside it, GT2_BELT_W wide; no teeth (they would have to mesh with every
pulley). MASS_G = length x GT2_BELT_MASS_G_PER_M [ESTIMATE].
- yaw_belt (parts/base/): 300-2GT, 1136.33 mm^3, 2.25 g; loop
  lib/base/layout.py yaw_belt_loop() (73.067 between axes), frame
  yaw_belt_frame() at YAW_BELT_Y -31.1 (the 120T's band, [REFERENCE]).
- elbow_belt (parts/joints/): 280-2GT, 1059.993 mm^3, 2.1 g; loop
  lib/upper_arm/layout.py elbow_belt_loop(); J1_BELT_Y 7.572.
- forearm_roll_belt (parts/joints/): 280-2GT, 1059.993 mm^3, 2.1 g; loop
  lib/forearm/layout.py roll_belt_loop(); a row of
  assemblies/forearm_roll_drive.py at the ring's mid-plane.
- wrist_belt (parts/joints/): 280-2GT round the idler, 1059.849 mm^3, 2.1 g;
  lib/forearm/layout.py wrist_belt_loop() / wrist_belt_frame().
Each loop's pitch length is its belt's: the wrist's exactly (the idler is
solved to it), the two-pulley ones at the textbook centre distance 0.04 (90T)
/ 0.23 (120T) long.

The 20Ts (lib/mounts.py MOTOR_PULLEY_MOUNTS): gt2_pulley_20t#3 on the base_yaw
motor (BASE_MOTOR_20T_HUB_Z 2.85, its hub in the motor plate's window) and #4
on the wrist motor (J2_MOTOR_20T_HUB_Z 7.75, its hub up in the web's pilot
slot), each band level with its driven pulley's. The belts (BELT_MOUNTS) ride
with their motors' links: yaw_belt#1 base_link, elbow_belt#1 upper_arm_link,
wrist_belt#1 forearm_link; the roll belt in the roll module's stator
(elbow_link). The three belt rows left tools/bom.py EXTRAS.

tests/test_belts.py: each belt a stock length, its loop that long, the band's
volume / bbox locks and its land / back at every wrap, each mounted loop's
circles on its pulleys' axes in their band plane (0.01), line-to-line contact
with its pulleys and the idler. tests/test_sweeps.py: the base_yaw belt joins
the yaw sweep's exclusions (it rides the turning 120T). Fit (the mounts'
interference budget and a scratch build): every belt touches only its pulleys
(and the wrist idler); nearest else - yaw 5.8 to the base and the mount,
elbow 3.6 to its motor and 4.7 to j1_link, roll 0.8 to the frame's cup rim,
1.7 to the forearm wall, wrist 1.5 under the web's rib.

Locks: placements expected leaf_occurrences 64 -> 69, solids 153 -> 162,
solid_volume 2090066.91 -> 2097080.336; the arm 88 -> 94 leaves, 246 -> 256
solids, bought leaves 52 -> 58; buy list 32 -> 36 parts, 52 -> 58 occurrences;
forearm_roll_drive EXPECTED leaves 8 -> 9, solids 23 -> 24, solid_volume
489009.4 -> 490069.393 (stator 7 / 22 / 451808.745), its bought leaves 5 -> 6.

robot (inertials from the drafts, the four meshes re-exported): base_link
1.156545 -> 1.166795 kg, upper_arm_link 1.294643 -> 1.296743, elbow_link
0.882714 -> 0.884814, forearm_link 0.648435 -> 0.658535; the arm 6.051 ->
6.075 kg. derive.py --check OK; validate --strict OK.

Docs: open_issues - the "belt-side hardware not modelled" and "roll / wrist
belts in EXTRAS" rows closed; robot/AGENTS.md (the base_yaw reduction, the link
table), assemblies/AGENTS.md, lib/AGENTS.md, docs/forearm_roll.md.

Checks: hash gate (no part changed beyond the previous commits); ./cadtool
pytest: 946 passed.

File: cad/robot/arm.urdf (robot description, URDF)
Before this commit: robot arm, 10 links, 9 joints
Links:
- link base_link: mass 1.156545 -> 1.166795
- link elbow_link: mass 0.882714 -> 0.884814
- link forearm_link: mass 0.648435 -> 0.658535
- link upper_arm_link: mass 1.294643 -> 1.296743

Commit message: cad: the forearm turned half a turn about its roll axis - the wrist-pitch motor on the upper arm's side
The wrist-pitch motor (nema17_40mm#3 + mks_servo42d#3) moves to the other side of the forearm: j2_link and everything
beyond it - the wrist bearings, the motor and its board, the wrist 90T and its M4s, j3_coupler#2, wrist_link, the
bracket, the pancake and the gripper - turn 180 deg about the forearm_roll axis from the capture. The roll drive keeps
its pose, its rotor too, so the printed hard stop and +/- FOREARM_ROLL_LIMIT_DEG stay; the forearm wall's 4 bolts (0 /
90 / 180 / 270 deg about the roll axis) take the pulley turned. Previewed and approved first (scratch build, renders,
sweeps).

- lib/placements.py: TURNS (LinkTurn: a turn about an axis in the anchor's frame, applied after the SHIFTS) - the
  forearm's, anchor j2_link#1, the roll drive's SHIFTS list, ForearmConfig.roll_turn_deg (new, LEGACY 0, DEFAULT 180;
  lib/params.py FOREARM_ROLL_TURN_DEG). location() / record_location() apply it (turned=False: the frame before it);
  shifted() turns points, turned() directions (kernel-free, robot/frames.py imports them), is_turned(), turn_line().
- tools/reference/mount_placements.py: a ModuleMount resolves its host unturned (the roll drive drives the joint the
  turn is about); the mounted records hosted on turned ones follow. reference/placements.json: the 8 records
  re-resolved (nema17_40mm#3, mks_servo42d#3, bearing_6806#5 / #6, gt2_pulley_90t#4, wrist_pulley_screws#1 /
  _nuts#1); forearm_roll_drive#1's pose unchanged (its note only); expected totals unchanged.
- robot/frames.py: FOREARM_ROLL_ORIGIN from the capture's roll point, shifted only (it lies on the turn's axis);
  WRIST_PITCH_AXIS (the capture's N turned: -N), WRIST_ROLL_AXIS, JAW_TRAVEL and WRIST_CENTRE turned with the forearm;
  the joints beyond the roll use them.
- robot/arm.urdf / arm.sdf (derive.py drafts): wrist_pitch origin xyz (0.016998, 0, 0.17) -> (-0.016997, -0.000007,
  0.17), rpy (-1.570799, -1.271722, -1.570793) -> (-1.570808, -1.271748, 1.570808); forearm_link COM (0.005138,
  -0.000013, 0.112869) -> (-0.005123, 0.000008, 0.112869), ixx 1.440980e-03 -> 1.440981e-03, ixy 2.446769e-07 ->
  2.482208e-07, ixz 1.299114e-04 -> -1.291062e-04, iyy 1.418393e-03 -> 1.418477e-03, iyz -3.164737e-08 ->
  5.993678e-08, izz 3.582283e-04 -> 3.583121e-04, mass 0.635166 unchanged; meshes/forearm_link.stl re-exported. The
  forearm_roll origin and every link past the wrist unchanged (their frames turn with them). At zero the gripper is
  rolled 180 deg from the SolidWorks capture (the SRDF home); the ledger says so.
- Tests: the turn (test_the_forearm_turns_about_its_roll_axis), the module record on its unturned host, the joint
  origins, the wrist axes through the wrist centre; tests/forearm/helpers.py in_drive_frame() / j2_link_in_drive_frame()
  - the roll drive's tests stay in j2_link's frame before the turn; tests/totals.py takes a turned record's bbox from
  its build.
- Docs: docs/forearm_roll.md (the forearm turned, §0 / §1 / §2 / §5), assemblies/AGENTS.md (turned occurrences),
  robot/AGENTS.md, tests/AGENTS.md, the URDF / SRDF notes.

Measured (preview, scratch build of main): the forearm's least gap to the upper arm over the elbow's range at any roll
20.9 -> 19.3 mm (j2_link itself; the motor and board farther), the wrist vs the forearm 5.2 mm unchanged. Hash gate:
every part STEP unchanged; assemblies/arm.step and robot/links/forearm_link.step changed, wrist_pitch_link /
wrist_roll_link / jaw_a_link / jaw_b_link at float noise (their inertials and meshes match). ./cadtool pytest: 903 passed;
derive.py --check OK; validate URDF / SRDF / SDF OK.

File: cad/robot/arm.urdf (robot description, URDF)
Before this commit: robot arm, 10 links, 9 joints
Joints:
- joint wrist_pitch: origin xyz=0.016998 0 0.17 rpy=-1.570799 -1.271722 -1.570793 -> xyz=-0.016997 -0.000007 0.17 rpy=-1.570808 -1.271748 1.570808

Commit message: cad: the wrist-pitch motor 11.5 mm down the forearm - a 280-2GT wrist belt, no idler, its connector sideways
The wrist-pitch motor moves nearer the roll pulley, on a belt the user can buy: 280 is a multipack length (the 258 was
not), and at its centre distance it needs no idler - the motor's slots tension it. Previewed and approved first.

- lib/forearm/params.py: RollEndParams.wrist_belt 258 [ESTIMATE] -> 280 [DESIGN]: J2_MOTOR_SLIDE_X -99.522 -> -88.028
  (centre distance 70.478 -> 81.972). slide_range (-103.5, -94.0) -> (-94.0, -84.5): the same 9.5 mm of travel, 3.47
  past the belt's centre distance toward the wall to tension it, 6.03 back to slip it on; the slots follow (centre_x
  (-110, -88) -> (-100.5, -78.5), side_x (-119, -78.5) -> (-109.5, -69)). New motor_wall_clear 4.5
  (FOREARM_MOTOR_WALL_CLEAR): the body that far off the wall screws' heads at the slots' wall end - it replaces the
  plug-to-wall rule.
- lib/mounts.py: nema17_40mm#3's spin (180, 0, 90) -> (180, 0, 180): the connector from +X (at the wall, where its plug
  capped the slide at -94) to j2_link's -Y - sideways, away from the elbow axis with the forearm turned; toward the wrist
  its plug's room came within 5.3 mm of wrist_link. reference/placements.json: nema17_40mm#3 and mks_servo42d#3
  re-resolved.
- robot/arm.urdf / arm.sdf forearm_link (derive.py drafts): mass 0.635166 -> 0.635538 (the slots moved), COM (-0.005123,
  0.000008, 0.112869) -> (-0.005111, 0.000136, 0.107539), ixx 1.440981e-03 -> 1.553398e-03, ixy 2.482208e-07 ->
  3.050343e-06, ixz -1.291062e-04 -> -1.687204e-04, iyy 1.418477e-03 -> 1.530835e-03, iyz 5.993678e-08 ->
  1.779991e-06, izz 3.583121e-04 -> 3.586626e-04; meshes/forearm_link.stl re-exported; the ledger's stale "264-2GT".
- Tests: test_params_invariants / test_roll_end take the body-to-heads rule; test_wrist_motor_plug_room_is_clear (the
  connector sideways, plug_clearance of room beyond it clear of j2_link and the board) replaces
  test_wrist_motor_plug_clears_the_wall.
- Docs: docs/forearm_roll.md §4 (the motor stands in front of three of the wall's screw heads: take it off to reach
  them) and §5; docs/open_issues.md - the wrist belt's row now the tension with no idler, the connector row names the
  wrist motor's; tools/bom.py the belt's note.

Measured in the built arm: wrist motor <-> forearm_roll_pulley 21.9 -> 17.0 mm, its board 30.3 -> 18.9; motor <->
forearm_roll_block 29.4; motor <-> j3_coupler / wrist_link 10.5 -> 22.0; the body face to the wall 22.5 -> 11.0, to its
M3 heads 19.5 -> 8.0 (4.5 at the slots' wall end). Hash gate: parts/joints/j2_link.step, assemblies/arm.step and
robot/links/forearm_link.step changed, nothing else. ./cadtool pytest: 903 passed; derive.py --check OK; validate URDF /
SRDF / SDF OK.

File: cad/robot/arm.urdf (robot description, URDF)
Before this commit: robot arm, 10 links, 9 joints
Links:
- link forearm_link: mass 0.635166 -> 0.635538

Commit message: cad: the roll motor can go into its frame - a 6 mm shaft slit through the plate to the +N face, the pocket 1.5 mm deeper
Why: the roll motor could not be fitted. Its Ø22 pilot boss sits in the
plate's 22.3 mm pilot slot and its 22 mm shaft runs through the plate, while
the pocket left the motor and its board 1 mm of axial play: the boss could not
drop out of the slot, and the motor locked after 0.5 mm of slide toward the
open +N face. docs/forearm_roll.md's "the motor into the pocket from the +N
face onto the plate" had no path.

Now the motor and its board slide in from the +N face motor_drop (2.25) low -
the pilot boss under the plate, the shaft along the new slit - and lift into
the pilot slot. RollDriveParams: pocket_rear 1.0 -> 2.5 (the pocket's rear
z -29.75 -> -31.25), new motor_drop 2.25 and shaft_slit 6.0 (the slit from the
pilot slot out through the +N face; the tension slots stay whole, 8.3 mm either
side of it). lib/forearm/roll.py build_block cuts it.

Numbers: forearm_roll_block 393483.106 -> 388800.691 mm^3 (499.7 -> 493.8 g
PETG), native reference re-accepted (import_native.py --only
forearm_roll_block --force); forearm_roll_drive EXPECTED solid_volume
524411.105 -> 519728.69, stator 486150.457 -> 481468.042 (leaves / solids
unchanged). robot: elbow_link mass 0.928428 -> 0.922482 kg, COM (1.646,
-19.395, 19.084) -> (1.812, -19.520, 19.001) mm, inertias from the drafts
(arm.urdf, arm.sdf); its mesh re-exported; the arm 6.104 kg.
placements.json unchanged.

Tests: test_stack holds the axial play >= motor_drop > the pilot's height and
the slit clear of the tension slots; test_frame_features probes the slit; new
slow test_the_motor_slides_in_from_the_open_face moves the motor and board in
from outside the frame in 2 mm steps and lifts them: no overlap.

Docs: docs/forearm_roll.md (the pocket's station, the plate's slit, assembly
step 6); docs/open_issues.md's frame-flex row notes the slit splits the
plate's +N half.

Checks: hash gate - only forearm_roll_block, forearm_roll_drive, arm and
elbow_link changed; ./cadtool pytest: 946 passed; derive.py --check OK;
validate --strict OK (URDF, SRDF), SDF OK.

File: cad/robot/arm.urdf (robot description, URDF)
Before this commit: robot arm, 10 links, 9 joints
Links:
- link elbow_link: mass 0.928428 -> 0.922482

Commit message: cad: the roll pulley 8 mm nearer its motor on the stock belt with a tensioner, the motor 5 mm up under its 20T
Why: the roll frame read too big, with a wide gap between its face and the
belt. The forearm_roll_pulley sat where the 280-2GT belt put it, 81.97 from
the motor; the motor and so the frame's face sat low, the 20T's hub 3.5 off
the face and 7.5 off the motor's face. The belts are stock lengths only and
each gets a tensioner (cad/AGENTS.md "Belts", the previous commit but one),
so the roll's centre distance becomes a design value with an idler taking up
the rest of the 280 belt. Chosen from a to-scale preview: 74 (nearer than ~73
the idler meets the ring's flange and the belt's far run); the frame's round
end and the wall between the motor and the shaft's bay stay.

The drive (lib/forearm/params.py RollDriveParams):
- centre_distance: derived from roll_belt (81.972) -> a field, 74.0 [DESIGN];
  roll_belt stays 280. ELBOW_ROLL_OFFSET 81.972 -> 74: the forearm, the wrist
  and the gripper sit 7.97 nearer the elbow axis (lib/placements.py SHIFTS).
- pulley_lift 3.5 (the 20T's hub before the plate's face) -> pulley_seat 0.5
  (its hub over the motor's pilot boss, down in the plate's pilot slot): the
  motor's face 24.85 -> 29.85, the frame's front face 28.85 -> 33.85, the
  bearing boss 8.75 -> 3.75 proud of it, the face 9.75 -> 4.75 under the
  ring's flange; the motor's shaft tip now 3.85 past the forearm wall's plane.
- new RollIdlerParams (the tensioner): a gt2_idler_20t on the belt's back on
  the run back from the ring, along 31.7 from the motor, pushed in till the
  280 loop closes (lib/forearm/layout.py roll_belt_loop / roll_idler_xy);
  on a riser on the frame's face (12 wide, a 7 wide land on the idler's
  inner ring), an M5 x 25 down through the idler and the riser's slot (+/- 3
  along N) into an M5 nut in a channel under the face from the open +N face
  (roof 3). The idler 3.7 off the ring's flange, 6.6 off the belt's far run
  (3.8 at the slot's deep end), the nut's channel 2.8 off the motor's pocket.

Parts: new roll_idler_screw (M5 x 25, 739.958 mm^3, 5.8 g) and roll_idler_nut
(M5, 168.216 mm^3, 1.3 g), purchased with no reference (lib/reference.py
NO_REFERENCE, tests/forearm/test_roll_idler.py locks them); gt2_idler_20t is
placed (its UNPLACED and its tools/bom.py EXTRAS row dropped). lib/fasteners.py
M5_PITCH 0.8. The drive's rows: the idler, the screw, the nut.

Numbers: forearm_roll_block 388800.691 -> 397064.588 mm^3 (493.8 -> 504.3 g
PETG), bbox 83 x 159.972 x 82.6 -> 83 x 152.0 x 83.8 (8 mm shorter), native
reference re-accepted; forearm_roll_belt's band 1059.993 -> 1059.849 mm^3,
its bbox 117.738 -> 109.766 long. forearm_roll_drive EXPECTED leaves 9 -> 12,
solids 24 -> 27, solid_volume 519728.69 -> 530037.771; stator 7 / 22 /
481468.042 -> 10 / 25 / 491777.123. The arm: 91 -> 94 leaves, 253 -> 256
solids, 55 -> 58 bought; tools/bom.py 33 -> 36 bought parts, 55 -> 58 pieces.
placements.json: mount_placements.py re-ran (every mounted record past the
elbow shifts). robot: forearm_roll origin y -0.081972 -> -0.074 (arm.urdf,
arm.sdf); elbow_link mass 0.922482 -> 0.945106 kg, COM (1.812, -19.520,
19.001) -> (4.211, -17.470, 19.125) mm, inertias from the drafts, its mesh
re-exported; the arm 6.104 -> 6.127 kg. The elbow's lower limit: the elbow
motor's board 4.6 -> 5.9 mm off the frame at -47 deg, its 1 mm line -51.0 ->
-54.0 deg (lib/params.py, docs/open_issues.md).

Tests: test_stack (the 20T on the pilot boss, the centre distance a design
value the stock belt is longer than), test_frame_features (the boss probe over
the new face), test_forearm_clears_the_elbow_while_rolling (the motor's shaft
and the tensioner's screw head pass the wall's plane: the rolling forearm stays
2 mm or more inside their radius about the roll axis), the module colours;
test_belts (the roll loop round its idler); test_wrist_idler (the idler is
placed, the wrist kit's axle and nut stay unplaced); new
tests/forearm/test_roll_idler.py (the loop, the clearances, the riser, slot
and channel on the frame, the kit's fit, the hardware's numbers).

Docs: docs/forearm_roll.md (the drive's belt and tensioner, the stations, the
riser, assembly step 6), docs/open_issues.md (the two belt-tensioner rows made
one: the roll's is designed; the elbow-limit row), robot/AGENTS.md, the URDF
ledger.

Checks: hash gate - forearm_roll_block, forearm_roll_belt, forearm_roll_drive,
arm and elbow_link changed; forearm_link, wrist_pitch_link, wrist_roll_link and
the jaw links' STEPs rewrite with float noise (their inertials and meshes check
unchanged); ./cadtool pytest: 962 passed; derive.py --check OK; validate
--strict OK (URDF, SRDF), SDF OK; ./cadtool lint clean.

File: cad/robot/arm.urdf (robot description, URDF)
Before this commit: robot arm, 10 links, 9 joints
Links:
- link elbow_link: mass 0.922482 -> 0.945106
Joints:
- joint forearm_roll: origin xyz=0.000001 -0.081972 0.025 rpy=3.141593 -1.570795 0 -> xyz=0.000001 -0.074 0.025 rpy=3.141593 -1.570795 0
