Commit message: cad: the roll frame 6 mm thinner, still symmetric - +/-30 about the roll axis, flush with the forearm's round wall
The roll frame (forearm_roll_block) was the widest thing at the elbow along the elbow axis: 66 mm, its
faces 3-4 mm past the round parts that turn about the roll axis (the forearm wall's Ø60, the 90T's
Ø59.2 flanges, the belt). ROLL_FRAME_R 33 -> 30 brings the underside, the open +N face and the tower
top in together, so the frame stays symmetric about the roll axis with the bearing boss centred on
its front face, and now lines up with the forearm wall's radius (wall_od / 2, held by test_stack).

The underside can only rise: the elbow flange under it stays where j1_link's bore and recess put it,
so the Ø72 lip runs up to the new underside (lip_x -35..-30, 2 -> 5 mm tall) and the frame sits
6.0 mm over j1_link's flat top instead of 3.0. The motor, its pocket (x_cradle -23), both 6806s, the
belt, the tensioner, the nuts and the M4 tips stay put. The tower's corners tighten (tower_corner_r
6 -> 3) so the Ø52 bearing boss stays 1 mm inside them on the flat of the front face.

Measured:
- frame along N 66 -> 60 mm; volume 397064.588 -> 360226.836 mm^3 (-36837.752); mass at
  PETG_DENSITY 504.3 -> 457.5 g; bbox 83.0 x 152.0 x 83.8 -> 80.0 x 149.0 x 83.8
- floor under the motor (web_t) 10 -> 7; wall round the shaft's bay 7.4 -> 4.4 (>= 3); round the
  bearing seats 11.9 -> 8.9 (>= 4); the boss 7 -> 4 inside the frame's three sides
- the roll motor's connector ends 2 inside the open pocket (was 5)
- forearm_roll_drive EXPECTED solid_volume 530037.771 -> 493200.019, stator 491777.123 -> 454939.371
  (rotor unchanged 38260.648); the arm's solid volume 3079935.4 -> 3043097.7 mm^3
- elbow_link mass 0.945106 -> 0.898322 kg, COM (0.004211, -0.01747, 0.019125) ->
  (0.004299, -0.015957, 0.018784) m, inertia re-derived (arm.urdf, arm.sdf); its mesh re-exported
  (solids 34, 481610.0 mm^3)

The native reference reference/native/forearm_roll_block.step is re-accepted (import_native.py
--force). Hash gate: only forearm_roll_block, forearm_roll_drive, arm and elbow_link changed.
Full suite green (962 tests), URDF / SRDF / SDF valid, derive.py --check OK.

File: cad/robot/arm.urdf (robot description, URDF)
Before this commit: robot arm, 10 links, 9 joints
Links:
- link elbow_link: mass 0.945106 -> 0.898322

Commit message: cad: an idler on the elbow belt in j1_link's old slit, the elbow motor 3.97 mm nearer the elbow
The elbow belt was the one belt with no tension adjustment: its motor sat on round holes at exactly
the stock 280 belt's centre distance (81.97), the loop 0.04 mm tight. Every belt gets a tensioner
(cad/AGENTS.md "Belts"), and j1_link's SolidWorks slit - 47 mm from the elbow axis, across both
strands - was for one. A stock 300 does not fit this span (taking up 20 mm puts the idler 0.5 mm
off the far strand) and the motor has no room toward the shoulder (its hole 1.8 mm off the drive's
shell), so the belt stays 280 and the motor moves in:

- ELBOW_MOTOR_CENTRES 81.97 -> 78.0 [DESIGN] (pad.x 88.03 -> 92.0): the open loop 272.41, so the
  280 has 7.6 mm for the idler to take up.
- ElbowIdlerParams: a gt2_idler_20t (gt2_idler_20t#1) on the belt's back, on the 90T -> 20T run, on
  the slit's line, pushed in till the loop is 280 (lib/belts.py idler_on_run): its axis 5.5 off the
  link's centre line, 10.5 off the far strand. Its slots run z -2.3 .. 22.7 (25 mm), so the one
  idler takes any belt from 272.4 to 288.5 mm, the 280 in the middle.
- The mount: the slab's underside is the face j1_link prints on, so the riser the roll frame grows
  is a printed spacer here (elbow_idler_spacer: a 12 riser, a 7 x 1 land on the bearing's inner
  ring, 3.2 tall). An M5 x 25 SHCS (elbow_idler_screw) goes up from under the idler through it and an
  M5 slot in a 6.5 floor into an M5 nut (elbow_idler_nut) in an 8.2 slot down from the slab's top
  face: the nut drops in from above and slides with the screw, which is turned from below. The
  stepped slot (4 wide through, a 10 wide counterbore from below) is gone from DEFAULT; LEGACY keeps
  it for the reference match.
- 20T wrap 148 -> 177 deg, 90T 212 -> 238 deg.

Measured:
- the elbow motor's board to the roll frame at the elbow's -47 deg limit 5.9 -> 2.3 mm, its 1 mm
  line -54.0 -> -49.0 deg (docs/open_issues.md); the idler 8.5 or more off the 90T and 14.1 off the
  20T anywhere in its slot; over the shoulder's range the elbow motor stays the part nearest the
  fork (21.1 -> 22.5 mm), the forearm and gripper 30.7 off the motor and the kit at the elbow's limits
- j1_link (DEFAULT) volume 368453.715 -> 372731.723 mm^3
- elbow_belt volume 1059.993 -> 1059.849 mm^3, bbox x 117.738 -> 113.766
- upper_arm_link mass 1.300888 -> 1.318719 kg, COM (0.059178, 0.000068, 0.03399) ->
  (0.060926, 0.000074, 0.033582) m, inertia as arm.urdf / arm.sdf; its mesh re-exported
- the arm: leaves 94 -> 98, solids 256 -> 260, bought / printed leaves 58 / 36 -> 61 / 37;
  placements.json 66 -> 70 part records, 159 -> 163 solids; the print list 29 parts / 36 pieces ->
  30 / 37, the buy list 36 / 58 -> 38 / 61
- new parts, no reference (tests/upper_arm/test_elbow_idler.py locks them): elbow_idler_spacer
  (printed, 211.273 mm^3), elbow_idler_screw (M5 x 25, 739.958 mm^3, 5.8 g), elbow_idler_nut (M5,
  168.216 mm^3, 1.3 g); gt2_idler_20t now x2

Checks: the hash gate (only j1_link, elbow_belt and arm changed, plus the three new parts),
./cadtool pytest green, derive.py --check OK, validate --strict on arm.urdf / arm.srdf, arm.sdf OK,
lint clean.

File: cad/robot/arm.urdf (robot description, URDF)
Before this commit: robot arm, 10 links, 9 joints
Links:
- link upper_arm_link: mass 1.300888 -> 1.318719

Commit message: cad: the base_yaw belt a 400 round an idler on the motor mount, the motor 48.93 mm further out
The base_yaw belt was the last running belt tensioned only by its motor's slots, and every belt gets an idler
(cad/AGENTS.md "Belts"). The stock 300 left no room for one. At its own centre distance (73.07) the exact loop was
already 0.23 longer than the belt. The motor could come only ~0.4 mm nearer the axis before its slots met the base's
posts. The one spot an idler fits, 1.6 - 3.4 off the 120T's flange, lies under the base's cap over the motor's face,
where no key reaches. The options were previewed before / after (renders at one scale, an overlay, the whole arm), and
the choice is a stock 400 with the motor further out and the elbow's kit on the mount's plate:

- YAW_BELT 300 -> 400 [DESIGN]. The motor's centre goes from centre_distance(300), 73.067, to YAW_MOTOR_X 122.0
  [DESIGN], on round holes: MOTOR_TRAVEL's +/-2.5 slots are gone and the window is the pilot's, +/-11.2. The open loop
  is 392.35, so the 400 leaves 7.65 for the idler.
- YawIdlerParams: a gt2_idler_20t (gt2_idler_20t#2) on the belt's back on the 120T -> 20T run. It sits 85.0 out from
  the axis on the belt's centre line, pushed in till the loop is 400 (lib/belts.py idler_on_run). Its axis is 2.96
  across the belt, 12.45 off the far strand, 20.1 off the 20T's flange and 36.9 off the 120T's.
- Its slot runs across the belt from -3.1 (3.0 off the far strand's teeth) to 24.1 (1.0 past touching the open strand).
  The one idler takes any belt from 392.4 to 405.3.
- The kit is the elbow's turned over: the mount stands on the table, so the screw is turned from above.
  - yaw_idler_spacer, printed, 4.3 tall: a 12 riser and a 7 x 1 land on the bearing's inner ring, on the plate's top.
  - yaw_idler_screw, an M5 x 25 SHCS, head-up on the idler. It runs down through the spacer and an M5 slot in the
    mount's 5 mm plate into yaw_idler_nut, an M5 nut under the plate; its tip ends 2.0 past the nut.
  - The nut is held flats-on between two rails grown down from the plate's underside: 8.2 apart, 3 thick, 5 deep,
    closed past the slot's ends.
- The mount follows the motor (mount_x1): its end wall moves 108.57 -> 157.50 from the axis, 57.5 past the foot's Ø200.
- A single truss V on the longer side walls would bridge ~40 mm in print plate-down; the limit is 30. So a wall wider
  than MountParams.bay (60) now splits into equal bays with a strut-wide post between. The side walls get two bays
  each (~17 mm bridges); the end wall keeps one (~26).
- 20T wrap 128.3 -> 180.5 deg, 120T wrap 231.7 -> 224.8 deg.
- lib/base/layout.py: yaw_belt_loop() takes the idler. yaw_belt_point() maps the belt's frame into the base's; the
  frame turns with the motor's 0.084 z. New: yaw_idler_xz(), yaw_idler_slot(), yaw_idler_y(), yaw_idler_spacer_h().
- lib/params.py: YAW_IDLER_Y -35.6, YAW_IDLER_SPACER_H 4.3, YAW_IDLER_NUT_Y -44.9, and the kit's masses.

Measured:
- base_motor_mount volume 52094.084 -> 83593.493 mm^3; its reference/native STEP re-accepted.
- base (DEFAULT) volume 413503.0 -> 413546.135 mm^3: the old slots no longer cut its plate past the joint.
- yaw_belt volume 1136.33 -> 1513.449 mm^3, bbox x 118.382 -> 167.315.
- base_link mass 1.166795 -> 1.220127 kg, COM (-0.028237, -0.000037, 0.050838) -> (-0.050249, -0.000005,
  0.051267) m; inertia as arm.urdf / arm.sdf; its mesh re-exported.
- The arm: leaves 98 -> 102, solids 260 -> 264, bought / printed leaves 61 / 37 -> 64 / 38.
- placements.json: 70 -> 74 part records, 163 -> 167 solids, volume 2097446.332 -> 2131677.733.
- The print list 30 parts / 37 pieces -> 31 / 38; the buy list 38 / 61 -> 40 / 64.
- New parts with no reference, locked by tests/base/test_yaw_idler.py: yaw_idler_spacer (printed, 309.545 mm^3),
  yaw_idler_screw (M5 x 25, 739.958 mm^3, 5.8 g), yaw_idler_nut (M5, 168.216 mm^3, 1.3 g). gt2_idler_20t is now x3.

docs/open_issues.md:
- Closed: the "base_yaw motor's hold" row. The motor is on round holes, the idler takes the tension, and the slots no
  longer cross the joint.
- The tensioner row now leaves only the wrist belt.
- The idler-land row adds the base's spacer.
- The base print row's bridges are now ~17 / ~26.

Checks:
- The hash gate: only base, base_motor_mount, yaw_belt, arm and robot/links/base_link changed, plus the three new parts.
- ./cadtool pytest green (1006, the base_yaw sweep round the longer mount included).
- derive.py --check OK; validate --strict OK on arm.urdf and arm.srdf, arm.sdf OK; lint clean.

File: cad/robot/arm.urdf (robot description, URDF)
Before this commit: robot arm, 10 links, 9 joints
Links:
- link base_link: mass 1.166795 -> 1.220127

Commit message: cad: the wrist roll drive - the pancake on the wrist-pitch axis, a 2:1 belt to a 40T on a 6806 pair beside it, the gripper bolted to it; the bracket dropped
The pancake and gripper_clamp_bracket hung 66-90 mm out past the wrist-pitch axis on wrist_link's tower, the gripper
direct-driven beyond them through the 20T its connector slid onto. The wrist now copies the elbow: the pancake sits ON
the wrist_pitch axis, centred on it, on the wrist plate's free face (the forearm's boss and the coupler fill the other
side), and belts 2:1 (WRIST_ROLL_RATIO, its 20T to a printed 40T) to a roll axis R' beside it - WRIST_ROLL_OFFSET
48.583 across the pitch axis in the wrist's swing plane, WRIST_ROLL_AXIS_H 27 over the plate's coupler face (44 off the
SolidWorks roll axis). The wrist is therefore no longer spherical: the wrist_roll axis misses the pitch axis and the
forearm roll's - an IK in software/control must be numeric (docs/open_issues.md).

- assemblies/wrist_roll_drive.py, a designed module like forearm_roll_drive (lib/mounts.py ModuleMount on wrist_link#1,
  turned with it - ModuleMount.turned, new: a module beyond the forearm's turn). Stator: the pancake (its plug spun to
  the open face), its 20T, the 6806-2RS pair back to back on a 2 mm lip, the belt (wrist_roll_belt, the stock 158-2GT at
  its centre distance, the pancake at its slots' middle). Rotor: wrist_roll_pulley (hub through bearing 2, the 40T band,
  the face the gripper's connector bolts to) and wrist_roll_shaft (hub through bearing 1, the rotor clamp's nuts, the
  stop lug) clamped by 4x M3 x 35, a Ø10 bore through both for the gripper servo's cable. EXPECTED: 7 leaves, 19
  solids, 70790.837 mm3 (stator 5 / 17 / 44991.257, rotor 2 / 2 / 25799.58).
- wrist_link IS the frame (lib/wrist/: WristRollParams, stack_positions, roll.py build_frame / build_pulley / build_shaft):
  DEFAULT keeps the plate's round end and j3_coupler#2's seat and adds the pancake's pocket (open on the far face, the
  plate in front slotted along the belt for its tension, the shaft's slit), the tower round R' (the seats, the lip, the
  bearing boss, the shaft's bay open on the far face with the stop's post) and a hex channel from the bay down to the
  one coupler nut the tower covers; the old tower and its end face go. LEGACY (the reference match) is unchanged.
  wrist_link 72321 -> 72402 mm3; wrist_roll_pulley 16178.7, wrist_roll_shaft 9620.9 (no reference, NO_REFERENCE).
- gripper_j3_connector converted (lib/wrist/connector.py): LEGACY reproduces the SolidWorks part (4713.0 vs 4713.027
  mm3, its 20-tooth bore as the circle of its area); DEFAULT bolts to the pulley's face - a hub, 4x M3 x 10 on Ø36 into
  nuts in the face, notches over the plate's holes for the servo holder's and cover's screws, the cable bore - one
  solid, 10308.5 mm3 (MULTI_BODY entry gone, its "not converted" row too).
- gripper_clamp_bracket dropped: part, reference STEP, CUSTOM row, manifest and README rows go, "brack for hand cmap" is
  SKIPPED_PRODUCTS and mount_placements.py moved its record to `skipped`; nema17_pancake#1 and gt2_pulley_20t#1 RETIRED.
  The gripper moves onto R' by one LinkShift (wrist_roll_drive: along -83.196, across 48.583, normal -44) in place of
  the wrist's -20 shortening shift. placements.json expected 70 / 163 / 2097446.332 -> 69 / 162 / 2086270.734.
- Robot: WRIST_ROLL_ORIGIN carried onto R' with the gripper (the axis unchanged, parallel); LINKS - wrist_pitch_link
  takes the stator, wrist_roll_link the rotor (no 20T#1). wrist_roll origin (0.089643, 0.000005, -0.016998) ->
  (0.026448, -0.048578, 0.027003); wrist_pitch_link 0.41432 -> 0.461415 kg, wrist_roll_link 0.16664 -> 0.198512 kg;
  both meshes re-exported.
- Limits: WRIST_PITCH_LIMITS_DEG (-105, 70) -> (-75, 125) - the tower's rear (stepped in behind the bay, z_tower_rear)
  stays 1.49 mm off the wrist-pitch motor's board at -75 and touches at -77, any roll; a finger meets that motor near
  +129 at roll 0 / 180. WRIST_ROLL_LIMIT_DEG 180 -> 166, 2 deg short of the printed stop at +/-168.66. The gripper rolls
  3.4 mm or more off the wrist and the forearm.
- What wrist_pitch carries: 698 -> 777 g, its centre of mass 88.9 -> 43.0 mm off the pitch axis, the static moment on
  the wrist-pitch motor 0.609 -> 0.328 N.m (1.014 -> 0.625 with 200 g at tool0); tool0 206.6 mm out along the roll axis
  -> 143.4 along R', 48.6 across, 44.0 up (151.4 off the pitch axis).
- No idler on this belt yet: the forearm roll's kit (its M5 nut in a channel under the frame's face) finds no room
  between the pocket, the pancake's screws, its pilot slot and the tower's seats; the pancake's slots tension it
  (docs/open_issues.md, as the wrist-pitch belt).
- lib/geom.py gains the belt drives' box / stop_wedge / slot_y / nut_slot (lifted from lib/forearm/roll.py, a pure move:
  the forearm roll's STEPs rebuild byte-identical).
- Locks: the arm 98 -> 102 leaves, 260 -> 263 solids, tints 61 / 37 -> 64 / 38; the print list 30 / 37 -> 31 / 38, the
  buy list 38 / 61 -> 39 / 64, bearing_6806 8 -> 10; the belt locks (wrist_roll_belt 598.693 mm3).
- Tests: tests/wrist/test_roll_drive.py (module frame and record, the stack, the stock belt, the rotor's walls, the
  connector's turn, totals, colours, presses, clean pairs against wrist_link, the rotor clear, the pancake's way in),
  tests/wrist/test_connector.py, wrist_link's DEFAULT probes, test_sweeps' wrist roll stop and gripper-rolling checks.
- Docs: docs/wrist_roll.md (new); cad/AGENTS.md, robot/, assemblies/, lib/, parts/, tests/ AGENTS.md; docs/forearm_roll.md
  and every statement of a spherical wrist (frames.py, arm.urdf / .srdf, forearm params); open_issues rows - the
  wrist-pitch range rewritten, the IK (a wrist offset), the belt's missing idler, the frame's flex, wrist_link's print
  orientation, the wrist roll's cable route and home sensor; the bracket and connector rows gone.

File: cad/robot/arm.urdf (robot description, URDF)
Before this commit: robot arm, 10 links, 9 joints
Links:
- link wrist_pitch_link: mass 0.41432 -> 0.461415
- link wrist_roll_link: mass 0.16664 -> 0.198512
Joints:
- joint wrist_pitch: limit lower=-1.832596 upper=1.22173 effort=5 velocity=1 -> lower=-1.308997 upper=2.181662 effort=5 velocity=1
- joint wrist_roll: limit lower=-3.141593 upper=3.141593 effort=1 velocity=2 -> lower=-2.897247 upper=2.897247 effort=1 velocity=2; origin xyz=0.089643 0.000005 -0.016998 rpy=-1.570799 -0.055534 -1.570796 -> xyz=0.026448 -0.048578 0.027003 rpy=-1.570799 -0.055534 -1.570796

Commit message: cad: j2_link an L at the wall, 5 mm shorter, a straight web and a Ø60 wrist boss
The forearm web (j2_link) takes the profile chosen on a preview page, in three rounds:

- The flange wall stops flush with the web's belt face, so the side profile is an L (the web and the wall on its
  motor side): its 13 mm belt-side stub is gone. The bottom wall screw's hole (Ø3.4 at z 9.5) would break out 0.2 mm
  under that face, so it keeps a Ø9 boss (RollEndParams.screw_boss_dia), its lower edge on the Ø40 recess's line
  (z 5). The gussets stay. Wall z -5..55 -> 8..55 (the boss down to z 5).
- SHORTENING 40 -> 45: elbow axis to wrist axis 170 -> 165. The wrist-pitch motor keeps the stock 280 belt's centre
  distance (81.97) and slides 5 mm toward the wall: motor_x -88.03 -> -83.03, slide (-94, -84.5) -> (-89, -81.5),
  slots centre_x (-100.5, -78.5) -> (-95.5, -75.0), side_x (-109.5, -69.0) -> (-104.5, -66.0); motor_wall_clear
  4.5 -> 1.5 (the wall screws were already reached with the motor off), so the tension travel past the belt's length
  is 1.5 (3.5) and the bottom screw's channel 19.0 (22.5) - the screw and its head exactly.
- The web no longer tapers from the Ø90 boss to the 60 mm wall: it runs straight, as wide as the wall (DEFAULT
  web.half_w 30). RollEndParams.neck_half_w, layout.neck_tangent() and web_half_width() go; link.straight_web()
  replaces necked_web().
- The wrist boss Ø90 -> Ø60, as wide as the web: its top drops 33.5 -> 27.5 to the bearing seat's top and the Ø80
  recess goes (WristBossParams.recess_dia may be None). j3_coupler's dust lip turns 0.5 over the top, its Ø78 flange
  4.5 over it - the same 0.5 running gap as before; 8.9 of wall round the Ø42.2 seat (23.9).

j2_link: 173186.8 -> 90018.6 mm^3, 219.9 -> 114.3 g solid PETG; 167 x 90 x 60 -> 147 x 60 x 50. Its own weight at
the elbow, forearm level: 0.295 -> 0.127 N.m.
forearm_link (arm.urdf / arm.sdf): mass 0.645638 -> 0.540015 kg; COM (-0.004707, 0.000135, 0.107419) ->
(-0.006961, 0.000162, 0.093197); ixx 1.563251e-03 -> 9.128842e-04, iyy 1.546627e-03 -> 9.615967e-04,
izz 3.663589e-04 -> 2.562004e-04, ixy 3.077238e-06 -> 2.876961e-06, ixz -1.672173e-04 -> -1.076438e-04,
iyz 1.777065e-06 -> 9.537962e-07. wrist_pitch origin z 0.17 -> 0.165. Arm total 6.23 -> 6.125 kg.
reference/placements.json: the mounted records regenerated (tools/reference/mount_placements.py) - the wrist bearings,
pulley, screws, nuts, motor, board, 20T and belt, and the wrist roll drive, follow the 5 mm.
robot/meshes/forearm_link.stl re-exported.
Locks: the wrist slide's tension room >= 3.0 -> >= 1.5 (tests/test_params_invariants.py);
tests/forearm/test_roll_end.py rewritten for the straight web, the cut wall and the boss.

Hash gate against main (same machine): j2_link, arm and forearm_link changed; wrist_pitch_link, wrist_roll_link and
jaw_a_link float noise (inspect diff: same geometry). ./cadtool pytest: 1040 passed. derive.py --check clean;
validate --strict OK (urdf, srdf; sdf --gz-check never).

File: cad/robot/arm.urdf (robot description, URDF)
Before this commit: robot arm, 10 links, 9 joints
Links:
- link forearm_link: mass 0.645638 -> 0.540015
Joints:
- joint wrist_pitch: origin xyz=-0.016997 -0.000007 0.17 rpy=-1.570808 -1.271748 1.570808 -> xyz=-0.016997 -0.000007 0.165 rpy=-1.570808 -1.271748 1.570808

Commit message: cad: j2_link's wall round again where forearm_roll_pulley seats
The L cut (the previous commit) stopped the flange wall at the web's belt face (z 8), but forearm_roll_pulley's
Ø59.19 ring, fastened to the wall's elbow face, reaches z -4.6. So the wall's straight edge ran across the pulley's
round face 12.6 above its bottom, the Ø40 locating recess broke out through that edge, and the bottom screw's Ø9 boss
hung below it as a lug. Chosen on a preview page over a 4 mm round lip with the L behind it: the wall is round again
all the way down - the hull of the Ø60 flange and the web's end section, as before the cut - so it covers the pulley's
ring all round, the recess is closed and the bottom screw's hole is inside the wall. RollEndParams.screw_boss_dia
goes; wall_outline() no longer cuts. Wall z 5..55 (its boss) -> -5..55. The straight web, the Ø60 wrist boss,
SHORTENING 45 and the motor slide stay.

j2_link: 90018.6 -> 93707.4 mm^3, 114.3 -> 119.0 g solid PETG; 147 x 60 x 50 -> 147 x 60 x 60.
forearm_link (arm.urdf / arm.sdf): mass 0.540015 -> 0.544699 kg; COM (-0.006961, 0.000162, 0.093197) ->
(-0.006709, 0.00016, 0.092843); ixx 9.128842e-04 -> 9.215829e-04, iyy 9.615967e-04 -> 9.735226e-04,
izz 2.562004e-04 -> 2.610379e-04, ixy 2.876961e-06 -> 2.899190e-06, ixz -1.076438e-04 -> -1.020476e-04,
iyz 9.537962e-07 -> 9.225217e-07. Arm total 6.125 -> 6.129 kg.
robot/meshes/forearm_link.stl re-exported; reference/placements.json unchanged (mount_placements.py run).
tests/forearm/test_roll_end.py: the boss probes out, the wall's belly back (bbox min Z -5, the recess closed).

Hash gate against the previous commit's build (same machine): j2_link, arm and forearm_link changed, nothing else.
./cadtool pytest: 1040 passed. derive.py --check clean; validate --strict OK (urdf, srdf; sdf --gz-check never).

File: cad/robot/arm.urdf (robot description, URDF)
Before this commit: robot arm, 10 links, 9 joints
Links:
- link forearm_link: mass 0.540015 -> 0.544699
