Commit message: cad: j1_motor_leg bolted to the motor plate's sleeve by 3 radial M4s
The motor plate's sleeve only slid in j1_motor_leg's ring (Ø70 in Ø70.4, 0.2 a
side) and nothing else held the plate: the output pins start at z 12, short of
its inner face at z 9, and the plate turns freely in its 6814. So the motor's
reaction torque reached the fork through friction alone.

Now 3 radial M4 x 20 (ForkParams.sleeve_screw_len) go through the leg's ring in
its middle (drive z -18, coupler x 42: lib/cycloidal/layout.py sleeve_bolt_z)
at the motor's flats - up and both sides, none down where the leg's post
stands (ShellParams.sleeve_bolt_deg) - heads on the ring's od (r 45; an M4 head
rocks 0.14 there, no seat), into M4 nuts pressed into lugs on the sleeve's
bore: 12 wide (sleeve_lug_w), from r 22.5 (sleeve_lug_r, 1.35 off the motor's
flats), 10 long from the sleeve's end (sleeve_lug_len), then 45 deg out to the
bore so the plate still prints on its inner face without support; each nut's
hex pocket from the lug's face out to r 28.2, 6.85 AF (sleeve_nut_af,
j3_coupler's press fit: the pocket opens toward the motor), flats across the
axis. The screws' ends are flush with the nuts' inner faces (sleeve_nut_r 25),
3.85 off the motor's flats. The leg's holes are 4.4 wide and 5.0 long along the
axis (sleeve_slot_len): the screws float +/-0.5 there, 1.5 of ring either side,
so the drive settles lengthwise - the hub's leg holds it - before they lock
it, and the fork never loads the 6814s along the axis. Two axial layouts (a lip
inside or outside the leg, 4 M4s into the sleeve's end) were drawn up and set
aside for this one.

The screws and nuts are not modelled (as the hub's and the foot's): two new
cycloidal_drive rows in tools/bom.py EXTRAS, 3 M4 x 20 + 3 M4 nuts
(lib/params.py CYCLOIDAL_SLEEVE_BOLT_COUNT 3, locked).

Numbers:
- j1_motor_leg 44,356.285 -> 43,831.851 mm^3 (56.3 -> 55.7 g PETG), bbox unchanged
- cycloidal_motor_plate 72,414.182 -> 75,642.270 mm^3 (92.0 -> 96.1 g), bbox unchanged
- assemblies/cycloidal_drive.py EXPECTED solid_volume 551,156.383 -> 554,384.471,
  stator 407,955.132 -> 411,183.220 (leaves / solids unchanged, rotor unchanged)
- reference/placements.json expected solid_volume 2,120,502.135 -> 2,119,977.701,
  j1_motor_leg#1's record 44,356.285 -> 43,831.851
- shoulder_link (arm.urdf, arm.sdf, meshes/shoulder_link.stl): mass 1.370307 -> 1.373741 kg,
  COM (-0.00075, 0.014225, -0.022097) -> (-0.000754, 0.014281, -0.022022) m,
  ixx 3.791606e-03 -> 3.797012e-03, iyy 2.836825e-03 -> 2.841720e-03,
  izz 2.065815e-03 -> 2.068940e-03, ixy 5.872290e-05 -> 5.875498e-05,
  ixz 2.273055e-05 -> 2.287850e-05, iyz -4.403984e-04 -> -4.427168e-04 kg m^2
- the plate's best print orientation (inner face down): faces under 45 deg
  65.8 -> 489.9 mm^2 (the lugs' 45 deg chamfers and the pockets' 4 mm bridges);
  each pocket closed toward the sleeve's end by a 0.575 skin (docs/open_issues.md)

Checks: the hash gate (87 STEPs; only j1_motor_leg, cycloidal_motor_plate,
cycloidal_drive, arm and robot/links/shoulder_link changed, the docstring-only
edits byte-identical), ./cadtool pytest 1042 passed, ./cadtool lint, validate
arm.urdf / arm.srdf --strict and arm.sdf, derive.py --check. Scratch checks:
no clash between the leg, the plate, the motor, its board, the shell ring, the
6814 and j1_coupler; a driver (Ø6 shaft, Ø22 handle) reaches each screw clear
of the arm at every shoulder angle in 5 deg steps, 2.0 outboard of the turning
shell; the upper arm stays 23.0 off the leg over the shoulder's range.

File: cad/robot/arm.urdf (robot description, URDF)
Before this commit: robot arm, 10 links, 9 joints
Links:
- link shoulder_link: mass 1.370307 -> 1.373741

Commit message: cad: a tensioner on the wrist belt - the motor 1.97 mm nearer the wrist on round holes, the idler under the web
Every belt gets a tensioner (cad/AGENTS.md "Belts"); the wrist belt was the last on j2_link still tensioned by its
motor's slots. An idler only ever lengthens the belt's path, so the stock 280 needs its motor nearer the wrist than the
belt's own centre distance - as previewed and approved:

- lib/forearm/params.py: WRIST_MOTOR_CENTRES 80.0 [DESIGN] (the 280's own 81.97 less 1.97); DEFAULT's motor_x
  -83.028 -> -85.0 (lib/params.py J2_MOTOR_SLIDE_X -> J2_MOTOR_X, J2_MOTOR_SLIDE_RANGE gone, WRIST_MOTOR_CENTRES
  re-exported) on round holes - MotorHoleParams (the Ø22.3 pilot, 4x M3 clearance on the 31 mm square) replaces the
  slots (ForearmConfig.slot / slide_range None; LEGACY keeps the SolidWorks slide); DEFAULT.idler = IdlerParams():
  the kit it kept since cad/forearm-flip, its +/- travel now a slot between slot_y's ends (4.7, 21.0) - in 4 past the
  stock belt's place, out 1 past just touching the open loop. The idler sits along 24 from the motor, pushed 11.32 into
  the loop; the open loop at 80.0 is 276.25, so the slot takes belts 276.25 .. 283.15.
- lib/forearm/link.py: round holes (or the slide), the idler's rib, slot and nut channel along slot_y; layout.py
  screw_channel runs into the pilot hole.
- lib/mounts.py WRIST_IDLER_MOUNTS: gt2_idler_20t#3, wrist_idler_screw#1, wrist_idler_nut#1 on j2_link (their
  placements.json records, arm.py rows and GROUPS, robot/frames.py forearm_link); the two M5 parts lose UNPLACED.
- lib/params.py WRIST_PITCH_LIMITS_DEG (-75, 125) -> (-74, 125): with the motor nearer, wrist_link's frame comes 0.44 mm
  off its board at -75 (was 1.49), 1.56 at -74; the sweeps (elbow, shoulder, gripper roll) clear with the idler in.
- j2_link: 93707.4 -> 99011.9 mm3 (119.0 -> 125.7 g PETG: the slots filled, the rib). wrist_belt: the 280 round the
  idler, exactly 280.000 (was the plain pair's 280.038); its band 1059.993 -> 1059.849 mm3, bbox size x 117.738 ->
  115.766.
- Locks: placements expected 73 -> 76 leaves, 166 -> 169 solids, solid_volume 2119977.701 -> 2121924.71; the arm 106
  -> 109 leaves, 267 -> 270 solids, bought leaves 67 -> 70; BOM 106 -> 109 occurrences, bought (41, 67) -> (43, 70); test_belts the wrist band; tests/forearm/test_wrist_idler.py rewritten for
  the placed kit (the stock belt round it, the band its slot takes, the stations, its slot and channel on j2_link, the
  kit's fit), test_roll_end / test_params_invariants / test_mounts for the round holes.
- robot/arm.urdf / arm.sdf: forearm_link mass 0.544699 -> 0.562795, COM (-0.006709, 0.00016, 0.092843) -> (-0.005892,
  0.00004, 0.094125), ixx 9.215829e-04 -> 9.153113e-04, iyy 9.735226e-04 -> 9.783129e-04, izz 2.610379e-04 ->
  2.748673e-04, ixy 2.899190e-06 -> 5.220259e-06, ixz -1.020476e-04 -> -9.961750e-05, iyz 9.225217e-07 ->
  1.818290e-06; wrist_pitch lower -1.308997 -> -1.291544; meshes/forearm_link.stl re-exported.
- Docs: docs/forearm_roll.md §4-5, docs/open_issues.md (the wrist belt's no-idler row closed; the tensioner, the lands
  and the wrist-pitch limit rows), lib/AGENTS.md, tests/AGENTS.md, assemblies/AGENTS.md.

File: cad/robot/arm.urdf (robot description, URDF)
Before this commit: robot arm, 10 links, 9 joints
Links:
- link forearm_link: mass 0.544699 -> 0.562795
Joints:
- joint wrist_pitch: limit lower=-1.308997 upper=2.181662 effort=5 velocity=1 -> lower=-1.291544 upper=2.181662 effort=5 velocity=1

Commit message: cad: room for the MKS boards' plugs - the elbow and wrist boards turned, the roll frame slotted
Every MKS SERVO42D board's plugs stay in as the arm moves, so each needs straight room out from its
headers at every pose: 10 mm at the two side headers, 5 mm at the motor cable's (measured on the bench).
lib/motors.py now carries the three headers' outlines from vendor/mks_servo42d.step
(MKS_SERVO42D_HEADERS) and that room (MKS_PLUG_ROOM); tests/test_sweeps.py
test_the_mks_boards_keep_their_plug_room sweeps each board against everything that moves relative to it.

Swept on main (worst pose, -X / +X / motor plug, mm): base yaw 11.2 / 11.0 / >=30 and the drive's board
>=30 everywhere - clear; the elbow board 6.9 (the drive's shell ring) / 6.8 (the roll frame at elbow -47)
/ >=30, the roll board 4.25 / 4.3 (its pocket's walls) / >=30, the wrist board 9.7 (the roll tensioner's
M5 head, forearm roll +79..+104) / 21.3 / 22.1 - short.

- A board bolts on through its motor's square screw pattern, so it can sit at any quarter turn
  (lib/mounts.py board_frame(turn_deg), BOARD_TURNS): the elbow board turned 90 deg - side plugs >=30, the
  motor plug 7.6 at the elbow's lower limit (12.5 from -33 up); the wrist board 270 deg - side plugs
  25.2 / 20.4, the motor plug 9.7 at forearm roll +84..+104. reference/placements.json: the
  mks_servo42d#2 / #3 records turned.
- No turn frees the roll board (each leaves a plug 2.5-4.3 off a wall or the pocket's floor):
  forearm_roll_block gets a plug slot off each side of its motor pocket (lib/forearm/layout.py
  plug_slots(): RollDriveParams.plug_clear 0.5 round each header, MKS_PLUG_ROOM past its face with the
  motor at the tension slide's far end and plug_spare 1.0 more - 13.5 past the face -, open through the
  +N face, so the motor goes in with its cables plugged); 3.9 of the round end and 9.1 under the tower
  left outside them. Block 360226.836 -> 353860.986 mm3 (reference/native/forearm_roll_block.step
  re-accepted); assemblies/forearm_roll_drive.py EXPECTED solid_volume 493200.019 -> 486834.169, stator
  454939.371 -> 448573.521.
- Inertials (robot/arm.urdf, arm.sdf): elbow_link 0.898322 -> 0.890238 kg, its COM and inertia;
  upper_arm_link and forearm_link COM and inertia (masses unchanged); the three links' meshes re-exported.
- Docs: docs/forearm_roll.md (the slots, the motor going in plugged), parts/joints/mks_servo42d.py (the
  headers), tests/AGENTS.md.

Checked: the hash gate (only forearm_roll_block, forearm_roll_drive, arm and the three links' STEPs
changed), ruff clean, ./cadtool pytest 1047 passed, URDF / SRDF / SDF validate, derive.py --check OK.

File: cad/robot/arm.urdf (robot description, URDF)
Before this commit: robot arm, 10 links, 9 joints
Links:
- link elbow_link: mass 0.898322 -> 0.890238

Commit message: cad: model the j1_coupler fork's screws and nuts
The screws and nuts that hold the cycloidal drive in j1_coupler's fork were only
tools/bom.py EXTRAS rows: on the buy list, absent from the model, the totals and the
inertials, so the fork showed empty counterbores and slots. They are now purchased
pattern parts with no reference (lib/reference.py NO_REFERENCE), mounted like the
base_yaw pulley's (lib/mounts.py FORK_MOUNTS, in shoulder_link, joint shoulder_pitch):

- fork_hub_screws / fork_hub_nuts: 4x M4 x 25 from the hub leg's counterbores along the
  drive's axis into the nuts captive in the output hub's flange, tips flush with them;
  hosted on j1_coupler#1
- fork_foot_screws / fork_foot_nuts: 2x M4 x 10 from j1_motor_leg's foot into the nuts
  in the disc's slots, 0.7 past them; hosted on j1_motor_leg#1
- fork_sleeve_screws / fork_sleeve_nuts: 3x M4 x 20 radially from the ring's od into the
  nuts pressed into the motor plate sleeve's lugs, tips flush; hosted on j1_motor_leg#1

No printed geometry changes: every frame comes from the fork's existing numbers
(lib/yaw_coupler/layout.py fork_*_screw_frame / _points / _nut_z, the sleeve's radial
pieces placed by lib/yaw_coupler/body.py toward_axis). The six EXTRAS rows go; EXTRAS
keeps no M4 row.

Measured:
- placements.json expected: leaf occurrences 76 -> 82, solids 169 -> 187, solid volume
  2121924.71 -> 2126292.027 mm^3 (+4367.3)
- masses (lib/params.py FORK_*_MASS_G, the modelled steel): hub screws 14.2 g, hub nuts
  3.0, foot screws 4.1, foot nuts 1.5, sleeve screws 9.2, sleeve nuts 2.3 - 34.3 g
- shoulder_link inertial: mass 1.373741 -> 1.408024 kg, COM (-0.000754, 0.014281,
  -0.022022) -> (-0.000741, 0.014089, -0.021707) m, ixx 3.797012e-03 -> 3.898356e-03,
  iyy 2.841720e-03 -> 2.908733e-03, izz 2.068940e-03 -> 2.137678e-03, ixy 5.875498e-05
  -> 6.098559e-05, ixz 2.287850e-05 -> 2.177568e-05, iyz -4.427168e-04 -> -4.257543e-04
  (arm.urdf / arm.sdf; robot/meshes/shoulder_link.stl re-exported); URDF total 6.177 kg
- the sleeve nuts' press in the lugs' 6.85 AF pockets: 3 x 3.2 deep, budgeted in
  test_motors_and_boards_clear_their_neighbours; the hub's and the foot's nuts are a
  slip fit (zero overlap)
- arm.step: leaves 109 -> 115, solids 270 -> 288, bought leaves 70 -> 76 (printed 39)
- BOM: bought parts 43 -> 49 (70 -> 76 occurrences), EXTRAS 18 -> 12 rows

Tests: tests/base/test_fork_bolts.py locks the six parts (pieces, volume, bbox, the
screws on their stations, the nuts' corners where their seats have them);
tests/test_mounts.py test_the_fork_bolts_reach_their_nuts (the arithmetic in the drive's
frame) and test_the_fork_bolts_hold_the_drive (the heads and nuts on their seats, the
designed press); j1_motor_leg#1 joins the neighbours of the interference sweep.
Hash gate: only assemblies/arm.step and robot/links/shoulder_link.step changed.

File: cad/robot/arm.urdf (robot description, URDF)
Before this commit: robot arm, 10 links, 9 joints
Links:
- link shoulder_link: mass 1.373741 -> 1.408024

Commit message: cad: model the wrist-pitch motor's 4x M3, heads flush in counterbores under j2_link's web
The wrist-pitch motor (nema17_40mm#3) stood on j2_link's four plain Ø3.4 holes with nothing holding it. The user asked
for its screws to be modelled, in counterbores, and picked flush heads with M3 x 12 (over a 2 mm deeper counterbore
with M3 x 10, whose counterbore would have come 1.55 mm from the wrist idler nut's channel along 2 mm of its height).
It is the elbow motor's screw and seat: j2_link's web is 11 thick, like the web under the elbow motor.

- New purchased part wrist_motor_screws (parts/joints/): 4x M3 x 12 SHCS (ISO 4762), lib/fasteners.py shcs(). It is a
  pattern part with no reference (lib/reference.py NO_REFERENCE), like elbow_motor_screws, and its pattern is
  lib/forearm/layout.py motor_hole_points() (new: the 31 mm square about the motor's axis, which j2_link's holes now
  use too).
- lib/forearm/params.py MotorHoleParams: screw (M3_SHCS), pocket_dia 5.7 (the drive motor plate's head pockets, the
  elbow's), thread 4.0 (bolt_hole_depth 4.5 - the drive's 0.5 margin). lib/params.py J2_MOTOR_SCREW_LEN = web 11 -
  head_h 3 + thread 4 = 12, WRIST_MOTOR_SCREWS_MASS_G 4.68 g.
- lib/forearm/link.py: four Ø5.7 x 3.0 counterbores in the web's underside (DEFAULT only; LEGACY's slide has none).
- lib/mounts.py MOTOR_SCREW_MOUNTS: wrist_motor_screws#1 hosted on j2_link#1 at (J2_MOTOR_X, 0, 11), +Z up j2_link's
  +Z; MOTOR_SCREWS is now both parts (AXES). placements.json rewritten by mount_placements.py. assemblies/arm.py
  OCCURRENCES and the forearm_link group, robot/frames.py LINKS.

Clearances (scratch build, then the in-place test): no overlap with j2_link, the motor (0.10 radial in its Ø3.2
holes, 4.0 of its 4.5 deep holes), its 20T (11.2), the wrist idler (3.2 under the heads), its screw (5.6) or its nut
(3.6). The idler's Ø18 flange passes under the -x +y head (9 % of it, its socket 0.45 clear in plan), so the screws go
in before the idler (docs/forearm_roll.md, the part's docstring).

Numbers:
- j2_link: volume 99011.936 -> 98814.675 mm^3 (125.75 -> 125.49 g PETG), faces 54 -> 62.
- wrist_motor_screws: 4 solids, 596.246 mm^3, bbox min (-18.25, -18.25, -3), size (36.5, 36.5, 15).
- placements expected: leaf_occurrences 76 -> 77, solids 169 -> 173, solid_volume 2121924.71 -> 2122520.956.
- arm: leaves 109 -> 110, solids 270 -> 274, bought leaves 70 -> 71.
- BOM: occurrences 109 -> 110, bought (parts, pieces) (43, 70) -> (44, 71); the new buy row "M3 x 12 socket head cap
  screw (ISO 4762)", 4 pieces, envelope.
- forearm_link inertial (robot/arm.urdf, arm.sdf; meshes/forearm_link.stl re-exported):
  - mass 0.562795 -> 0.567225 kg;
  - COM (-0.005892, -0.00005, 0.094012) -> (-0.00576, -0.000049, 0.093942);
  - ixx 9.164659e-04 -> 9.189617e-04, iyy 9.789843e-04 -> 9.817487e-04, izz 2.753505e-04 -> 2.777577e-04;
  - ixy 3.211444e-06 -> 3.207921e-06, ixz -1.021093e-04 -> -1.014419e-04, iyz 1.275165e-06 -> 1.277050e-06;
  - the URDF's total 6.143 -> 6.147 kg.

Tests:
- tests/forearm/test_wrist_motor_screws.py (new): the part's numbers, the elbow motor's screw / counterbore / thread,
  the counterbores clear of the idler nut's channel (1.55 across, below its floor), probed on j2_link, the heads flush
  in place and no interference with the motor, its 20T or the idler kit.
- tests/test_mounts.py: the elbow motor's screw test now covers both motors (parametrized).
- tests/test_bom.py: both motors' buy rows; the counts. test_parts_convention MULTI_BODY wrist_motor_screws 4;
  test_placements and test_assembly the counts above.

Docs: docs/forearm_roll.md, tests/AGENTS.md, lib/AGENTS.md, robot/AGENTS.md (the forearm_link row, which now also
lists the wrist belt's idler kit it was missing).

File: cad/robot/arm.urdf (robot description, URDF)
Before this commit: robot arm, 10 links, 9 joints
Links:
- link forearm_link: mass 0.562795 -> 0.567225

Commit message: cad: the wrist roll's MKS board on the pancake, wrist_link's pocket open behind it
The wrist-roll pancake was the only stepper on the arm without its MKS SERVO42D. The board's
encoder reads a magnet on the motor's rear shaft end, so it can only sit on the pancake's rear
face - where wrist_link's pocket had its rear wall. That wall goes: a window takes the board
(chosen over enclosing the board in a deeper pocket, after a preview).

- The board: a wrist_roll_drive stator row on the pancake's rear face, turned with it
  (motor_spin_deg 90: its motor plug toward the pancake's connector at the open face, the side
  plugs along the belt).
- The window (lib/wrist/layout.py board_window): the board's housing square (board_w 43) + the
  tension travel (pad_slot_len 5) + board_clear 0.45 either side, from the frame's rear to
  board_clear in front of the pancake's rear face (the housing starts at that face), open on +X
  like the pocket, so the motor and its board go in together. board_clear rather than
  pocket_clear 0.75: the window's wall to the shaft's bay keeps 1.53 (the frame's rule 1.5; 1.98
  before, over the bay's lowest 1.55 mm).
- The frame's rear behind the pocket comes up to the tower's: z_rear -16.25 -> -14.6
  (z_tower_rear folded into it). The rims the window would leave either side sat 0.15 mm inside
  the side plugs' MKS_PLUG_ROOM.

Measured: wrist_link 72402.0 -> 65566.9 mm^3 (92.0 -> 83.3 g PETG). The board 0.45 off the
window at both ends of the slide, 0.50 off the plate's free face, its back 11.0 behind the
frame's rear; its side plugs' rooms 1.5 off the frame; board and plug rooms more than 15 mm off
the forearm over the wrist pitch range, the board 9.62 off the roll shaft.

Locks: wrist_roll_drive EXPECTED leaves 7 -> 8, solids 19 -> 32, volume 70790.837 -> 84570.171
(stator 5 -> 6, 17 -> 30, 44991.257 -> 58770.592); arm leaves 109 -> 110, solids 270 -> 283,
bought leaves 70 -> 71; BOM bought pieces 70 -> 71. wrist_pitch_link mass 0.461415 -> 0.487734 kg
(COM and inertia re-derived, URDF and SDF), the arm 6.143 -> 6.169 kg; its mesh re-exported.

Tests: the window and the board's seat and turn, the motor and board sliding in together and at
the slide's ends, KIT_OVERLAP 317.7 mm^3 (the board's M3 x 30 run through the pancake's own M3 in
the same holes), a wrist_pitch_link entry in the plug-room sweep.

Open (docs/open_issues.md): the board's screw length on a pancake (the kit's M3 x 30 reach
MKS_SERVO42D_SCREW_REACH into a 23 mm body; ~M3 x 25 likely), wrist_roll added to the CAN-id
row, the frame-flex row notes the open rear.

File: cad/robot/arm.urdf (robot description, URDF)
Before this commit: robot arm, 10 links, 9 joints
Links:
- link wrist_pitch_link: mass 0.461415 -> 0.487734
