Commit message: cad: base_motor_mount becomes the base's other half - full width to a round end, the foot round it, slits round both
The motor mount looked out of place beside the base: an upright box with V-truss walls and ears, next to a base that
leans out at 10.8 degrees on a chamfered foot. The new shape was chosen on rendered previews, in three rounds: the
base's D carried on at full width to a matching round end, the foot all round, the joint bolts inside; then plain
slits through the walls (not framed windows with grills: they print without bridges), as an even ring.

The mount (lib/base/body.py build_motor_mount):
- The walls are the base's leaning planes carried on past the joint face, shell.wall (5) thick, to a round end about
  mount_end_x() - the base's round half mirrored, its radius the walls' at each height (64.63 at the plate's top,
  78.36 at the table). The end reaches mount_x1() at the plate's top: 157.5 -> 158.5, now that the wall is the base's 5
  (was MountParams.wall 4).
- The foot carries on round it (the flange to r 100 and the chamfer, flush with the base's at the joint), with 4 more
  M5 holes and spot-faces (FootParams.mount_hole_deg, the base's round half's mirrored).
- The ears are gone. Two posts at the joint face (MountParams.post_t 8, from the window out to the wall) mirror the
  base's; the 4 M4 run through both, the heads on the mount's posts' inner faces, turned from underneath with the base
  off the table. The bolt pattern is unchanged (JointParams.bolt_out 10 keeps z +/- 41.58), so the base's holes and
  nut pockets, the screws and the nuts are the same.
- The truss is gone: MountParams loses wall, ear_w, ear_t, strut and bay; layout.py truss_panels(), body.py _strut()
  and _truss_windows() are removed.
- Its plate, the motor's seat and the idler's seat are unchanged; the idler's rails are now clipped to the walls'
  inside.

The slits (new SlitParams, layout.py slit_band() / slits(), body.py _slit_cuts()), in the base and the mount: 3 x 32
with round ends, cut straight across through the wall, in one band 28 to 60 above the table (4 over the foot's
chamfer, 7.1 under the plate). 10 mm pitch along the wall: 22 round each round end and the straight sides at multiples
of 10 from the axis, none within 2 of the two parts' posts (x 45 to 65). 30 in the base, 26 in the mount. The slits
are too narrow for fingers: the board's plugs are still reached from underneath.

Measured:
- base: 413546.1 -> 399435.1 mm^3 (525.2 -> 507.3 g PETG solid), bbox unchanged.
- base_motor_mount: 83593.5 -> 282427.5 mm^3 (106.2 -> 358.7 g), bbox 102.5 x 72.1 x 95.167 -> 138.87 x 72.1 x 200;
  it reaches 157.5 -> 193.87 from the base_yaw axis. The MKS board is 10.0 -> 16.77 from it; the motor, the belt,
  the idler and the screws are as before (belt 5.8, idler 4.3).
- reference/native/base_motor_mount.step re-accepted (tools/reference/import_native.py --force), its manifest entry
  with it.
- reference/placements.json (mount_placements.py): expected solid_volume 2121924.71 -> 2320758.692.
- base_link (arm.urdf and arm.sdf): mass 1.220127 -> 1.454725 kg, COM (-50.249, -0.005, 51.267) ->
  (-62.693, -0.003, 46.427) mm, ixx / iyy / izz 3.075990e-3 / 7.334967e-3 / 7.781149e-3 -> 4.362671e-3 /
  8.839905e-3 / 9.979556e-3, ixy / ixz / iyz 9.613928e-6 / -3.536246e-4 / 1.404988e-6 -> 9.710122e-6 /
  -8.264923e-4 / 1.412202e-6. robot/meshes/base_link.stl re-exported.

Tests: tests/base/test_motor_mount.py rewritten for the new mount (its outline the base's carried on, flush at the
joint, the round end and its foot holes, the posts and bolts, every slit cut in both parts); test_foot.py's volume
lock and one side probe moved between two slits; test_base.py and test_yaw_idler.py follow the renamed fields.

docs/open_issues.md: the joint row names the posts and the heads' way in; the print row says the mount, printed plate
down, has its foot on top - the chamfer at ~50 degrees from vertical and the flange's rim want supports.

File: cad/robot/arm.urdf (robot description, URDF)
Before this commit: robot arm, 10 links, 9 joints
Links:
- link base_link: mass 1.220127 -> 1.454725

Commit message: cad: the roll motor's 4x M3 x 8, heads flush in counterbores in a 7 mm plate; the motor 3 mm back, no slide
The forearm roll motor (nema17_40mm:forearm_roll) hung on four tension slots in the roll frame's 4 mm plate with no
screws modelled. The user asked for its screws, in counterbores, and said the motor need not slide: the idler on the
frame's face already tensions the roll belt. A 4 mm plate cannot take a 3 mm counterbore, so the user picked, from four
options (preview page first), the motor 3 mm back with the plate grown to 7 mm toward it - over 5 mm back (M3 x 10),
7 mm back (M3 x 12, the elbow / wrist screw, but a 1.5 mm plug-slot wall and the 20T 2 mm off the shaft's tip) and
pads on the front face (the heads 3 mm proud of it).

- lib/forearm/params.py RollDriveParams: pad_t 4 -> 7 (4 under the heads + head_h), pulley_seat 0.5 -> 3.5 (the front
  face, the 20T and the belt stay; the motor's face goes back 3); the slide's pad_slot_len, pad_bolt_dia and
  pad_pilot_w are gone, replaced by motor_holes: MotorHoleParams - the wrist-pitch motor's round holes, Ø5.7 x 3
  counterbores and 4.0 thread (the elbow motor's), its docstring now covering both motors.
- lib/forearm/layout.py: stack_positions z_motor_screws (the counterbores' floor, z_front - head_h); motor_pocket and
  plug_slots lose the slide's +/- 2.5.
- lib/forearm/roll.py build_block: the Ø22.3 pilot hole and four Ø3.4 holes, each with its Ø5.7 x 3 counterbore from
  the front face, in place of the five slots (slot_y no longer imported).
- New purchased part roll_motor_screws (parts/joints/): 4x M3 x 8 SHCS (ISO 4762), lib/fasteners.py shcs(), a
  pattern part with no reference (lib/reference.py NO_REFERENCE), like wrist_motor_screws; lib/params.py
  ROLL_MOTOR_SCREW_LEN = pad_t - head_h + thread = 8, ROLL_MOTOR_SCREWS_MASS_G 3.79 g. Its row in
  assemblies/forearm_roll_drive.py (on the motor's axis at z_motor_screws, turned over: heads up), so the stator
  (elbow_link) carries it. tools/bom.py: the EXTRAS row "M3 x 8 ... the roll motor to the frame's plate" goes - the
  screws are a modelled buy row now.
- reference/native/forearm_roll_block.step re-accepted (tools/reference/import_native.py --only forearm_roll_block
  --force) and its manifest entry.

Clearances (scratch build, then the in-place test): no overlap of the screws with the frame, the motor (0.10 radial in
its tapped holes, 4.0 of their 4.5), the 20T (11.2), the belt (6.5), the idler (11.6), its screw or nut (15.0); the
board 0.75 off the pocket's walls (was 1.5 with the slide room); the thinnest wall at a plug slot 3.92 -> 4.12; the
idler nut's channel 2.75 -> 5.25 off the pocket; the shaft's tip 51.85 -> 48.85, 2.05 past the 20T's end and still past
the forearm wall's plane. The motor still slides in from the open +N face (test_the_motor_slides_in_from_the_open_face).

Numbers:
- forearm_roll_block: volume 353860.986 -> 367622.565 mm^3 (449.4 -> 466.9 g PETG), bbox unchanged (80 x 149 x 83.8).
- Stations: z_motor_face 29.85 -> 26.85, z_motor_board -9.65 -> -12.65, z_motor_screws 30.85 (new); the pocket
  +/- 24.75 -> +/- 22.25 in y, its rear -26.25 -> -29.25; each plug slot 13.5 -> 11.0 long.
- roll_motor_screws: 4 solids, 483.148 mm^3, bbox min (-18.25, -18.25, -3), size (36.5, 36.5, 11).
- forearm_roll_drive EXPECTED: leaves 12 -> 13, solids 27 -> 31, solid_volume 486834.169 -> 501078.896; stator leaves
  10 -> 11, solids 25 -> 29, solid_volume 448573.521 -> 462818.248; rotor unchanged.
- arm: leaves 117 -> 118, solids 305 -> 309, bought leaves 78 -> 79.
- BOM: occurrences 117 -> 118, bought (parts, pieces) (50, 78) -> (51, 79); the new buy row "M3 x 8 socket head cap
  screw (ISO 4762)", 4 pieces, envelope; one EXTRAS row fewer.
- elbow_link inertial (robot/arm.urdf, arm.sdf; meshes/elbow_link.stl re-exported):
  - mass 0.890238 -> 0.911507 kg;
  - COM (0.004506, -0.016091, 0.018623) -> (0.004063, -0.015717, 0.018835);
  - ixx 1.459372e-03 -> 1.484110e-03, iyy 7.619559e-04 -> 7.672604e-04, izz 1.416372e-03 -> 1.432633e-03;
  - ixy 1.418712e-04 -> 1.481999e-04, ixz -2.059059e-05 -> -1.948857e-05, iyz 6.973625e-05 -> 6.670557e-05;
  - the URDF's total 6.443 -> 6.464 kg.

Hash gate (against the main checkout's STEPs, same machine): changed as meant - forearm_roll_block,
forearm_roll_drive, arm, robot/links/elbow_link (+ the new roll_motor_screws). base_link, shoulder_link, forearm_link
and wrist_pitch_link also differ, but main's copies predate its last merges (cadgen reads them STALE there); this
change touches only the drive's stator. placements.json unchanged (mount_placements.py).

Tests:
- tests/forearm/test_roll_motor_screws.py (new): the part's numbers, the elbow / wrist motors' head, counterbore and
  thread through a 7 mm plate (M3 x 8), the stations, the round holes and counterbores probed on the frame (no slide),
  the heads flush in the module and clear of everything in it.
- tests/forearm/test_roll_drive.py: the pocket without the slide, the slit between the counterbores, the module's
  colours (10 bought leaves); tests/test_bom.py: the counts, the roll drive's buy list, the three motors' screw rows;
  test_parts_convention MULTI_BODY roll_motor_screws 4; test_assembly the counts above.

Docs: docs/forearm_roll.md (the frame row, the pocket / plug slot / plate stations, the assembly step, the links),
docs/open_issues.md (the 20T's seat row no longer quotes 0.5), tests/AGENTS.md, lib/AGENTS.md, robot/AGENTS.md (the
elbow_link row), robot/frames.py's elbow_link comment.

File: cad/robot/arm.urdf (robot description, URDF)
Before this commit: robot arm, 10 links, 9 joints
Links:
- link elbow_link: mass 0.890238 -> 0.911507

Commit message: cad: the base_yaw motor's 4x M3 x 8, heads flush in counterbores, on a 2 mm pad; the pilot in a round hole
The base_yaw motor (nema17_48mm#1) hung under base_motor_mount's 5 mm plate on four plain Ø3.4 holes with no screws
modelled, its pilot in a square 22.4 window. The user asked for its screws, counterbored, and for the pilot to sit in a
round cutout like the drive motor's. A 5 mm plate leaves 2 mm under a 3 mm counterbore, so the user picked, from three
options (preview page first), a 2 mm pad under the plate round the motor's face with the motor 2 mm lower - 4 under
the heads and the roll motor's M3 x 8 - over keeping the 5 mm plate (2 under the heads, M3 x 6) and a 4 mm pad (6 under
the heads, M3 x 10, the board 1 mm off the table); and a round through hole over a stepped one: the 20T's hub dips
2.2 mm into the plate, so a blind pilot recess like the drive plate's is not possible.

- lib/base/params.py MotorParams: holes (MotorHoleParams, the wrist and roll motors' seat: the Ø22.3 pilot hole, Ø3.4
  holes, Ø5.7 x 3 counterbores, M3, 4.0 of thread) and pad_t, both None / 0 on LEGACY; DEFAULT takes them
  (YAW_MOTOR_PAD 2.0). WINDOW_CLEAR and DEFAULT's window_x / window_half_z are gone (the window is LEGACY's only).
  BOARD_CLEAR 5.0 -> 3.0 with the pad in the bottom face's sum, so the bottom face stays at -112.0.
- lib/base/layout.py: motor_face_y() (the pad's underside, -46.9) and motor_screw_y() (the counterbores' floor, -42.9).
- lib/base/body.py _motor_seat: with motor.holes, the pad (the NEMA 17 face's 42.3 square), the round pilot hole and the
  four holes through plate and pad, each counterbored from the plate's top.
- lib/params.py: BASE_MOTOR_PATTERN_CENTRE on the pad's face; YAW_MOTOR_SCREW_Y, YAW_MOTOR_SCREW_LEN (8) and
  YAW_MOTOR_SCREWS_MASS_G (3.79 g) new.
- New purchased part yaw_motor_screws (parts/base/): 4x M3 x 8 SHCS (ISO 4762), a pattern part with no reference
  (lib/reference.py NO_REFERENCE), like roll_motor_screws. lib/mounts.py MOTOR_SCREW_MOUNTS: yaw_motor_screws#1 hosted on
  base_motor_mount#1 at (122, -42.9, 0.084), +Z down the base's -Y; MOTOR_SCREWS (AXES) takes it. assemblies/arm.py
  OCCURRENCES and the base_link group, robot/frames.py LINKS. placements.json rewritten by mount_placements.py.
- reference/native/base_motor_mount.step re-accepted (tools/reference/import_native.py --only base_motor_mount --force)
  and its manifest entry.

Clearances (scratch build, then the tests in place): no overlap of the screws with the mount; the screws 11.17 from the
20T, 5.97 from the belt, 13.84 from the idler, 16.16 / 19.66 / 17.65 from its spacer, screw and nut. The 20T's hub 3.15
clear of the pilot hole all round (3.2 to the old window's flats). The screws' thread in the vendor motor's tapped holes
(modelled at the M3 minor diameter, the screws at the major) is 37.05 mm^3 - the drive's motor bolts' budget, now in
test_motors_and_boards_clear_their_neighbours. The board 3.0 above the table (was 5.0), 17.1 from the mount; the 20T
stays level with the 120T, 2 mm further up the shaft: its hub face 2.85 -> 4.85 from the motor's face, the shaft's tip
2.7 past its top (was 4.7).

Numbers:
- base_motor_mount: volume 282427.475 -> 285510.96 mm^3 (358.68 -> 362.60 g PETG), bbox unchanged (138.87 x 72.1 x 200).
- Stations: BASE_MOTOR_PATTERN_CENTRE y -44.9 -> -46.9, BASE_MOTOR_TABLE_CLEAR 5.0 -> 3.0, BASE_MOTOR_20T_HUB_Z
  2.85 -> 4.85; YAW_MOTOR_SCREW_Y -42.9 (new).
- yaw_motor_screws: 4 solids, 483.148 mm^3, bbox min (-18.25, -18.25, -3), size (36.5, 36.5, 11).
- placements expected: leaf_occurrences 83 -> 84, solids 191 -> 195, solid_volume 2325722.255 -> 2329288.888.
- arm: leaves 118 -> 119, solids 309 -> 313, bought leaves 79 -> 80.
- BOM: occurrences 118 -> 119, bought (parts, occurrences) (51, 79) -> (52, 80); the new buy row "M3 x 8 socket head
  cap screw (ISO 4762)", 4 pieces, envelope.
- base_link inertial (robot/arm.urdf, arm.sdf; meshes/base_link.stl re-exported):
  - mass 1.454725 -> 1.462434 kg;
  - COM (-0.062693, -0.000003, 0.046427) -> (-0.063005, -0.000003, 0.045942);
  - ixx 4.362671e-03 -> 4.378077e-03, iyy 8.839905e-03 -> 8.882283e-03, izz 9.979556e-03 -> 1.000960e-02;
  - ixy 9.710122e-06 -> 9.749555e-06, ixz -8.264923e-04 -> -8.682607e-04, iyz 1.412202e-06 -> 1.486790e-06;
  - the URDF's total 6.464 -> 6.471 kg.

Hash gate (against the main checkout's STEPs, same machine): changed as meant - base_motor_mount, arm, robot/links/
base_link (+ the new yaw_motor_screws). base.step's bytes differ too (its plate runs through _motor_seat before the
lobe is cut off at the joint): ./cadtool inspect diff reads the same geometry (tol 1e-6).

Tests:
- tests/base/test_yaw_motor_screws.py (new): the part's numbers, the roll motor's screw in the wrist motor's
  counterbores through the plate and its pad (M3 x 8, 4 under the heads, 4.0 of thread), the heads flush in place and
  clear of the mount, the board, the 20T, the belt and the idler kit.
- tests/base/test_motor_mount.py: the seat (the round pilot hole, the pad, the counterbores - probed on the mount), the
  motor, its screws and its 20T clear of the mount.
- tests/test_mounts.py: the motor-screw test covers the base_yaw motor (parametrized); the screws' thread in the motor
  is a designed overlap. tests/base/test_base.py: the pattern centre on the pad's face. tests/test_bom.py: the buy row,
  the counts; test_parts_convention MULTI_BODY yaw_motor_screws 4; test_placements, test_assembly and
  test_yaw_pulley_bolts the counts above.

Docs: robot/AGENTS.md (the base_yaw and base_link rows), lib/AGENTS.md, tests/AGENTS.md, base_motor_mount's docstring.

File: cad/robot/arm.urdf (robot description, URDF)
Before this commit: robot arm, 10 links, 9 joints
Links:
- link base_link: mass 1.454725 -> 1.462434

Commit message: cad: the elbow pulley 90T -> 108T on a stock 300 belt (5.4:1), its idler 1.9 mm nearer the motor
Why: more torque at the elbow, which is short of holding the forearm level. A bigger driven pulley is the step that
needs no new stage. With the elbow motor where it is (ELBOW_MOTOR_CENTRES 78, its board 2.3 mm off the roll frame at
the elbow's lower limit), 108 teeth is the most the stock belts and the tensioner rules of
tests/upper_arm/test_elbow_idler.py take: a 110T leaves the 300 only 3.35 mm over its open loop, and 115T or more needs
the motor nearer the elbow. Chosen from a to-scale preview (scratch build, before / after renders, overlay).

The pulley: gt2_pulley_108t (parts/joints/), lib/pulley/params.py ELBOW = DEFAULT with GT2_PULLEY_108T_TEETH and its
rim's inside grown with the teeth (rim_dia 53 -> 64.459156, the 90T's wall kept), as YAW is for the 120T. The hub,
web height, bore and M4 holes are the 90T's, so it takes the same mount frame on the lower elbow bearing
(gt2_pulley_108t#1 replaces gt2_pulley_90t#3, still hosted on the retired gt2_pulley_90t#1 and turned
pulley_bolt_deg) and the same elbow_pulley_screws / _nuts. No reference file (lib/reference.py NO_REFERENCE); its
numbers are in tests/pulley/test_gt2_pulley_108t.py. Flange Ø59.188 -> Ø70.647; volume 23975.641 -> 31390.961 mm^3
(30.4 -> 39.9 g in PETG). Role elbow_pitch (label gt2_pulley_108t:elbow_pitch); the wrist's 90T keeps j3.
ELBOW_RATIO = GT2_PULLEY_108T_TEETH / GT2_PULLEY_20T_TEETH = 5.4 in lib/params.py, the elbow's reduction in
robot/AGENTS.md and robot/frames.py; GT2_RATIO (4.5) is now the wrist's alone. Elbow torque about 1.1-1.8 ->
1.3-2.2 N·m, still under the ~2.4 static (URDF masses) - docs/open_issues.md keeps the second-stage row open.

The belt: ELBOW_BELT 280 -> 300 (in both multipacks; the belts are now 2x 280, 1x 300, 1x 400, 1x 158). Open loop
272.4 -> 294.2. elbow_belt volume 1059.849 -> 1135.449 mm^3.

The tensioner: the idler's line gets its own parameter, ElbowIdlerParams.along = 29.1 from the motor's axis
(lib/upper_arm/layout.py elbow_idler_x()), 1.9 nearer the motor than the stepped slot's line (x 123 -> 121.1), so its
flange keeps 5.0 off the 108T's pitch circle at the slots' inner end. slot_z (-2.3, 22.7) -> (-4.0, 25.1): in to 3.0
off the far strand's teeth, out past touching the open loop's strand. On the 300 the idler sits at z 9.857 (was
5.545). The slot takes 294.2 .. 315.7 (was 272.4 .. 288.5): the stock belt 5.8 above the open loop and 15.7 under the
longest. Fit: the idler's flange 5.56 off the 108T's flange at its place (8.73 off the 90T's), 4.74 at the slot's
inner end, 4.58 nearest (z 0) - test_the_kit_fits asks 5.0 at the place and PULLEY_CLEAR_AT_ENDS 4.5 at the slot's
ends (was 5.0 at both ends). The nut's slot 3.4 off the motor's hole (was 5.3; the rule is 3.0); the idler 4.4 off
the motor's screw heads (was 7.4), its nut 4.1 off the motor body (was 6.0). The pulley stays 3.0 under j1_link.
j1_link volume 372731.723 -> 372030.418 mm^3 (the slots 4.1 longer).

Numbers that changed:
- placements.json expected solid_volume 2329288.888 -> 2336779.808 (the mounted records regenerated by
  tools/reference/mount_placements.py).
- print list: 32 -> 33 parts (39 to print, unchanged: the 90T 2 -> 1, the 108T 1).
- upper_arm_link: mass 1.318719 -> 1.317978 kg, COM (0.060964, 0.000026, 0.033582) -> (0.060932, -0.000006,
  0.033589), ixx 1.684041e-03 -> 1.684781e-03, ixy -1.394608e-06 -> 1.175714e-06, ixz 7.519974e-04 ->
  7.513569e-04, iyy 6.389485e-03 -> 6.388052e-03, iyz -1.297730e-06 -> -2.876412e-06, izz 6.775386e-03 ->
  6.774821e-03; mesh re-exported (66 solids, 610827.3 mm^3).
- elbow_link: mass 0.911507 -> 0.920925 kg, COM (0.004063, -0.015717, 0.018835) -> (0.004021, -0.015556,
  0.018202), ixx 1.484110e-03 -> 1.527059e-03, ixy 1.481999e-04 -> 1.487957e-04, ixz -1.948857e-05 ->
  -2.183490e-05, iyy 7.672604e-04 -> 8.080608e-04, iyz 6.670557e-05 -> 7.577451e-05, izz 1.432633e-03 ->
  1.444870e-03; mesh re-exported (38 solids, 496904.2 mm^3).
- the robot: 6.471 -> 6.480 kg.

The hash gate names arm.step, j1_link.step, elbow_belt.step and the upper_arm_link / elbow_link link STEPs (+ the
new gt2_pulley_108t.step); every other part STEP byte-identical. derive.py --check: URDF and SDF OK; validate:
URDF / SRDF strict OK, SDF OK.

File: cad/robot/arm.urdf (robot description, URDF)
Before this commit: robot arm, 10 links, 9 joints
Links:
- link elbow_link: mass 0.911507 -> 0.920925
- link upper_arm_link: mass 1.318719 -> 1.317978
