Commit message: cad: the roll frame's end an octagon about the elbow axis, straight-sided with sharp corners
forearm_roll_block (the roll drive's frame on the elbow) was a teardrop seen along the elbow axis: an r 45 circle
round the elbow axis hulled up to the tower. Restyled to read more geometric: three outlines were previewed (an
octagon, a square end with 45-deg corners, a pointed hexagon), all keeping the rear line; the octagon was chosen,
with sharp edges (no chamfer: a cover will go over the open +N face later), the round bearing boss kept, and
j1_link's round end left round.

- lib/forearm/roll.py profile(): the circle becomes a regular octagon (RollDriveParams.end_sides 8), a flat on each
  axis end_r off the elbow axis (on j1_link's round end), its corners 48.7 out; hulled to the tower with sharp
  corners (Rectangle, not RectangleRounded), cut off at the front face and behind rear_line() - the line the round
  end's hull ran (tangent to the end_r circle and an r 3 circle in the tower's rear-top corner), which the elbow
  motor's board passes nearest at the elbow's lower limit; the octagon's corner behind it is cut off.
- RollDriveParams.tower_corner_r -> rear_line_r (same 3.0): it now only sets the rear line.
- tests/forearm/test_roll_drive.py: test_frame_features probes the end's two corners and the rear line; test_stack's
  bearing-boss rule reads "4 inside the frame's three sides" (no rounded corner to stay off).
- docs/forearm_roll.md, the docstrings: the octagonal end; docs/open_issues.md: the elbow-limit row names the rear
  line (move it in to lift the forearm further back), the print row: the end now rises off the bed in a 45-deg
  facet (the round end's support goes); a new row: the cover over the open +N face (planned, not designed, no
  fixings yet - the face stays flat, its edges sharp).

Numbers:
- forearm_roll_block: volume 367622.6 -> 376143.1 mm3 (+8520.5, +2.3 %), 466.9 -> 477.7 g PETG; bbox unchanged
  (80.0 x 149.0 x 83.8); reference/native/forearm_roll_block.step re-accepted (import_native.py --force).
- forearm_roll_drive EXPECTED: solid_volume 501078.896 -> 509599.438; stator 462818.248 -> 471338.79.
- elbow_link (arm.urdf, arm.sdf): mass 0.920925 -> 0.931746 kg; COM (0.004021, -0.015556, 0.018202) ->
  (0.003798, -0.01504, 0.018281); ixx 1.527059e-03 -> 1.558041e-03, iyy 8.080608e-04 -> 8.228793e-04,
  izz 1.444870e-03 -> 1.483188e-03, ixy 1.487957e-04 -> 1.558103e-04, ixz -2.183490e-05 -> -2.043727e-05,
  iyz 7.577451e-05 -> 7.254324e-05; robot/meshes/elbow_link.stl re-exported. The arm 6.480 -> 6.491 kg.
- Clearances unchanged: the elbow motor's board 2.27 mm off the frame at -47 deg (the rear line is the round
  end's); the base and the shoulder 30 mm or more off it with the arm folded back (shoulder at its upper limit).

Checks: hash gate against main's build (only forearm_roll_block, forearm_roll_drive, arm and
robot/links/elbow_link change), ./cadtool lint, pytest fast lane and full suite (1150 passed),
derive.py --check, validate arm.urdf / arm.srdf --strict and arm.sdf.

File: cad/robot/arm.urdf (robot description, URDF)
Before this commit: robot arm, 10 links, 9 joints
Links:
- link elbow_link: mass 0.920925 -> 0.931746

Commit message: cad: the roll frame opens through its bottom and back, its side closed; the roll's 6806 pair 19 mm apart
The roll frame (forearm_roll_block) was open on its whole side (+N) face - the motor dropped in from there, the board's
plugs rode down slots off it, the shaft and bearing 1 went into the bay through it - and a cover over it was planned.
The side face is now closed and the openings moved:

- The motor's pocket opens down through the octagon's bottom face: the motor and its board slide up into it
  motor_drop back (the pilot boss under the plate), then forward into the pilot hole. The shaft's slit through the
  plate runs from the pilot hole down to the bottom instead of out to the side.
- The motor is turned a quarter clockwise seen from the pulley side (motor_spin_deg 90 -> 0): its own connector and
  the board's motor header point down into the opening, their short wire there - no hole in the side for it.
- The board's two side plugs now face the walls (the side wall, the floor): a groove inside each wall from the plug
  down out through the bottom, plug_skin (1 mm) of wall outside; the motor slides up with them plugged, each cable
  bent straight down at its plug. That leaves 8.5 mm of straight room (layout.side_plug_room) against the measured
  MKS_PLUG_ROOM 10 mm straight out: test_sweeps gives these two plugs side_plug_room, and a new open_issues row asks
  for a fit check with the real plugs. The old plug slots off the pocket are gone.
- The side wall over the pocket (side_t) is as thick as the floor (web_t, 7 mm).
- The idler's M5 nut channel no longer runs out to the side face: closed at both ends, the nut goes in from the
  motor's pocket before the motor (RollIdlerParams.entry: a recess in the plate's inner face, which the motor's face
  then shuts). The idler keeps its M5 x 25.
- The shaft's bay is bored on through the frame's back (bay_r 25.6, the rear line) instead of opening on the side:
  the shaft, bearing 1 pressed on it, goes in along the axis from behind. The tower's rear in the profile is now its
  own parameter (tower_rear 0.75, it was the old bay floor less tower_wall), so the outline - the rear line the elbow
  motor's board passes at the elbow's lower limit - does not move. bay_clear and tower_wall are gone.

The roll's 6806 pair moves apart: the lip between their outer rings becomes a 12 mm spacer (lip 2 -> 12), the pair
9 -> 19 mm apart centre to centre, so each bearing takes the forearm's bending moment over twice the span (about
250 -> 120 N each with the forearm straight out and 200 g in the gripper, estimated from the URDF masses). Bearing 2
stays right under the 90T; bearing 1, the shaft and the hard stop move 10 mm back, the stop lug 2.34 mm inside the rear
line at any roll angle.

The rotor splits at bearing 1 now: the pulley's hub is the long piece - its Ø30.3 journal through bearing 2, then a
Ø29.9 neck (neck_dia, under the bearing's bore so bearing 2 slides over it) through the spacer to bearing 1's front
face (z_meet = z_lip) -, and the shaft is only the collar that holds bearing 1 (its journal through it, the shoulder,
the flange with the clamp's nuts and the stop lug). Each bearing is still pressed on its own journal from its own end
(99.5 mm^3 each, unchanged). The rotor clamp's screws grow M3 x 35 -> M3 x 45 (clamp_screw_len); they leave 1.0 mm of
wall along the pulley's neck (1.2 along the journal). The 20T, the belt, the 90T and the idler stay where they were.

Numbers:
- forearm_roll_block: 376.1 -> 325.4 cm3 (-50.7, about -64 g PETG); reference/native/forearm_roll_block.step accepted
- forearm_roll_shaft: 12.32 -> 11.89 cm3, 17.85 -> 16.85 mm long; reference/native/forearm_roll_shaft.step accepted
- forearm_roll_pulley: 25.94 -> 30.45 cm3, its hub 8 -> 19 mm below its shoulder
- forearm_roll_drive EXPECTED solid_volume 509599.438 -> 462895.938 (stator 471338.79 -> 420559.434,
  rotor 38260.648 -> 42336.503); leaves 13, solids 31 unchanged
- robot/arm.urdf + arm.sdf: elbow_link 0.931746 -> 0.867256 kg, forearm_link 0.567225 -> 0.572401 kg (their COM and
  inertia from derive.py); total mass 6.491 -> 6.432 kg; elbow_link and forearm_link meshes re-exported
- the elbow motor's board at the elbow's lower limit: 2.27 mm from the frame before, 2.91 mm now (it passes the
  back bore's rim); it passes 8.7 mm under the bottom between elbow +60 and +90 deg
- tools/bom.py's rotor clamp line follows clamp_screw_len (M3 x 45)

Docs: docs/forearm_roll.md (spec table, section 1, the stations, printing, the assembly sequence). docs/open_issues.md:
the side-cover row closed (the side face is closed); the frame-flex, rotor-pair, home-sensor and cable-route rows
updated; a row added for the side plugs' 8.5 mm.

Checks: the hash gate (only the three roll parts, the drive and the arm changed); ./cadtool pytest (fast lane and the
full suite) green; derive.py --check OK; validate arm.urdf / arm.srdf --strict, arm.sdf OK; lint clean.

File: cad/robot/arm.urdf (robot description, URDF)
Before this commit: robot arm, 10 links, 9 joints
Links:
- link elbow_link: mass 0.931746 -> 0.867256
- link forearm_link: mass 0.567225 -> 0.572401

Commit message: cad: the wrist's gripper to its outer side - the wrist bends down to -150, the elbow folds to 144
Asked from the CAD Viewer: the wrist should point down, and the elbow should fold further, its range taking
precedence over the other joints'. The elbow's upper limit (90) was a leftover of the old forearm wall, which no
longer reaches the upper arm; the gripper is what set the room after it. Previewed and approved first (scratch build,
renders, sweeps).

- lib/wrist/params.py WristRollParams.side (new, -1 [DESIGN]): the wrist roll axis R' - the gripper - sits
  WRIST_ROLL_OFFSET along wrist_link's -Y, the outer side (away from the upper arm when the elbow folds, the forearm
  turned), not +Y. The frame builds as the other side's mirror image (lib/wrist/layout.py module_frame_in_host, y_motor,
  frame_y_span; roll.py profile; link.py the bay's nut channel); the rotor and every bought row are placed, not
  mirrored (the belt's row turned -90). wrist_link 65566.928 mm3 unchanged, its box y -39.001..78.583 ->
  -78.583..39.001; the wrist roll drive's totals unchanged.
- lib/placements.py: the gripper's shift across wrist_link by side x centre_distance; reference/placements.json:
  wrist_roll_drive#1 re-resolved (mount_placements.py), world (-217.950, 360.459, -7.973) -> (-130.702, 402.851,
  -13.606).
- WRIST_PITCH_LIMITS_DEG (-74, 125) -> (-150, 38): the long range now bends the gripper down. Up, the wrist roll
  drive's tower meets the wrist-pitch motor (1.09 mm at +40, 3+ at +38); down, the gripper reaches the forearm roll's
  frame (1.78 mm at -160) and, the elbow at 0, the upper arm (touching by -158) - 3+ mm off both at -150 at any forearm
  and gripper roll.
- ELBOW_PITCH_LIMITS_DEG (-47, 90) -> (-47, 144): the upper set by the arm's own parts - 2 deg short of where the
  wrist-pitch motor's board, folded back with the shoulder at its upper limit, puts its side plug's room into the base
  (clear at 145, 55 mm3 at 146; clear to 148 with the shoulder at 64); the wrist body clears the base and j1_coupler
  by 1+ mm to 150 at any forearm roll and wrist pitch (touching by 153). The lower unchanged.
- ELBOW_GRIPPER_FREE_DEG 92 (new [DESIGN]): the gripper keeps 1 mm off the arm at any forearm roll and wrist pitch up
  to it (1+ mm at 94, touching j1_link by 97 with the wrist at -150); folded further a planner keeps it out - a new
  docs/open_issues.md row (the SRDF disables only adjacent pairs, so a planner checks those).
- tests: test_sweeps.py test_the_elbow_limits_keep_the_forearm_and_the_wrist_off_the_upper_arm (was ..._and_the_gripper_...):
  the forearm and the wrist body at the elbow's limits, the gripper at the lower and at ELBOW_GRIPPER_FREE_DEG; the
  elbow board's plug-room sweep takes the gripper up to ELBOW_GRIPPER_FREE_DEG; the wrist tests and test_placements
  follow side; test_roll_drive checks R' on the outer side; test_params_invariants locks the limits.
- robot/arm.urdf / arm.sdf (derive.py drafts): elbow_pitch upper 1.570796 -> 2.513274, wrist_pitch (-1.291544,
  2.181662) -> (-2.617994, 0.663225); wrist_roll origin xyz (0.026448, -0.048578, 0.027003) -> (0.026448, 0.048588,
  0.027002); wrist_pitch_link COM (0.000654, -0.009606, 0.014245) -> (0.000654, 0.009587, 0.014245), ixx 5.770768e-04
  -> 5.773343e-04, ixy 2.785436e-05 -> -2.814436e-05, ixz -4.143470e-06 -> -4.143395e-06, iyy 3.625183e-04 ->
  3.625179e-04, iyz 5.659935e-05 -> -5.650043e-05, izz 3.765258e-04 -> 3.767836e-04, mass 0.487734 unchanged;
  meshes/wrist_pitch_link.stl re-exported; the ledger says the gripper is the planner's past ELBOW_GRIPPER_FREE_DEG.
- Docs: docs/wrist_roll.md (which side, the module frame), docs/open_issues.md (the wrist pitch and elbow rows, the
  gripper's new row), docs/forearm_roll.md (no limit numbers), tests/AGENTS.md.

Hash gate: parts/wrist/wrist_link.step, assemblies/wrist_roll_drive.step and assemblies/arm.step changed, nothing
else. ./cadtool pytest: 1150 passed; derive.py --check OK; validate URDF / SRDF / SDF OK; lint clean.

File: cad/robot/arm.urdf (robot description, URDF)
Before this commit: robot arm, 10 links, 9 joints
Joints:
- joint elbow_pitch: limit lower=-0.820305 upper=1.570796 effort=5 velocity=1 -> lower=-0.820305 upper=2.513274 effort=5 velocity=1
- joint wrist_pitch: limit lower=-1.291544 upper=2.181662 effort=5 velocity=1 -> lower=-2.617994 upper=0.663225 effort=5 velocity=1
- joint wrist_roll: origin xyz=0.026448 -0.048578 0.027003 rpy=-1.570799 -0.055534 -1.570796 -> xyz=0.026448 0.048588 0.027002 rpy=-1.570799 -0.055534 -1.570796

Commit message: cad: the forearm roll rotor's clamp modelled - 4x M3 x 45 + 4 M3 nuts on the rotor
The roll rotor's clamp (RollDriveParams clamp_*: 4x M3 from the pulley's front face
through both pieces and both 6806 inner rings into nuts in the shaft's flange) had its
holes, head counterbores and nut pockets in the printed parts but no fasteners: the
screws and nuts were two tools/bom.py EXTRAS rows. They are parts now, placed in
forearm_roll_drive on the rotor (forearm_link), so the model, the totals, the buy list
and the inertials carry them.

- parts/joints/roll_clamp_screws: 4x M3 x 45 SHCS (ISO 4762), no reference (envelope,
  lib/fasteners.py shcs()), 1529.299 mm^3, MASS_G 12.0 g (ROLL_CLAMP_SCREWS_MASS_G).
  Row: turned over onto the counterbores' floor (z_clamp_head 46.75): the heads' tops
  0.25 under the pulley's face (z 49.75), the tips at the shaft's rear face (z 1.75).
- parts/joints/roll_clamp_nuts: 4x M3 hex nut (ISO 4032), no reference (hex_nut(), a
  corner radial as each pocket's slot holds it), 183.635 mm^3, MASS_G 1.44 g
  (ROLL_CLAMP_NUTS_MASS_G). Row at z_clamp_nut 2.75: on their seats at 5.15, 2 pitches
  short of the tips.
- No printed part changes. Fit: 0 mm^3 against every part of the drive, nothing else
  in the arm within 3 mm; the heads touch the pulley, the nuts the shaft, the shanks
  0.2 clear of the Ø3.4 holes; a nut turned 5 deg runs into the shaft's flange.
- tools/bom.py: the two clamp EXTRAS rows removed (now modelled buy rows, same counts).
- Locks: forearm_roll_drive EXPECTED leaves 13 -> 15, solids 31 -> 39, solid_volume
  462895.938 -> 464608.872; rotor leaves 2 -> 4, solids 2 -> 10, solid_volume
  42336.503 -> 44049.437 (stator unchanged); module tints bought 10 -> 12; the arm
  (tests/test_assembly.py) leaves 119 -> 121, solids 313 -> 321, bought leaves 80 -> 82; tests/test_bom.py
  placed leaves 119 -> 121, buy list 52 parts / 80 pieces -> 54 / 82; MULTI_BODY +2.
  New tests/forearm/test_roll_clamp.py locks both parts' numbers and the fit.
- forearm_link (robot/arm.urdf, arm.sdf): mass 0.572401 -> 0.585848 kg, COM
  (-0.005708, -0.000049, 0.093041) -> (-0.005577, -0.000048, 0.091495) m, ixx
  9.688013e-04 -> 1.032887e-03, iyy 1.031759e-03 -> 1.096272e-03, izz 2.787129e-04 ->
  2.811862e-04, ixy 3.206490e-06 -> 3.202921e-06, ixz -9.845830e-05 -> -9.340406e-05,
  iyz 1.301759e-06 -> 1.343907e-06; the arm 6.4317 -> 6.4451 kg. Its mesh re-exported.
  (derive.py --check checks the SDF's joints only, so its inertial was copied from
  --sdf-draft by hand like the URDF's.)
- Hash gate: of the 99 STEPs only assemblies/arm.step, assemblies/forearm_roll_drive.step
  and robot/links/forearm_link.step changed (+ the two new part STEPs).
- Docs: docs/forearm_roll.md (the clamp row, the link masses, assembly steps 4-5),
  docs/open_issues.md (the nut-pocket row: these four nuts modelled), robot/AGENTS.md,
  tests/AGENTS.md, the URDF ledger.

File: cad/robot/arm.urdf (robot description, URDF)
Before this commit: robot arm, 10 links, 9 joints
Links:
- link forearm_link: mass 0.572401 -> 0.585848

Commit message: cad: removable back panel on the forearm roll frame - flush, held by magnets
The roll shaft sat behind a bare Ø51.2 hole in the frame's slanted rear face. The
back now takes a removable panel: lift it off and the shaft, its clamp nuts and the
stop post are open to reach; put it back and the back is closed, flush.

- forearm_roll_block: the rear face stepped BackPanelParams.t (2.5) across its full
  width, from the tower's top down to `bottom` (56 below the roll axis' point, along
  the face); the bay's opening grown down below its bore to `opening_bottom` (R6
  corners, `opening_depth` 12 in - 8.8 of frame left over the motor's pocket); 4
  magnet pockets in the step's floor (3.7 of wall to the bay, 3.4 to the side faces).
- forearm_roll_back_panel (new, printed, no reference): the plate in the step, its
  outer face ON the rear line; relieved run_gap off the shaft's rear face and its
  lug's sweep (1.2 mm at its thinnest, over the bay's top edge); a U rim on its inner
  face locates it in the opening; prints outer face down.
- roll_back_magnets (new, bought, no reference): 4 pairs of 6 x 2 mm N52 discs, one
  in the frame's step, one in the panel, each pressed to its pocket's bottom.
- lib/forearm/roll.py back_face / back_point / back_opening / build_back_panel;
  lib/forearm/params.py BackPanelParams (RollDriveParams.back); lib/params.py
  NDFEB_DENSITY, ROLL_BACK_MAGNETS_MASS_G.
- The forearm's cables no longer pass through the bay (nothing passes the panel):
  their route is open - the docs/open_issues.md cable-route row rewritten, the
  rotor's Ø18 bore left as it is. A new estimates row for the panel's hold and the
  magnets' stray field (on-axis estimate: ~0.3 mT at the roll motor's MKS encoder,
  ~0.5 mT at the elbow motor's near the elbow's lower limit, ~2 mT at the home
  sensor's site); the home-sensor row keeps the chip 20 mm off the top magnets.

The elbow's range is unchanged: the panel is flush, so the elbow motor's board at
-47 deg passes it at 2.27 mm (2.91 to today's frame, over the open hole) and comes
within 1 mm at -49.0 deg - the figures docs/open_issues.md already gives for the
rear line.

Numbers:
- forearm_roll_block 325363.751 -> 306232.873 mm3 (faces 126 -> 144); its native
  reference re-accepted (tools/reference/import_native.py --only forearm_roll_block
  --force)
- forearm_roll_back_panel 13702.812 mm3 (17.4 g); roll_back_magnets 8 solids,
  452.389 mm3 (3.4 g)
- forearm_roll_drive EXPECTED: leaves 15 -> 17, solids 39 -> 48, volume 464608.872 ->
  459633.195; stator 11 -> 13, 29 -> 38, 420559.434 -> 415583.758 (rotor unchanged)
- elbow_link mass 0.867256 -> 0.863755 kg, COM and inertia re-derived (arm.urdf,
  arm.sdf), its mesh re-exported
- arm leaves 121 -> 123, solids 321 -> 330, link tints 82/39 -> 83/40; the drive's
  tints 12/3 -> 13/4; bom printed (33, 39) -> (34, 40), bought (54, 82) -> (55, 83)

Checks: ./cadtool pytest (fast lane 716 passed; full suite 1181 passed + the two
lock tests re-run after the bumps); the hash gate - only the frame, the drive and the
arm changed (eight more STEPs differed in bytes only, same geometry per inspect
diff); derive.py --check OK; validate arm.urdf / arm.srdf --strict, arm.sdf OK;
snapshots looked at; new tests/forearm/test_roll_back_panel.py.

File: cad/robot/arm.urdf (robot description, URDF)
Before this commit: robot arm, 10 links, 9 joints
Links:
- link elbow_link: mass 0.867256 -> 0.863755

Commit message: cad: j2_link's web dropped 13 mm toward its belt side, level with the roll wall's bottom
The user wanted the forearm's web further toward its belt side, into the face of the roll wall
that hung below it, so the wrist belt and its pulleys sit further from the roll axis. Chosen
from a preview of 4 / 8 / 13 mm: 13, the web's underside level with the wall's round bottom.

The roll wall stays on the roll axis; the web, the wrist boss and everything on them drop
WEB_DROP (lib/forearm/params.py, derived: LEGACY web z0 - the wall's bottom = 13) along the
wrist_pitch axis toward the belt side:
- DEFAULT web z 8..19 -> -5..6; boss seat_z1 / z1 27.5 -> 14.5, lip_z (17, 19) -> (4, 6);
  roll_end.wrist_belt_z 0.3 -> -12.7 (J2_BELT_Z); J2_MOTOR_WEB_FACE_Z 19 -> 6;
  IdlerParams.nut_floor 11 -> -2 (3 of web under the nut, as before).
- The wrist and all beyond it drop with the web: the j2_link LinkShift gets normal_z =
  DEFAULT - LEGACY web z0 (-13) along j2_link's +Z (lib/placements.py), so the wrist bearings,
  the 90T, j3_coupler, wrist_link, the wrist roll drive and the gripper follow; the motor, its
  board and screws, the 20T, the belt and the idler kit follow the web through lib/mounts.py.
- The forearm roll axis no longer passes through the wrist centre: it crosses the wrist_pitch
  axis 13 mm from it (the gripper rides 13 mm off the roll axis). robot/frames.py, the roll
  drive's test and docs say so.
- The web's foot corners, now level with the round bottom, would reach 42.4 from the roll axis
  where the roll tensioner's screw head passes (38.05 out): the wall's elbow-side band
  (RollEndParams.relief_t 5.3) is cut back to relief_r 36.0 about the roll axis; its
  wrist-side 2.7 keeps the whole foot. Wall to that head: 3.57 -> 2.05 mm (the check asks 2).
- The wall's bottom M3's head (z 9.5) now clears the web's top face (0.25 over it with the
  0.5 clearance): no channel under the web any more (screws_under_the_web is empty); the
  wrist-pitch motor stands in front of all four wall heads (was three).

Measured:
- j2_link 98814.7 -> 101420.4 mm^3, 125.5 -> 128.8 g; its lowest point is now the wrist idler's
  rib (z -8.2), under the wall's bottom.
- forearm_link 0.585848 -> 0.589157 kg, COM x -0.005577 -> 0.005535 (URDF / SDF inertials
  copied from derive.py's drafts); wrist_pitch joint origin x -0.016997 -> -0.003997.
- The wrist belt's plane 24.7 -> 37.7 mm from the roll axis; j2_link to the upper arm at the
  elbow limits, any roll: 26.1 -> 21.8 mm.
- Hash gate vs main: j2_link, arm and the forearm_link link STEP changed; base,
  base_motor_mount, j1_link, j1_motor_leg, gripper_j3_connector, cycloidal_drive and gripper
  changed bytes only - cadgen's edge / vertex name labels, the same geometry by
  ./cadtool inspect diff.

Checks: ./cadtool lint, ./cadtool pytest (full suite, -n 4), derive.py --check, ./cadtool
validate on arm.urdf / arm.srdf / arm.sdf, mount_placements.py re-run, forearm_link mesh
re-exported, snapshots looked at.

File: cad/robot/arm.urdf (robot description, URDF)
Before this commit: robot arm, 10 links, 9 joints
Links:
- link forearm_link: mass 0.585848 -> 0.589157
Joints:
- joint wrist_pitch: origin xyz=-0.016997 -0.000007 0.165 rpy=-1.570808 -1.271748 1.570808 -> xyz=-0.003997 -0.000007 0.165 rpy=-1.570808 -1.271748 1.570808
