Commit message: cad: j1 fork legs one size, straight-sided, their posts inside the disc's rim
The fork's two legs each were a round top on a 50 mm post - the hub leg a Ø70.3 disc, the motor leg a Ø90 ring -
and the user found them looking like lollipops: they wanted the legs of one uniform width. Previewed as scratch
builds (claude.ai artifact, two rounds): the user picked both legs alike at the motor ring's size (over each leg at
its own width), then asked that the legs not go over the round base; of the two versions shown for that (45 degree
feet only, or the posts cut to the rim as well) they chose the posts inside the rim.

What changes (lib/yaw_coupler/, DEFAULT only - LEGACY and the reference match are untouched):
- ForkParams.hub_plate_r (35.15, the hub's own od / 2) and leg_half_z (25) are gone: both legs' round tops are
  plate_r (45) and their posts plate_r either side (50 -> 90 wide), straight sides. The hub leg's disc Ø70.3 -> Ø90,
  9.85 past the hub's od; the hub's counterbores 6.45 -> 16.3 inside its edge.
- New ForkParams.foot_deg (45) and layout.fork_leg_bound(): the posts stay inside the disc's rim about the base_yaw
  axis - within the disc's drafted side to its top edge (r 54.193 at y 19.988), the feet out at 45 degrees to the
  rim (r 57.981, the disc's underside) 3.788 higher, then the rim on up. body._leg_room() keeps each leg's round top
  whole; _fork() and build_motor_leg() cut their leg to it. The posts' sides follow the rim: 87.6 wide at the legs'
  inner faces, 70.6 at their outer faces. Only the round tops pass the rim, at the drive's axis (corners r 64.35):
  the motor ring could not stay inside - its wall beside the bore would be 0.1 at its outer face - and it already
  reached that far before this change.
- j1_coupler 218829.632 -> 243739.485 mm3 (PETG 277.9 -> 309.5 g); j1_motor_leg 43831.851 -> 53162.870 mm3
  (55.7 -> 67.5 g); the two +34240.9 mm3, +43.5 g. Bounding boxes: the coupler's top 125.25 -> 135.10 (its disc at
  the motor leg's height), the motor leg's unchanged.
- reference/placements.json (mount_placements.py): j1_motor_leg#1 solid_volume 43831.851 -> 53162.87; expected
  solid_volume 2336779.808 -> 2346110.827 (solids and leaves unchanged).
- shoulder_link inertial (arm.urdf, arm.sdf, from derive.py's drafts): mass 1.408024 -> 1.451510 kg; COM
  (-0.000741, 0.014089, -0.021707) -> (-0.000687, 0.013095, -0.021727); ixx 3.898356e-03 -> 4.057553e-03, iyy
  2.908733e-03 -> 3.007590e-03, izz 2.137678e-03 -> 2.290222e-03, ixy 6.098559e-05 -> 6.472020e-05, ixz
  2.177568e-05 -> 1.974061e-05, iyz -4.257543e-04 -> -3.997381e-04. The robot's total mass 6.442 -> 6.485 kg.
  robot/meshes/shoulder_link.stl re-exported.
- Tests (tests/yaw_coupler/test_j1_coupler.py): the hub-disc-is-the-hub's-od rule replaced (plate_r 9.85 past the
  hub, counterbores 16.3 inside), the bound's profile and the ring's 0.1 wall pinned; the slow probes check the posts'
  sides on the rim, the 45 degree feet, nothing past the disc's side below its top face, the round tops whole past
  the rim, the outer-face draft on its own cone; the motor leg's volume lock 43831.851 -> 53162.870.
- Docs: the ForkParams / body / layout docstrings, the j1_coupler and j1_motor_leg docstrings, lib/AGENTS.md,
  docs/cycloidal_drive.md, docs/open_issues.md (the fork's shapes row). cad/AGENTS.md Gotchas: a source edited while
  a gen runs can leave the arm's document holding the old geometry under the new key (seen on this branch: the hash
  gate passed while the arm still had the old legs; gen --force cleared it).

Checks: ./cadtool lint clean; ./cadtool pytest: 1180 passed and 3 failed on the locks above (test_assembly's arm
total, test_robot's shoulder_link mesh and link masses), all 3 passing after the bumps; the fast lane (716) and
test_placements / test_bom again after placements.json. Hash gate (the arm built in this worktree before the edit):
geometry changed only in j1_coupler, j1_motor_leg and the arm; the forced rebuild also rewrote the bytes of base,
base_motor_mount, j1_link, cycloidal_eccentric_shaft, gripper_j3_connector, cycloidal_drive and gripper -
inspect diff: the same geometry (tol 1e-6). No clash with any other part in the rest pose (scratch overlap check);
the shoulder's sweep in test_sweeps passes. derive.py --check clean; validate arm.urdf / arm.srdf --strict and
arm.sdf OK. Snapshots of the arm, the shoulder link from both sides and the two parts looked at.

File: cad/robot/arm.urdf (robot description, URDF)
Before this commit: robot arm, 10 links, 9 joints
Links:
- link shoulder_link: mass 1.408024 -> 1.451510

Commit message: cad: j1_link slimmed - 18 deep, 76 wide, its elbow end R36
The upper arm's solid slab was still the old plate's full outline, 23 deep and 90 wide with an R45 elbow end. It is
slimmed for mass, which the shoulder's cycloidal drive carries: the size picked from a preview of depth, width and
elbow-end options, the roll frame left as it is.

- Depth: ElbowParams.relief_y -1 -> -6, the recess floor - the slab's top level with the upper 6806's top, as deep as
  the elbow's bearing stack (23 -> 18); no recess is left (link.py _cut_elbow_stack skips a recess whose floor is the
  top face).
- Plan: ArmParams width 76 (the plate's 90), end_r 36 (45), bend_r 20. link.py _outline: the slab keeps its width over
  the elbow idler's slots (layout.py slab_taper_x, 125.2 along the link) and tapers straight onto the narrower end (a
  hull of the two), the bend R20; a wider end it flares into through R20 fillets, an end as wide as the slab gives the
  plate's stadium. Symmetric about the centreline.
- The roll frame is unchanged: its octagonal end (flats R45) now overhangs the arm's R36 end by 9; its underside rides
  11.0 over the arm's flat top (6.0), its dust lip 6 over it (1), its boss 2.0 (FACE_GAP, as before). The elbow's
  6806s are -2RS.

Rules changed on purpose (they held the old size, not a clearance):
- tests/forearm/test_roll_drive.py: the frame's end_r == the arm's round end -> >= (UPPER_ARM_END_R 45 -> 36);
  UPPER_ARM_FACE_Z -11 -> -16, UPPER_ARM_RECESS removed (the boss and the journal's edge are measured over the flat
  top, at the old recess floor's height).
- tests/upper_arm/test_elbow_idler.py: slab past the idler nut slot's outer end >= 10 -> >= 8 (8.1 at 76 wide), and
  the slab keeps its width over the slots (slab_taper_x).
- tests/upper_arm/test_j1_link.py: the probes follow the new outline and top; the old cap's elbow sockets now fall
  outside the slab.

Numbers:
- j1_link: volume 372030.418 -> 289599.124 mm^3, faces 192 -> 196, PETG mass 472.5 -> 367.8 g (-104.7 g), bbox max X
  215 -> 206 (size 279.6 x 52 x 116.0 -> 270.6 x 52 x 116.0).
- Slab beside the elbow motor's hole 23.4 -> 16.4, past the idler nut slot 15.1 -> 8.1, round the elbow seat (Ø42.2)
  23.9 -> 14.9; the 108T's flange (r 35.3) 0.7 inside the end's edge (9.7).
- arm.step: volume 3254850.174 -> 3172418.880 mm^3; only j1_link differs (inspect diff).
- upper_arm_link inertial (arm.urdf, arm.sdf): mass 1.317978 -> 1.213291 kg; COM (0.060932, -0.000006, 0.033589)
  -> (0.054658, -0.000024, 0.034877) m; ixx 1.684781e-03 -> 1.523279e-03, iyy 6.388052e-03 -> 5.503463e-03,
  izz 6.774821e-03 -> 5.789567e-03, ixy 1.175714e-06 -> 2.643311e-06, ixz 7.513569e-04 -> 6.193402e-04,
  iyz -2.876412e-06 -> -3.076585e-06; the URDF's total mass 6.489 -> 6.384 kg. robot/meshes/upper_arm_link.stl
  re-exported.
- Its gravity torque on the shoulder, the arm level: 0.137 N.m less (the 104.7 g taken off sat 134 mm out).
- Print (docs/open_issues.md): ~229 -> ~220 square turned 45 deg on the bed; ~1,090 -> ~740 mm^2 facing down below 45
  deg (dfam-check orientations, rot_plus_90_x: the hub end down).

Checks: the hash gate (a forced arm rebuild: the other rewritten STEPs are the same geometry by inspect diff), the
fast lane and the full suite (1184 passed, the sweeps included), derive.py --check, validate --strict (URDF, SRDF,
SDF), snapshots of the arm, the upper arm and a centreline cut looked at.

File: cad/robot/arm.urdf (robot description, URDF)
Before this commit: robot arm, 10 links, 9 joints
Links:
- link upper_arm_link: mass 1.317978 -> 1.213291

Commit message: cad: the elbow pulley 108T -> 90T on a stock 280 belt, a 5:1 gearbox to carry the reduction
Why: a 5:1 planetary gearbox (StepperOnline EG17-G5) was bought for the elbow motor, so the belt no longer has to
carry the elbow's whole reduction and its driven pulley can shrink. Chosen from a to-scale preview (scratch builds of
each size against the repo's idler rules and clearance tests): on a stock belt only 90T and 80T fit - 78T and smaller
need the motor moved toward the shoulder, where its board meets the cycloidal drive (78T, 6 mm back) or the motor
runs into j1_link (76T, 7 mm back). 90T keeps the motor where it is and is the wrist's own pulley part.

The pulley: the elbow's driven pulley is the 90T again (gt2_pulley_90t, DEFAULT). gt2_pulley_108t, its test, lib/pulley
ELBOW and GT2_PULLEY_108T_TEETH are removed. The mount gt2_pulley_90t#3 (hosted on the retired gt2_pulley_90t#1,
PULLEY_SEAT_SHIFT out, turned pulley_bolt_deg) replaces gt2_pulley_108t#1; its label is gt2_pulley_90t:j2 (the j2 / j3
roles of the two 90Ts again), elbow_link carries it. Flange 70.647 -> 59.188 mm; volume 31390.961 -> 23975.641 mm^3
(39.9 -> 30.4 g in PETG). ELBOW_RATIO = GT2_PULLEY_90T_TEETH / GT2_PULLEY_20T_TEETH = 4.5 (was 5.4): the belt alone.

The gearbox is not modelled: docs/open_issues.md replaces the elbow's second-stage row with one for it (its seat on
j1_link's web, the motor and board further out on +N, an 8 mm keyed 20T, the clearances again, ELBOW_RATIO with it;
the joint's reduction becomes 5 x ELBOW_RATIO).

The belt: ELBOW_BELT 300 -> 280. Open loop 294.2 -> 272.4. elbow_belt volume 1135.449 -> 1059.849 mm^3, bbox
119.496 x 69.507 -> 113.766 x 58.048 mm.

The tensioner: ElbowIdlerParams.along stays 29.1; slot_z (-4.0, 25.1) -> (-1.7, 22.4) (in to 3.0 off the far strand's
teeth, out past touching the open loop's strand). The slot takes 272.4 .. 287.3 (was 294.2 .. 315.7); on the 280 the
idler sits at z 5.114 (was 9.857). The idler's flange is 10.57 off the 90T's flange at its place (was 5.56 off the
108T's), 10.34 at the slot's inner end, 10.31 nearest. The slab runs 10.8 past the nut slot's outer end (was 8.1).
j1_link volume 289599.124 -> 290249.374 mm^3 (367.8 -> 368.6 g; the slots shorter).

Numbers that changed:
- placements.json expected solid_volume 2346110.827 -> 2338619.907 (mount_placements.py).
- print list: 34 -> 33 parts (40 to print, unchanged: the 90T 1 -> 2, the 108T gone).
- upper_arm_link: mass 1.213291 -> 1.213966 kg, COM (0.054658, -0.000024, 0.034877) -> (0.054685, 0.000017,
  0.034868), ixx 1.523279e-03 -> 1.522482e-03, ixy 2.643311e-06 -> -6.808605e-07, ixz 6.193402e-04 -> 6.195951e-04,
  iyy 5.503463e-03 -> 5.503910e-03, iyz -3.076585e-06 -> -1.251264e-06, izz 5.789567e-03 -> 5.788954e-03; mesh
  re-exported (66 solids, 528970.7 mm^3).
- elbow_link: mass 0.863755 -> 0.854338 kg, COM (0.004758, -0.017876, 0.018815) -> (0.004811, -0.018073, 0.019498),
  ixx 1.395560e-03 -> 1.351127e-03, ixy 1.639097e-04 -> 1.630992e-04, ixz -2.578565e-05 -> -2.297989e-05,
  iyy 8.076585e-04 -> 7.660524e-04, iyz 9.554408e-05 -> 8.501111e-05, izz 1.282434e-03 -> 1.269396e-03; mesh
  re-exported (47 solids, 442254.4 mm^3).
- the robot: 6.384 -> 6.375 kg.

The hash gate names arm.step, j1_link.step, elbow_belt.step and the upper_arm_link / elbow_link link STEPs
(gt2_pulley_108t.step gone). The forced rebuild also rewrote base, base_motor_mount, j1_coupler, j1_motor_leg,
gripper_j3_connector, cycloidal_drive, gripper and the base_link / shoulder_link / wrist_roll_link link STEPs:
inspect diff reads them as the same geometry. Checks: fast lane 713 passed; full suite 1174 passed + the j1_link lock
bumped and re-run; derive.py --check URDF and SDF OK; validate URDF / SRDF strict OK, SDF OK; lint clean.

File: cad/robot/arm.urdf (robot description, URDF)
Before this commit: robot arm, 10 links, 9 joints
Links:
- link elbow_link: mass 0.863755 -> 0.854338
- link upper_arm_link: mass 1.213291 -> 1.213966

Commit message: cad: the roll frame's octagonal end R45 -> R42
The roll frame's octagon about the elbow axis was sized to the upper arm's old R45 round end; since the arm was slimmed
to an R36 end it stood 9 proud of it all round. It comes in to R42, close to the least the frame allows: the roll
motor's pocket keeps 5 of wall outside its top corners (36.75 off the elbow axis: 41.75), and the lip (Ø72) 5 inside
the flats (41). The frame cannot match R36 - its motor's pocket alone reaches past it.

- RollDriveParams.end_r 45 -> 42. The rear line, tangent to the end_r circle, turns -63.32 -> -65.18 deg; the back
  panel and its magnets, flush on it, follow. The octagon's lower front facet now cuts the front of the motor's plate
  back below 25.6 under the elbow axis (the motor's face and its screws well clear): test_frame_features' slit probe at
  25 under the axis instead of 30.
- reference/native/forearm_roll_block.step re-accepted (import_native.py --force), the manifest with it.
- The elbow's lower limit's notes (lib/params.py ELBOW_PITCH_LIMITS_DEG, docs/open_issues.md) were out of date: they
  had the frame 2.3 off the elbow motor's board at -47 and 1 mm off it at -49. Measured, its nearest is the elbow motor
  itself: 6.45 at -47 and 1 mm at -55.5 with R45; with R42 8.4 at -47 and 1 mm at -58.0. Past -47 nothing is swept.
- The frame's docstring had its underside 6.0 over j1_link's top (11.0 since the arm was slimmed).

Numbers:
- forearm_roll_block: volume 306232.873 -> 285909.451 mm^3 (PETG 388.9 -> 363.1 g), its corners 48.7 -> 45.5 off the
  elbow axis, 9 -> 6 beyond the arm's end.
- forearm_roll_back_panel: 13702.812 -> 13607.761 mm^3, bbox min (-29.9, -50.981139, -38.230792) -> (-29.9, -51.693655,
  -35.47194), size (59.8, 80.881139, 42.878529) -> (59.8, 81.593655, 40.012516); roll_back_magnets (452.389) bbox min
  (-26.5, -48.528686, -36.167118) -> (-26.5, -49.126433, -33.513521), size (53.0, 75.154777, 40.572188) -> (53.0,
  76.186489, 38.238522).
- The rules on the end: the motor pocket's wall 8.25 -> 5.25 (>= 5), the lip's 9.0 -> 6.0 (>= 5), the shaft's stop lug
  inside the rear line 2.34 -> 2.23 (>= 2).
- forearm_roll_drive EXPECTED solid_volume 459633.195 -> 439214.722, the stator's 415583.758 -> 395165.284 (the rotor's
  44049.437 as it was); arm.step volume 3172418.880 -> 3152000.406 mm^3, only those three leaves differ (inspect diff).
- elbow_link inertial (arm.urdf, arm.sdf): mass 0.863755 -> 0.837824 kg; COM (0.004758, -0.017876, 0.018815) ->
  (0.005724, -0.01841, 0.018624) m; ixx 1.395560e-03 -> 1.352909e-03, iyy 8.076585e-04 -> 7.578529e-04, izz
  1.282434e-03 -> 1.210698e-03, ixy 1.639097e-04 -> 1.550444e-04, ixz -2.578565e-05 -> -3.094294e-05, iyz 9.554408e-05
  -> 9.839554e-05; the URDF's total mass 6.384 -> 6.358 kg; robot/meshes/elbow_link.stl re-exported.

Checks: the hash gate (a forced arm rebuild: the other rewritten STEPs the same geometry by inspect diff), the fast
lane, the full suite (1184: the sweeps included; the 6 locks it named bumped and re-run), derive.py --check,
validate --strict (URDF, SRDF, SDF), snapshots of the arm and the roll drive looked at.

File: cad/robot/arm.urdf (robot description, URDF)
Before this commit: robot arm, 10 links, 9 joints
Links:
- link elbow_link: mass 0.863755 -> 0.837824
